File: Kicad/mini/pic16bit.kicad_pcb (KiCad board)
At the start: 2 copper layers, 80 x 100 mm, 88 parts, among them IC201 TLV1117-33, IC202 dsPIC33/PIC24F, IC301 CAT4002A, IC302 MCP2221A, K101 PE-450-4X6X-BLACK, K201 *Power & UART, K202 MCU 1, K203 MCU 1, K204 ICSP, K205 MCU 2, K206 MCU 2, K301 HARWIN-254-F-1X08-VERTICAL, K302 HARWIN-254-F-1X06-VERTICAL, P301 PIHER-PT10MV-10K, P302 PIHER-PT10MV-10K

Commit message: Update Mini
Parts:
- IC202: value dsPIC33/PIC24F -> MICROCHIP-PIC24FJ64GA102-ISP
- IC301: value CAT4002A -> ONSEMI-CAT4002A-SOT-23
- IC302: value MCP2221A -> MICROCHIP-MCP2221A-ISL
- K301: footprint tronixio:zzHARWIN-M20-782084x -> tronixio:HARWIN-M20-782084x
- R201, R202, R203, R204, R205, R301, R302, R303, R304, R305, R306, R307, R308, R309, R310, R311, R312, R313, R314, R315, R316, R317, R318, R319, R320: footprint tronixio:RESISTOR-1206 -> tronixio:LED-1206

Commit message: Update
Parts:
- IC301: value ONSEMI-CAT4002A-SOT-23 -> CAT4002A
- IC302: value MICROCHIP-MCP2221A-ISL -> MCP2221A
- R201, R202, R203, R204, R205, R301, R302, R303, R304, R305, R306, R308, R309, R310, R311, R312, R313, R314, R315, R316, R317, R318, R319, R320: footprint tronixio:LED-1206 -> tronixio:RESISTOR-1206
- R307: value 2K4 -> 10K; footprint tronixio:LED-1206 -> tronixio:RESISTOR-1206

Commit message: Update Kicad
Parts:
- added TP203: KEYSTONE-2000-3, tronixio:KEYSTONE-2000-3, F.Cu at (70.5, 90.5)
- IC202: footprint tronixio:DIP-28-W762 -> tronixio:DIP-28-W762-SOCKET
- moved JP204 9.79 mm to (128.0, 95.5), turned to 180 degrees
- moved C206 7.08 mm to (135.6, 93.2)
- moved JP205 1.23 mm to (131.8, 94.5)
- moved S201 1.11 mm to (70.5, 98.1)
- moved TP201 0.50 mm to (81.5, 143.5)
- moved TP202 0.50 mm to (132.5, 143.5)
- moved C202 0.25 mm to (82.0, 103.8)
- moved R201 0.25 mm to (84.5, 103.8)
- moved R202 0.25 mm to (87.0, 103.8)
Routing:
- net Net-(IC202-Pad19): track 46.9 -> 29.3 mm, vias 0 -> 1
- net +3V3: track 415.7 -> 402.9 mm
- net Net-(IC202-Pad20): track 40.5 -> 39.3 mm
- net Net-(IC302-Pad4): track 12.6 -> 11.9 mm
- net Net-(C206-Pad1): track 5.03 -> 4.34 mm

Commit message: Update Kicad
Connections:
- IC202 pad 5: PGC/UTX/RB1 -> /HID/PGC/URX/RB1
- JP303 pad 2: PGC/UTX/RB1 -> /HID/PGC/URX/RB1
- K202 pad 5: PGC/UTX/RB1 -> /HID/PGC/URX/RB1
- K203 pad 5: PGC/UTX/RB1 -> /HID/PGC/URX/RB1
Routing:
- net PGC/UTX/RB1: track 134.5 -> 0.00 mm, vias 2 -> 0
- net /HID/PGC/URX/RB1: track 0.00 -> 78.5 mm, vias 0 -> 1
Changed lines of the file:
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@@
   (net 69 "Net-(IC202-Pad25)")
   (net 70 "Net-(IC202-Pad26)")
+  (net 71 "/HID/PGC{slash}URX{slash}RB1")
   (footprint "tronixio:NHD-C0220BIZ" locked (layer "F.Cu")
     (at 109 69)
@@
       (net 48 "PGD{slash}UTX{slash}RB0") (pinfunction "Pin_4") (pintype "passive"))
     (pad "5" thru_hole circle locked (at 0 10.16 90) (size 1.8 1.8) (drill 0.7) (layers *.Cu *.Mask)
-      (net 49 "PGC{slash}UTX{slash}RB1") (pinfunction "Pin_5") (pintype "passive"))
+      (net 71 "/HID/PGC{slash}URX{slash}RB1") (pinfunction "Pin_5") (pintype "passive"))
     (pad "6" thru_hole circle locked (at 0 12.7 90) (size 1.8 1.8) (drill 0.7) (layers *.Cu *.Mask)
       (net 52 "Net-(IC202-Pad6)") (pinfunction "Pin_6") (pintype "passive"))
@@
       (net 30 "Net-(IC302-Pad6)") (pinfunction "1") (pintype "passive"))
     (pad "2" thru_hole circle locked (at 0 2.54) (size 1.8 1.8) (drill 0.8) (layers *.Cu *.Mask)
-      (net 49 "PGC{slash}UTX{slash}RB1") (pinfunction "2") (pintype "passive"))
+      (net 71 "/HID/PGC{slash}URX{slash}RB1") (pinfunction "2") (pintype "passive"))
     (model "${KICAD6_USER_3DMODEL_DIR}/Header/HARWIN-M20-999024x.wrl"
       (offset (xyz 0 0 0))
@@
       (net 48 "PGD{slash}UTX{slash}RB0") (pinfunction "RB0/PGD1") (pintype "bidirectional"))
     (pad "5" thru_hole oval locked (at 0 10.16 90) (size 2.4 1.6) (drill 0.7) (layers *.Cu *.Mask)
-      (net 49 "PGC{slash}UTX{slash}RB1") (pinfunction "RB1/PGC1") (pintype "bidirectional"))
+      (net 71 "/HID/PGC{slash}URX{slash}RB1") (pinfunction "RB1/PGC1") (pintype "bidirectional"))
     (pad "6" thru_hole oval locked (at 0 12.7 90) (size 2.4 1.6) (drill 0.7) (layers *.Cu *.Mask)
       (net 52 "Net-(IC202-Pad6)") (pinfunction "RB2") (pintype "bidirectional"))
@@
     (fp_arc (start -0.3 4.4) (mid -0.923087 4.342349) (end -1.5 4.1) (layer "F.Fab") (width 0.1))
     (fp_arc (start 0.9 -5.2) (mid 4.903738 -1.844893) (end 4 3.3) (layer "F.Fab") (width 0.1))
-    (fp_arc (start 1.5 4.1) (mid 0.923087 4.342349) (end 0.3 4.4) (layer "F.Fab") (width 0.1))
+    (fp_arc (start 1.5 4.1) (mid 0.923087 4.34235) (end 0.3 4.4) (layer "F.Fab") (width 0.1))
     (fp_circle (center 0 0) (end 1.6 0) (layer "F.Fab") (width 0.1) (fill none))
     (fp_circle (center -2.5 5.3) (end -1.5 5.3) (layer "F.Fab") (width 0.1) (fill none))
@@
       (net 48 "PGD{slash}UTX{slash}RB0") (pinfunction "Pin_4") (pintype "passive"))
     (pad "5" thru_hole circle locked (at 0 10.16 90) (size 1.8 1.8) (drill 0.8) (layers *.Cu *.Mask)
-      (net 49 "PGC{slash}UTX{slash}RB1") (pinfunction "Pin_5") (pintype "passive"))
+      (net 71 "/HID/PGC{slash}URX{slash}RB1") (pinfunction "Pin_5") (pintype "passive"))
     (pad "6" thru_hole circle locked (at 0 12.7 90) (size 1.8 1.8) (drill 0.8) (layers *.Cu *.Mask)
       (net 52 "Net-(IC202-Pad6)") (pinfunction "Pin_6") (pintype "passive"))
@@
     (fp_line (start -1.5 5.3) (end 1.5 5.3) (layer "F.Fab") (width 0.1))
     (fp_arc (start -4 3.3) (mid -4.903738 -1.844892) (end -0.9 -5.2) (layer "F.Fab") (width 0.1))
-    (fp_arc (start 1.5 4.1) (mid 0.923087 4.342349) (end 0.3 4.4) (layer "F.Fab") (width 0.1))
+    (fp_arc (start 1.5 4.1) (mid 0.923087 4.34235) (end 0.3 4.4) (layer "F.Fab") (width 0.1))
     (fp_arc (start 0.9 -5.2) (mid 4.903738 -1.844893) (end 4 3.3) (layer "F.Fab") (width 0.1))
     (fp_arc (start -0.3 4.4) (mid -0.923087 4.342349) (end -1.5 4.1) (layer "F.Fab") (width 0.1))
@@
   (segment (start 98.12 145.1) (end 98.12 142.25) (width 0.4) (layer "B.Cu") (net 48))
   (segment (start 96.845 99.375) (end 96.845 100.01) (width 0.4) (layer "B.Cu") (net 48))
-  (segment (start 108.34 73.5) (end 124.84 57) (width 0.4) (layer "F.Cu") (net 49))
-  (segment (start 85.745 110.5) (end 100.66 110.5) (width 0.4) (layer "F.Cu") (net 49))
-  (segment (start 78.43 99.375) (end 78.43 103.185) (width 0.4) (layer "F.Cu") (net 49))
-  (segment (start 99.385 73.5) (end 108.34 73.5) (width 0.4) (layer "F.Cu") (net 49))
-  (segment (start 78.43 103.185) (end 85.745 110.5) (width 0.4) (layer "F.Cu") (net 49))
-  (via (at 100.66 110.5) (size 0.6) (drill 0.3) (layers "F.Cu" "B.Cu") (net 49))
-  (via (at 99.385 73.5) (size 0.6) (drill 0.3) (layers "F.Cu" "B.Cu") (net 49))
-  (segment (start 100.655 98.105) (end 99.385 99.375) (width 0.4) (layer "B.Cu") (net 49))
-  (segment (start 100.66 107.635) (end 99.385 106.36) (width 0.4) (layer "B.Cu") (net 49))
-  (segment (start 100.655 93.66) (end 99.385 92.39) (width 0.4) (layer "B.Cu") (net 49))
-  (segment (start 99.385 106.36) (end 99.385 104.455) (width 0.4) (layer "B.Cu") (net 49))
-  (segment (start 100.66 142.25) (end 100.66 145.1) (width 0.4) (layer "B.Cu") (net 49))
-  (segment (start 100.66 94.3) (end 100.655 94.295) (width 0.4) (layer "B.Cu") (net 49))
-  (segment (start 99.385 92.39) (end 99.385 73.5) (width 0.4) (layer "B.Cu") (net 49))
-  (segment (start 100.655 94.295) (end 100.655 93.66) (width 0.4) (layer "B.Cu") (net 49))
-  (segment (start 100.66 142.25) (end 100.66 107.635) (width 0.4) (layer "B.Cu") (net 49))
-  (segment (start 100.66 96.75) (end 100.66 98.1) (width 0.4) (layer "B.Cu") (net 49))
-  (segment (start 99.385 100.01) (end 99.385 104.455) (width 0.2) (layer "B.Cu") (net 49))
-  (segment (start 100.66 98.1) (end 100.655 98.105) (width 0.4) (layer "B.Cu") (net 49))
-  (segment (start 99.385 99.375) (end 99.385 100.01) (width 0.4) (layer "B.Cu") (net 49))
-  (segment (start 100.66 96.75) (end 100.66 94.3) (width 0.4) (layer "B.Cu") (net 49))
   (segment (start 93.04 142.25) (end 93.04 107.635) (width 0.4) (layer "B.Cu") (net 50))
   (segment (start 91.765 100.01) (end 91.765 104.455) (width 0.2) (layer "B.Cu") (net 50))
@@
   (segment (start 95.58 103.75) (end 95.58 100.9) (width 0.4) (layer "B.Cu") (net 70))
   (segment (start 96.845 98.105) (end 95.58 99.37) (width 0.4) (layer "B.Cu") (net 70))
+  (segment (start 85.745 110.5) (end 100.66 110.5) (width 0.4) (layer "F.Cu") (net 71))
+  (segment (start 78.43 99.375) (end 78.43 103.185) (width 0.4) (layer "F.Cu") (net 71))
+  (segment (start 78.43 103.185) (end 85.745 110.5) (width 0.4) (layer "F.Cu") (net 71))
+  (via (at 100.66 110.5) (size 0.6) (drill 0.3) (layers "F.Cu" "B.Cu") (net 71))
+  (segment (start 100.655 98.105) (end 99.385 99.375) (width 0.4) (layer "B.Cu") (net 71))
+  (segment (start 100.66 107.635) (end 99.385 106.36) (width 0.4) (layer "B.Cu") (net 71))
+  (segment (start 99.385 106.36) (end 99.385 104.455) (width 0.4) (layer "B.Cu") (net 71))
+  (segment (start 100.66 142.25) (end 100.66 145.1) (width 0.4) (layer "B.Cu") (net 71))
+  (segment (start 100.66 142.25) (end 100.66 107.635) (width 0.4) (layer "B.Cu") (net 71))
+  (segment (start 100.66 96.75) (end 100.66 98.1) (width 0.4) (layer "B.Cu") (net 71))
+  (segment (start 99.385 100.01) (end 99.385 104.455) (width 0.2) (layer "B.Cu") (net 71))
+  (segment (start 100.66 98.1) (end 100.655 98.105) (width 0.4) (layer "B.Cu") (net 71))
+  (segment (start 99.385 99.375) (end 99.385 100.01) (width 0.4) (layer "B.Cu") (net 71))
   (zone (net 3) (net_name "+3V3") (layer "F.Cu") (hatch edge 0.508)
     (connect_pads yes (clearance 0.35))

Commit message: Update
Other:
- board text added: "S"
Changed lines of the file:
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@@
     (fp_arc (start -0.3 4.4) (mid -0.923087 4.342349) (end -1.5 4.1) (layer "F.Fab") (width 0.1))
     (fp_arc (start 0.9 -5.2) (mid 4.903738 -1.844893) (end 4 3.3) (layer "F.Fab") (width 0.1))
-    (fp_arc (start 1.5 4.1) (mid 0.923087 4.34235) (end 0.3 4.4) (layer "F.Fab") (width 0.1))
+    (fp_arc (start 1.5 4.1) (mid 0.923087 4.342349) (end 0.3 4.4) (layer "F.Fab") (width 0.1))
     (fp_circle (center 0 0) (end 1.6 0) (layer "F.Fab") (width 0.1) (fill none))
     (fp_circle (center -2.5 5.3) (end -1.5 5.3) (layer "F.Fab") (width 0.1) (fill none))
@@
     (fp_line (start -1.5 5.3) (end 1.5 5.3) (layer "F.Fab") (width 0.1))
     (fp_arc (start -4 3.3) (mid -4.903738 -1.844892) (end -0.9 -5.2) (layer "F.Fab") (width 0.1))
-    (fp_arc (start 1.5 4.1) (mid 0.923087 4.34235) (end 0.3 4.4) (layer "F.Fab") (width 0.1))
+    (fp_arc (start 1.5 4.1) (mid 0.923087 4.342349) (end 0.3 4.4) (layer "F.Fab") (width 0.1))
     (fp_arc (start 0.9 -5.2) (mid 4.903738 -1.844893) (end 4 3.3) (layer "F.Fab") (width 0.1))
     (fp_arc (start -0.3 4.4) (mid -0.923087 4.342349) (end -1.5 4.1) (layer "F.Fab") (width 0.1))
@@
     (effects (font (size 1 1) (thickness 0.15)))
   )
-  (gr_text "+3V3" (at 128 97 270) (layer "F.SilkS")
-    (effects (font (size 1 1) (thickness 0.15)) (justify left))
+  (gr_text "+3V3" (at 128 97 90) (layer "F.SilkS")
+    (effects (font (size 1 1) (thickness 0.15)) (justify right))
   )
   (gr_text "BCKL" (at 70.5 79.5) (layer "F.SilkS")
@@
     (effects (font (size 1 1) (thickness 0.15)) (justify right))
   )
-  (gr_text "S3" (at 133 114) (layer "F.SilkS")
+  (gr_text "S" (at 133 114) (layer "F.SilkS")
     (effects (font (size 1 1) (thickness 0.15)) (justify left))
   )
