File: Kicad/mini/pic16bit.kicad_pcb (KiCad board)
At the start: 2 copper layers, 80 x 100 mm, 89 parts, among them IC201 TLV1117-33, IC202 MICROCHIP-PIC24FJ64GA102-ISP, IC301 CAT4002A, IC302 MCP2221A, K101 PE-450-4X6X-BLACK, K201 *Power & UART, K202 MCU 1, K203 MCU 1, K204 ICSP, K205 MCU 2, K206 MCU 2, K301 HARWIN-254-F-1X08-VERTICAL, K302 HARWIN-254-F-1X06-VERTICAL, P301 PIHER-PT10MV-10K, P302 PIHER-PT10MV-10K

Commit message: Update
Parts:
- added kibuzzard-627E464E: G***, kibuzzard-627E464E, F.Cu at (94.5, 52.5)
- added kibuzzard-627E46F0: G***, kibuzzard-627E46F0, F.Cu at (97.0, 53.6)
- added kibuzzard-627E4750: G***, kibuzzard-627E4750, F.Cu at (72.8, 90.5)
- added kibuzzard-627E4750: G***, kibuzzard-627E4750, F.Cu at (79.5, 129.5)
- added kibuzzard-627E4750: G***, kibuzzard-627E4750, F.Cu at (134.8, 118.2)
- added kibuzzard-627E477E: G***, kibuzzard-627E477E, F.Cu at (79.5, 123.0)
- added kibuzzard-627E47DC: G***, kibuzzard-627E47DC, F.Cu at (77.5, 143.5)
- added kibuzzard-627E47F4: G***, kibuzzard-627E47F4, F.Cu at (136.5, 143.5)
- added kibuzzard-627E94B6: G***, kibuzzard-627E94B6, F.Cu at (128.0, 99.5)
- JP301: value EN BCKL -> BCKL
- K203, K206: footprint tronixio:zzHARWIN-M20-782144x -> tronixio:HARWIN-M20-782144x
Connections:
- IC202 pad 5: /HID/PGC/URX/RB1 -> PGC/URX/RB1
- JP303 pad 2: /HID/PGC/URX/RB1 -> PGC/URX/RB1
- K202 pad 5: /HID/PGC/URX/RB1 -> PGC/URX/RB1
- K203 pad 5: /HID/PGC/URX/RB1 -> PGC/URX/RB1
- K204 pad 2: PGC/UTX/RB1 -> PGC/URX/RB1
Routing:
- net PGC/URX/RB1: track 0.00 -> 134.3 mm, vias 0 -> 2
- net /HID/PGC/URX/RB1: track 78.5 -> 0.00 mm, vias 1 -> 0
Other:
- board text removed: "+3V3"
- board text removed: "+5V IN"

Commit message: Update pic16bit.kicad_pcb
Routing:
- net +3V3: vias 22 -> 20
Changed lines of the file:
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@@
     (fp_arc (start -0.3 4.4) (mid -0.923087 4.342349) (end -1.5 4.1) (layer "F.Fab") (width 0.1))
     (fp_arc (start 0.9 -5.2) (mid 4.903738 -1.844893) (end 4 3.3) (layer "F.Fab") (width 0.1))
-    (fp_arc (start 1.5 4.1) (mid 0.923087 4.342349) (end 0.3 4.4) (layer "F.Fab") (width 0.1))
+    (fp_arc (start 1.5 4.1) (mid 0.923087 4.34235) (end 0.3 4.4) (layer "F.Fab") (width 0.1))
     (fp_circle (center 0 0) (end 1.6 0) (layer "F.Fab") (width 0.1) (fill none))
     (fp_circle (center -2.5 5.3) (end -1.5 5.3) (layer "F.Fab") (width 0.1) (fill none))
@@
     (fp_line (start -1.5 5.3) (end 1.5 5.3) (layer "F.Fab") (width 0.1))
     (fp_arc (start -4 3.3) (mid -4.903738 -1.844892) (end -0.9 -5.2) (layer "F.Fab") (width 0.1))
-    (fp_arc (start 1.5 4.1) (mid 0.923087 4.342349) (end 0.3 4.4) (layer "F.Fab") (width 0.1))
+    (fp_arc (start 1.5 4.1) (mid 0.923087 4.34235) (end 0.3 4.4) (layer "F.Fab") (width 0.1))
     (fp_arc (start 0.9 -5.2) (mid 4.903738 -1.844893) (end 4 3.3) (layer "F.Fab") (width 0.1))
     (fp_arc (start -0.3 4.4) (mid -0.923087 4.342349) (end -1.5 4.1) (layer "F.Fab") (width 0.1))
@@
   (via (at 104.5 52) (size 0.6) (drill 0.3) (layers "F.Cu" "B.Cu") (net 3))
   (via (at 73 124) (size 0.6) (drill 0.3) (layers "F.Cu" "B.Cu") (net 3))
-  (via (at 111 57) (size 1) (drill 0.5) (layers "F.Cu" "B.Cu") (free) (net 3))
-  (via (at 113 49) (size 1) (drill 0.5) (layers "F.Cu" "B.Cu") (free) (net 3))
+  (via (at 113 49.25) (size 1) (drill 0.5) (layers "F.Cu" "B.Cu") (free) (net 3))
   (via (at 90.5 76.5) (size 0.6) (drill 0.3) (layers "F.Cu" "B.Cu") (net 3))
-  (via (at 115 57) (size 1) (drill 0.5) (layers "F.Cu" "B.Cu") (free) (net 3))
+  (via (at 115 56.75) (size 1) (drill 0.5) (layers "F.Cu" "B.Cu") (free) (net 3))
   (via (at 84.5 103.75) (size 0.6) (drill 0.3) (layers "F.Cu" "B.Cu") (net 3))
-  (via (at 115 49) (size 1) (drill 0.5) (layers "F.Cu" "B.Cu") (free) (net 3))
-  (via (at 113 57) (size 1) (drill 0.5) (layers "F.Cu" "B.Cu") (free) (net 3))
-  (via (at 119 49) (size 1) (drill 0.5) (layers "F.Cu" "B.Cu") (free) (net 3))
+  (via (at 115 49.25) (size 1) (drill 0.5) (layers "F.Cu" "B.Cu") (free) (net 3))
+  (via (at 113 56.75) (size 1) (drill 0.5) (layers "F.Cu" "B.Cu") (free) (net 3))
+  (via (at 119 49.25) (size 1) (drill 0.5) (layers "F.Cu" "B.Cu") (free) (net 3))
   (via (at 120.98 107.5) (size 0.6) (drill 0.3) (layers "F.Cu" "B.Cu") (net 3))
   (via (at 73 136) (size 0.6) (drill 0.3) (layers "F.Cu" "B.Cu") (net 3))
   (via (at 87.5 76.5) (size 0.6) (drill 0.3) (layers "F.Cu" "B.Cu") (net 3))
   (via (at 119 53) (size 1) (drill 0.5) (layers "F.Cu" "B.Cu") (free) (net 3))
-  (via (at 117 49) (size 1) (drill 0.5) (layers "F.Cu" "B.Cu") (free) (net 3))
+  (via (at 117 49.25) (size 1) (drill 0.5) (layers "F.Cu" "B.Cu") (free) (net 3))
   (via (at 137.25 134) (size 0.6) (drill 0.3) (layers "F.Cu" "B.Cu") (net 3))
   (via (at 113 76.5) (size 0.6) (drill 0.3) (layers "F.Cu" "B.Cu") (net 3))
   (via (at 119 55) (size 1) (drill 0.5) (layers "F.Cu" "B.Cu") (free) (net 3))
-  (via (at 111 49) (size 1) (drill 0.5) (layers "F.Cu" "B.Cu") (free) (net 3))
-  (via (at 119 57) (size 1) (drill 0.5) (layers "F.Cu" "B.Cu") (free) (net 3))
-  (via (at 117 57) (size 1) (drill 0.5) (layers "F.Cu" "B.Cu") (free) (net 3))
+  (via (at 119 56.75) (size 1) (drill 0.5) (layers "F.Cu" "B.Cu") (free) (net 3))
+  (via (at 117 56.75) (size 1) (drill 0.5) (layers "F.Cu" "B.Cu") (free) (net 3))
   (segment (start 87.5 76.5) (end 84.5 73.5) (width 0.5) (layer "B.Cu") (net 3))
   (segment (start 84.5 119.82) (end 84.5 105.25) (width 0.5) (layer "B.Cu") (net 3))

Commit message: Update
Parts:
- removed IC201: TLV1117-33, tronixio:SOT-223-3
- removed IC202: MICROCHIP-PIC24FJ64GA102-ISP, tronixio:DIP-28-W762-SOCKET
- removed IC301: CAT4002A, tronixio:SOT-23-6
- removed IC302: MCP2221A, tronixio:SOIC-SL-14
- added U201: TLV1117-33, tronixio:SOT-223-3, F.Cu at (110.0, 53.0)
- added U202: MICROCHIP-PIC24FJ64GA102-ISP, tronixio:DIP-28-W762, F.Cu at (90.5, 96.8)
- added U301: CAT4002A, tronixio:SOT-23-6, B.Cu at (75.0, 65.7)
- added U302: MCP2221A, tronixio:SOIC-SL-14, B.Cu at (84.5, 58.0)
- K302: footprint tronixio:zzHARWIN-M20-782064x -> tronixio:HARWIN-M20-782064x

Commit message: Update
Parts:
- F201: value F050 -> 500mA
- JP201: value *Power IN -> Power IN
- JP205: value VCAP -> VCA
- P301, P302: value PIHER-PT10MV-10K -> 10K
- R315: value 10K -> 1K
- S303: value BOURNS-PEC12R-24DENTS -> BOURNS-PEC12R-24DENTS-SWITCH; footprint tronixio:BOURNS-PEC12R -> tronixio:BOURNS-PEC12R-SWITCH
- U202: value MICROCHIP-PIC24FJ64GA102-ISP -> PIC24/dsPIC32; footprint tronixio:DIP-28-W762 -> tronixio:DIP-28-W762-SOCKET
- U302: value MCP2221A -> MCP2221A-ISL; footprint tronixio:SOIC-SL-14 -> tronixio:SOIC-14

Commit message: Update
Parts:
- C201, C202, C203, C204, C205, C301, C302, C303, C304, C305, C306, C307: footprint tronixio:CAPACITOR-1206 -> tronixio:CAPACITOR-SMD-1206
- F201: footprint tronixio:FUSE-1206 -> tronixio:FUSE-SMD-1206
- LED201, LED301, LED302: footprint tronixio:LED-1206 -> tronixio:LED-SMD-1206
- R201, R202, R203, R204, R205, R301, R302, R303, R304, R305, R306, R307, R308, R309, R310, R311, R312, R313, R314, R315, R316, R317, R318, R319, R320: footprint tronixio:RESISTOR-1206 -> tronixio:RESISTOR-SMD-1206
- U202: footprint tronixio:DIP-28-W762-SOCKET -> tronixio:DIP-28-W762

Commit message: Update
Parts:
- JP205: value VCA -> VCAP
- U301: footprint tronixio:SOT-23-6 -> tronixioZZZ:SC-70-6
- U302: value MCP2221A-ISL -> MCP2221A
- moved U301 0.30 mm to (75.0, 65.4)
Routing:
- net GND: track 112.8 -> 117.6 mm
- net +5V: track 63.8 -> 64.5 mm
