File: Kicad/mini/pic16bit.kicad_pcb (KiCad board)
At the start: 2 copper layers, 80 x 100 mm, 100 parts, among them K101 PE-450-4X6X-BLACK, K201 *Power & UART, K202 MCU 1, K203 MCU 1, K204 ICSP, K205 MCU 2, K206 MCU 2, K301 HARWIN-254-F-1X08-VERTICAL, K302 HARWIN-254-F-1X06-VERTICAL, P301 10K, P302 10K, U201 TLV1117-33, U202 PIC24/dsPIC32, U301 CAT4002A, U302 MCP2221A

Commit message: Up
Parts:
- C206: footprint tronixio:KEMET-C322 -> tronixio:CAPACITOR-SMD-1206
- H101, H102, H103, H104: value KEYSTONE-9055 -> 9055
- K201: footprint tronixio:FCI-USB-TYPE-B-MICRO-THT -> tronixio:USB-TYPE-B-MICRO-TH
- TP201, TP202: value KEYSTONE-5006 -> 5006
- TP203: value KEYSTONE-2000-3 -> 2000-3
- U202: footprint tronixio:DIP-28-W762 -> tronixio:DIP-28-W762-SOCKET
- moved C206 0.24 mm to (135.5, 93.0)
- moved JP205 0.23 mm to (131.8, 94.3)
- turned S303 to 180 degrees
Connections:
- S303 pad 4: GND -> Net-(R309-Pad2)
- S303 pad 5: Net-(R309-Pad2) -> GND
Routing:
- net GND: track 117.6 -> 116.3 mm, vias 4 -> 5
- net Net-(K205-Pin_9): track 39.3 -> 40.2 mm
- net Net-(C206-Pad1): track 4.34 -> 3.83 mm

Commit message: Up
Parts:
- C206: moved to B.Cu
- moved JP205 0.23 mm to (132.0, 94.3)
Routing:
- net GND: track 116.3 -> 114.8 mm, vias 5 -> 4
Changed lines of the file:
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@@
     )
   )
-  (footprint "tronixio:CAPACITOR-SMD-1206" (layer "F.Cu")
-    (at 135.5 93 -90)
-    (property "Mouser" "791-1206X106J250CT")
-    (property "Sheetfile" "pic16bit-mcu.kicad_sch")
-    (property "Sheetname" "MCU")
-    (property "Tolerance" "5%")
-    (property "Voltage" "25V")
-    (property "ki_description" "Unpolarized Capacitor")
-    (attr smd)
-    (fp_text reference "C206" (at 0 2 -90) (layer "F.SilkS") hide
-        (effects (font (size 1 1) (thickness 0.15)))
-    )
-    (fp_text value "10µ" (at 0 2 -90) (layer "F.Fab")
-        (effects (font (size 1 1) (thickness 0.15)))
-    )
-    (fp_line (start -0.6 -0.9) (end 0.6 -0.9)
-      (stroke (width 0.15) (type solid)) (layer "F.SilkS"))
-    (fp_line (start -0.6 0.9) (end 0.6 0.9)
-      (stroke (width 0.15) (type solid)) (layer "F.SilkS"))
-    (fp_rect (start -2.3 1) (end 2.3 -1)
-      (stroke (width 0.05) (type solid)) (fill none) (layer "F.CrtYd"))
-    (pad "1" smd roundrect (at -1.5 0 270) (size 1.3 1.75) (layers "F.Cu" "F.Paste" "F.Mask") (roundrect_rratio 0.1)
-      (net 36 "Net-(C206-Pad1)") (pintype "passive"))
-    (pad "2" smd roundrect (at 1.5 0 270) (size 1.3 1.75) (layers "F.Cu" "F.Paste" "F.Mask") (roundrect_rratio 0.1)
-      (net 2 "GND") (pintype "passive"))
-    (model "${KICAD_USER_3DMODEL_DIR}/SMD/CAPACITOR-1206.wrl"
-      (offset (xyz 0 0 0))
-      (scale (xyz 1 1 1))
-      (rotate (xyz 0 0 0))
-    )
-  )
   (footprint "kibuzzard-627E477E" (layer "F.Cu")
     (at 79.5 123 -90)
@@
   )
   (footprint "tronixio:HARWIN-M20-999024x" (layer "F.Cu")
-    (at 131.77 94.27 180)
+    (at 132 94.27 180)
     (property "Mouser" "855-M20-999024")
     (property "Sheetfile" "pic16bit-mcu.kicad_sch")
@@
   )
   (footprint "tronixio:CAPACITOR-SMD-1206" (layer "B.Cu")
+    (at 135.5 93 -90)
+    (property "Mouser" "791-1206X106J250CT")
+    (property "Sheetfile" "pic16bit-mcu.kicad_sch")
+    (property "Sheetname" "MCU")
+    (property "Tolerance" "5%")
+    (property "Voltage" "25V")
+    (property "ki_description" "Unpolarized Capacitor")
+    (attr smd)
+    (fp_text reference "C206" (at 0 -2 90) (layer "B.SilkS") hide
+        (effects (font (size 1 1) (thickness 0.15)) (justify mirror))
+    )
+    (fp_text value "10µ" (at 0 -2 90) (layer "B.Fab")
+        (effects (font (size 1 1) (thickness 0.15)) (justify mirror))
+    )
+    (fp_line (start -0.6 -0.9) (end 0.6 -0.9)
+      (stroke (width 0.15) (type solid)) (layer "B.SilkS"))
+    (fp_line (start -0.6 0.9) (end 0.6 0.9)
+      (stroke (width 0.15) (type solid)) (layer "B.SilkS"))
+    (fp_rect (start -2.3 -1) (end 2.3 1)
+      (stroke (width 0.05) (type solid)) (fill none) (layer "B.CrtYd"))
+    (pad "1" smd roundrect (at -1.5 0 270) (size 1.3 1.75) (layers "B.Cu" "B.Paste" "B.Mask") (roundrect_rratio 0.1)
+      (net 36 "Net-(C206-Pad1)") (pintype "passive"))
+    (pad "2" smd roundrect (at 1.5 0 270) (size 1.3 1.75) (layers "B.Cu" "B.Paste" "B.Mask") (roundrect_rratio 0.1)
+      (net 2 "GND") (pintype "passive"))
+    (model "${KICAD_USER_3DMODEL_DIR}/SMD/CAPACITOR-1206.wrl"
+      (offset (xyz 0 0 0))
+      (scale (xyz 1 1 1))
+      (rotate (xyz 0 0 0))
+    )
+  )
+  (footprint "tronixio:CAPACITOR-SMD-1206" (layer "B.Cu")
     (at 90.5 58 -90)
     (property "Mouser" "80-C1206C104J5R")
@@
   (gr_line (start 70 132) (end 70 140)
     (stroke (width 0.2) (type solid)) (layer "F.SilkS"))
-  (gr_line (start 138 88.5) (end 130.5 88.5)
+  (gr_line (start 133.5 90) (end 130.5 90)
     (stroke (width 0.2) (type solid)) (layer "F.SilkS"))
   (gr_line (start 70 120) (end 70 128)
@@
   (gr_rect (start 105.5 48.5) (end 120 57.5)
     (stroke (width 0.1) (type solid)) (fill solid) (layer "B.Mask"))
-  (gr_rect (start 109 48.5) (end 120 57.5)
+  (gr_rect (start 108.5 48.5) (end 120 57.5)
     (stroke (width 0.1) (type solid)) (fill solid) (layer "F.Mask"))
   (gr_line (start 57 47) (end 56.5 47)
@@
     (effects (font (size 1 1) (thickness 0.15)) (justify left))
   )
-  (gr_text "VCAP" (at 138 87.5) (layer "F.SilkS")
-    (effects (font (size 1 1) (thickness 0.15)) (justify right))
+  (gr_text "VCAP" (at 132 89) (layer "F.SilkS")
+    (effects (font (size 1 1) (thickness 0.15)))
   )
   (gr_text "PIC16-Bit Mini Trainer - Rev.A - (01/2022) - SCALE 100%" (at 67 162) (layer "Dwgs.User")
@@
   (segment (start 69.4 96.005) (end 69.4 98.105) (width 0.5) (layer "F.Cu") (net 2))
   (segment (start 69.4 100.205) (end 69.4 98.105) (width 0.5) (layer "F.Cu") (net 2))
-  (segment (start 135.5 94.5) (end 135.5 96) (width 0.5) (layer "F.Cu") (net 2))
   (segment (start 83.2 50) (end 82.3 49.1) (width 0.4) (layer "F.Cu") (net 2))
   (via (at 104.5 50.25) (size 0.6) (drill 0.3) (layers "F.Cu" "B.Cu") (net 2))
   (via (at 108.28 116.66) (size 0.6) (drill 0.3) (layers "F.Cu" "B.Cu") (net 2))
   (via (at 69.4 98.105) (size 0.6) (drill 0.3) (layers "F.Cu" "B.Cu") (net 2))
-  (via (at 135.5 96) (size 0.6) (drill 0.3) (layers "F.Cu" "B.Cu") (net 2))
   (via (at 101.5 54) (size 0.6) (drill 0.3) (layers "F.Cu" "B.Cu") (net 2))
   (segment (start 107.005 104.995) (end 107 105) (width 0.2) (layer "B.Cu") (net 2))
@@
   (via (at 81.96 59) (size 0.6) (drill 0.3) (layers "F.Cu" "B.Cu") (net 31))
   (segment (start 81.96 60.8) (end 81.96 59) (width 0.4) (layer "B.Cu") (net 31))
-  (segment (start 131.77 95.73) (end 131.77 94.27) (width 0.5) (layer "F.Cu") (net 32))
+  (segment (start 112.72 99) (end 129 99) (width 0.5) (layer "F.Cu") (net 32))
+  (segment (start 132 96) (end 132 94.27) (width 0.5) (layer "F.Cu") (net 32))
+  (segment (start 129 99) (end 132 96) (width 0.5) (layer "F.Cu") (net 32))
   (segment (start 110.82 100.9) (end 112.72 99) (width 0.5) (layer "F.Cu") (net 32))
-  (segment (start 112.72 99) (end 128.5 99) (width 0.5) (layer "F.Cu") (net 32))
-  (segment (start 128.5 99) (end 131.77 95.73) (width 0.5) (layer "F.Cu") (net 32))
   (segment (start 110.82 100.9) (end 110.82 103.75) (width 0.5) (layer "B.Cu") (net 32))
   (segment (start 112.085 98.105) (end 110.82 99.37) (width 0.4) (layer "B.Cu") (net 32))
@@
   (segment (start 75.89 96.835) (end 78.5 94.225) (width 0.5) (layer "B.Cu") (net 35))
   (segment (start 85.77 56.77) (end 85.77 55.2) (width 0.5) (layer "B.Cu") (net 35))
-  (segment (start 131.77 91.73) (end 133.77 91.73) (width 0.5) (layer "F.Cu") (net 36))
-  (segment (start 135.5 91.5) (end 134 91.5) (width 0.5) (layer "F.Cu") (net 36))
-  (segment (start 133.77 91.73) (end 134 91.5) (width 0.5) (layer "F.Cu") (net 36))
+  (segment (start 132 91.73) (end 133.77 91.73) (width 0.5) (layer "B.Cu") (net 36))
+  (segment (start 133.77 91.73) (end 134 91.5) (width 0.5) (layer "B.Cu") (net 36))
+  (segment (start 134 91.5) (end 135.5 91.5) (width 0.5) (layer "B.Cu") (net 36))
   (segment (start 84.84 111.5) (end 98.12 111.5) (width 0.5) (layer "F.Cu") (net 37))
   (segment (start 75.89 102.55) (end 84.84 111.5) (width 0.5) (layer "F.Cu") (net 37))
@@
       (pts
         (xy 120 57.5)
-        (xy 109 57.5)
-        (xy 109 48.5)
+        (xy 108.5 57.5)
+        (xy 108.5 48.5)
         (xy 120 48.5)
       )

Commit message: Up
Parts:
- H101, H102, H103, H104: value 9055 -> KEYSTONE-9055
- TP201, TP202: value 5006 -> KEYSTONE-5006
- TP203: value 2000-3 -> KEYSTONE-2000-3
Changed lines of the file:
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@@
         (effects (font (size 1 1) (thickness 0.15)))
     )
-    (fp_text value "5006" (at 0 2.5 90) (layer "F.Fab")
+    (fp_text value "KEYSTONE-5006" (at 0 2.5 90) (layer "F.Fab")
         (effects (font (size 1 1) (thickness 0.15)))
     )
@@
         (effects (font (size 1 1) (thickness 0.15)))
     )
-    (fp_text value "9055" (at 0 3.5) (layer "F.Fab") hide
+    (fp_text value "KEYSTONE-9055" (at 0 3.5) (layer "F.Fab") hide
         (effects (font (size 1 1) (thickness 0.15)))
     )
@@
         (effects (font (size 1 1) (thickness 0.15)))
     )
-    (fp_text value "2000-3" (at 0 2) (layer "F.Fab")
+    (fp_text value "KEYSTONE-2000-3" (at 0 2) (layer "F.Fab")
         (effects (font (size 1 1) (thickness 0.15)))
     )
@@
         (effects (font (size 1 1) (thickness 0.15)))
     )
-    (fp_text value "5006" (at 0 2.5 90) (layer "F.Fab")
+    (fp_text value "KEYSTONE-5006" (at 0 2.5 90) (layer "F.Fab")
         (effects (font (size 1 1) (thickness 0.15)))
     )
@@
         (effects (font (size 1 1) (thickness 0.15)))
     )
-    (fp_text value "9055" (at 0 3.5) (layer "F.Fab") hide
+    (fp_text value "KEYSTONE-9055" (at 0 3.5) (layer "F.Fab") hide
         (effects (font (size 1 1) (thickness 0.15)))
     )
@@
         (effects (font (size 1 1) (thickness 0.15)))
     )
-    (fp_text value "9055" (at 0 3.5) (layer "F.Fab") hide
+    (fp_text value "KEYSTONE-9055" (at 0 3.5) (layer "F.Fab") hide
         (effects (font (size 1 1) (thickness 0.15)))
     )
@@
         (effects (font (size 1 1) (thickness 0.15)))
     )
-    (fp_text value "9055" (at 0 3.5) (layer "F.Fab") hide
+    (fp_text value "KEYSTONE-9055" (at 0 3.5) (layer "F.Fab") hide
         (effects (font (size 1 1) (thickness 0.15)))
     )
@@
   )
   (zone (net 2) (net_name "GND") (layer "B.Cu") (name "GND") (hatch none 0.5)
-    (connect_pads (clearance 0.5))
+    (connect_pads yes (clearance 0.5))
     (min_thickness 0.3) (filled_areas_thickness no)
     (fill yes (thermal_gap 0.5) (thermal_bridge_width 0.5))

Commit message: Up
Parts:
- H101, H102, H103, H104: value KEYSTONE-9055 -> 9055
- TP201, TP202: value KEYSTONE-5006 -> 5006
- TP203: value KEYSTONE-2000-3 -> 2000-3
Changed lines of the file:
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@@
     )
     (pad_to_mask_clearance 0)
-    (grid_origin 67 147)
+    (aux_axis_origin 67 147)
     (pcbplotparams
       (layerselection 0x00011fc_ffffffff)
@@
     (fp_arc (start 0.9 -5.2) (mid 4.903738 -1.844893) (end 4 3.3)
       (stroke (width 0.1) (type solid)) (layer "F.Fab"))
-    (fp_arc (start 1.5 4.1) (mid 0.923087 4.34235) (end 0.3 4.4)
+    (fp_arc (start 1.5 4.1) (mid 0.923087 4.342349) (end 0.3 4.4)
       (stroke (width 0.1) (type solid)) (layer "F.Fab"))
     (fp_circle (center -2.5 5.3) (end -1.5 5.3)
@@
         (effects (font (size 1 1) (thickness 0.15)))
     )
-    (fp_text value "KEYSTONE-5006" (at 0 2.5 90) (layer "F.Fab")
+    (fp_text value "5006" (at 0 2.5 90) (layer "F.Fab")
         (effects (font (size 1 1) (thickness 0.15)))
     )
@@
         (effects (font (size 1 1) (thickness 0.15)))
     )
-    (fp_text value "KEYSTONE-9055" (at 0 3.5) (layer "F.Fab") hide
+    (fp_text value "9055" (at 0 3.5) (layer "F.Fab") hide
         (effects (font (size 1 1) (thickness 0.15)))
     )
@@
         (effects (font (size 1 1) (thickness 0.15)))
     )
-    (fp_text value "KEYSTONE-2000-3" (at 0 2) (layer "F.Fab")
+    (fp_text value "2000-3" (at 0 2) (layer "F.Fab")
         (effects (font (size 1 1) (thickness 0.15)))
     )
@@
         (effects (font (size 1 1) (thickness 0.15)))
     )
-    (fp_text value "KEYSTONE-5006" (at 0 2.5 90) (layer "F.Fab")
+    (fp_text value "5006" (at 0 2.5 90) (layer "F.Fab")
         (effects (font (size 1 1) (thickness 0.15)))
     )
@@
         (effects (font (size 1 1) (thickness 0.15)))
     )
-    (fp_text value "KEYSTONE-9055" (at 0 3.5) (layer "F.Fab") hide
+    (fp_text value "9055" (at 0 3.5) (layer "F.Fab") hide
         (effects (font (size 1 1) (thickness 0.15)))
     )
@@
     (fp_arc (start 0.9 -5.2) (mid 4.903738 -1.844893) (end 4 3.3)
       (stroke (width 0.1) (type solid)) (layer "F.Fab"))
-    (fp_arc (start 1.5 4.1) (mid 0.923087 4.34235) (end 0.3 4.4)
+    (fp_arc (start 1.5 4.1) (mid 0.923087 4.342349) (end 0.3 4.4)
       (stroke (width 0.1) (type solid)) (layer "F.Fab"))
     (fp_circle (center -2.5 5.3) (end -1.5 5.3)
@@
         (effects (font (size 1 1) (thickness 0.15)))
     )
-    (fp_text value "KEYSTONE-9055" (at 0 3.5) (layer "F.Fab") hide
+    (fp_text value "9055" (at 0 3.5) (layer "F.Fab") hide
         (effects (font (size 1 1) (thickness 0.15)))
     )
@@
         (effects (font (size 1 1) (thickness 0.15)))
     )
-    (fp_text value "KEYSTONE-9055" (at 0 3.5) (layer "F.Fab") hide
+    (fp_text value "9055" (at 0 3.5) (layer "F.Fab") hide
         (effects (font (size 1 1) (thickness 0.15)))
     )
@@
   )
   (dimension (type aligned) (layer "Dwgs.User")
+    (pts (xy 67 147) (xy 67 144))
+    (height -2)
+    (gr_text "3.00 mm" (at 63 145.5 90) (layer "Dwgs.User")
+      (effects (font (size 1 1) (thickness 0.15)))
+    )
+    (format (prefix "") (suffix "") (units 2) (units_format 1) (precision 2))
+    (style (thickness 0.1) (arrow_length 1) (text_position_mode 2) (extension_height 0.58642) (extension_offset 0.5) keep_text_aligned)
+  )
+  (dimension (type aligned) (layer "Dwgs.User")
+    (pts (xy 67 147) (xy 70 147))
+    (height 2)
+    (gr_text "3.00 mm" (at 68.5 151) (layer "Dwgs.User")
+      (effects (font (size 1 1) (thickness 0.15)))
+    )
+    (format (prefix "") (suffix "") (units 2) (units_format 1) (precision 2))
+    (style (thickness 0.1) (arrow_length 1) (text_position_mode 2) (extension_height 0.58642) (extension_offset 0.5) keep_text_aligned)
+  )
+  (dimension (type aligned) (layer "Dwgs.User")

Commit message: Update
Parts:
- U202: footprint tronixio:DIP-28-W762-SOCKET -> tronixio:DIP-28-W762

Commit message: Update Mini Kicad 8
Parts:
- removed kibuzzard-627E464E (x2): G***, kibuzzard-627E464E
- removed kibuzzard-627E46F0: G***, kibuzzard-627E46F0
- removed kibuzzard-627E4750 (x3): G***, kibuzzard-627E4750
- removed kibuzzard-627E477E: G***, kibuzzard-627E477E
- removed kibuzzard-627E47DC: G***, kibuzzard-627E47DC
- removed kibuzzard-627E47F4: G***, kibuzzard-627E47F4
- removed kibuzzard-627E94B6: G***, kibuzzard-627E94B6
- removed kibuzzard-640F1A35: G***, kibuzzard-640F1A35
- added kibuzzard-65F5FF8A: G***, kibuzzard-65F5FF8A, B.Cu at (94.5, 52.5)
- added kibuzzard-65F5FF96: G***, kibuzzard-65F5FF96, B.Cu at (97.0, 52.5)
- added kibuzzard-65F5FFA5: G***, kibuzzard-65F5FFA5, F.Cu at (94.5, 52.5)
- added kibuzzard-65F5FFB1: G***, kibuzzard-65F5FFB1, F.Cu at (97.0, 53.6)
- added kibuzzard-65F5FFC7: G***, kibuzzard-65F5FFC7, F.Cu at (128.0, 99.5)
- added kibuzzard-65F5FFD5: G***, kibuzzard-65F5FFD5, F.Cu at (79.5, 123.0)
- added kibuzzard-65F5FFE7: G***, kibuzzard-65F5FFE7, F.Cu at (79.5, 129.5)
- added kibuzzard-65F5FFF2: G***, kibuzzard-65F5FFF2, F.Cu at (134.8, 118.2)
- added kibuzzard-65F60000: G***, kibuzzard-65F60000, F.Cu at (77.5, 143.5)
- added kibuzzard-65F6000E: G***, kibuzzard-65F6000E, F.Cu at (136.5, 143.5)
- added kibuzzard-65F60022: G***, kibuzzard-65F60022, F.Cu at (72.8, 90.5)
- H101, H102, H103, H104: value 9055 -> KEYSTONE-9055
- TP201, TP202: value 5006 -> KEYSTONE-5006
- TP203: value 2000-3 -> KEYSTONE-2000-3
- U201: footprint tronixio:SOT-223-3 -> tronixio:SOT-223-3-TABPIN2
Connections:
- net +3V3 renamed POWER-+3V3
- net +5V renamed POWER-+5V
- net GND renamed POWER-GND

Commit message: Update Mini
Routing:
- net Net-(U301-EN): track 26.7 -> 28.6 mm

Commit message: Up
Parts:
- U202: value PIC24/dsPIC32 -> PIC24/dsPIC33
- moved H101 94.0 mm to (70.0, 50.0)
- moved H103 94.0 mm to (144.0, 144.0)
- moved H102 74.0 mm to (70.0, 144.0)
- moved H104 74.0 mm to (144.0, 50.0)
