File: Kicad/mini/pic16bit-hid.kicad_sch (KiCad schematic)
At the start: 43 parts, among them IC301 CAT4002A, IC302 MCP2221A, K301 HARWIN-254-F-1X08-VERTICAL, K302 HARWIN-254-F-1X06-VERTICAL, P301 PIHER-PT10MV-10K, P302 PIHER-PT10MV-10K

Commit message: Update Mini
Parts:
- removed IC301: CAT4002A, tronixio:SOT-23-6, symbol tronixio:CAT4002A
- removed IC302: MCP2221A, tronixio:SOIC-SL-14, symbol tronixio:MCP2221A-ISL
- added IC301: ONSEMI-CAT4002A-SOT-23, tronixio:SOT-23-6, symbol tronixio:ONSEMI-CAT4002A-SOT-23
- added IC302: MICROCHIP-MCP2221A-ISL, tronixio:SOIC-SL-14, symbol tronixio:MICROCHIP-MCP2221A-ISL
- BB301: MOUSER 854-BB170 -> (none); Mouser (none) -> 854-BB170
- C301, C302, C304, C305, C306, C307: footprint tronixio:CAPACITOR-1206 -> (none)
- C303: value 1µ -> (none); footprint tronixio:CAPACITOR-1206 -> (none)
- JP301, JP302, JP303: MOUSER 855-M20-999024 -> (none); Mouser (none) -> 855-M20-999024
- K301: footprint tronixio:zzHARWIN-M20-782084x -> tronixio:HARWIN-M20-782084x; MOUSER 855-M20-999084 -> (none); Mouser (none) -> 855-M20-999084
- K302: value HARWIN-254-F-1X06-VERTICAL -> (none); footprint tronixio:zzHARWIN-M20-782064x -> (none); MOUSER 855-M20-782064 -> (none); Mouser (none) -> 855-M20-782064
- LCD301: MOUSER 763-C0220BIZ-FSW-FBW -> (none); Mouser (none) -> 763-C0220BIZ-FSW-FBW
- LED301, LED302: footprint tronixio:LED-1206 -> (none); MOUSER 604-APT2012LSECKJ4RV -> (none); Mouser (none) -> 604-APT2012LSECKJ4RV
- P301, P302: MOUSER 531-PT10MV-10K -> (none); Mouser (none) -> 531-PT10MV-10K; NAME 10K -> (none); Name (none) -> 10K
- R301, R302, R303, R304, R305, R306, R307, R308, R309, R310, R311, R312, R313, R314, R315, R316, R317, R318, R319, R320: footprint tronixio:RESISTOR-1206 -> (none)
- S301: value S1 -> (none); MOUSER 611-KSA0M911LFT -> (none); Mouser (none) -> 611-KSA0M911LFT
- S302: value S2 -> (none); MOUSER 611-KSA0M911LFT -> (none); Mouser (none) -> 611-KSA0M911LFT
- S303: MOUSER 652-PEC12R-4215F-S24 -> (none); Mouser (none) -> 652-PEC12R-4215F-S24
Connections:
- net +3V3: now also IC302.1 (VDD), IC302.11 (VUSB)
- net +5V: now also IC301.3 (VIN)
- net BCKL: now also IC301.6 (LED1)
- net D+: now also IC302.13 (D+)
- net D-: now also IC302.12 (D-)
- net GND: now also IC301.2 (GND), IC302.14 (VSS)
- net SCL: now also IC302.10 (SCL)
- net SDA: now also IC302.9 (SDA)
- net at JP303.1, R317.2: now also IC302.6 (UTx)
- net at LED302.1 (K): now also IC302.2 (GP0)
- net at LED301.1 (K): now also IC302.3 (GP1)
- net at R313.2: now also IC302.4 (~{RESET})
- net at JP302.1, R316.2: now also IC302.5 (URx)
- net at JP301.2, R307.1: now also IC301.1 (EN)
- net at R308.1: now also IC301.5 (RSET)

Commit message: Update
Parts:
- C301, C302, C304, C305, C306, C307: footprint (none) -> tronixio:CAPACITOR-1206
- C303: value (none) -> 1µ; footprint (none) -> tronixio:CAPACITOR-1206
- IC301: value ONSEMI-CAT4002A-SOT-23 -> (none); footprint tronixio:SOT-23-6 -> (none)
- IC302: value MICROCHIP-MCP2221A-ISL -> (none); footprint tronixio:SOIC-SL-14 -> (none)
- K302: value (none) -> HARWIN-254-F-1X06-VERTICAL; footprint (none) -> tronixio:zzHARWIN-M20-782064x
- LED301, LED302: footprint (none) -> tronixio:LED-1206
- R301, R302, R303, R304, R305, R306, R308, R309, R310, R311, R312, R313, R314, R315, R316, R317, R318, R319, R320: footprint (none) -> tronixio:RESISTOR-1206
- R307: value 2K4 -> (none); footprint (none) -> tronixio:RESISTOR-1206
- S301: value (none) -> S1
- S302: value (none) -> S2
Changed lines of the file:
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@@
       (effects (font (size 1.15 1.15)) (justify left))
     )
-    (property "Footprint" "" (id 2) (at 185.42 160.02 0)
+    (property "Footprint" "tronixio:CAPACITOR-1206" (id 2) (at 185.42 160.02 0)
       (effects (font (size 1 1)) hide)
     )
@@
       (effects (font (size 1.15 1.15)))
     )
-    (property "Footprint" "" (id 2) (at 101.6 129.54 0)
+    (property "Footprint" "tronixio:RESISTOR-1206" (id 2) (at 101.6 129.54 0)
       (effects (font (size 1 1)) hide)
     )
@@
       (effects (font (size 1.15 1.15)) (justify right))
     )
-    (property "Footprint" "" (id 2) (at 121.92 86.36 0)
+    (property "Footprint" "tronixio:CAPACITOR-1206" (id 2) (at 121.92 86.36 0)
       (effects (font (size 1 1)) hide)
     )
@@
       (effects (font (size 1.15 1.15)))
     )
-    (property "Value" "ONSEMI-CAT4002A-SOT-23" (id 1) (at 137.16 74.93 0)
-      (effects (font (size 1 1)) hide)
-    )
-    (property "Footprint" "tronixio:SOT-23-6" (id 2) (at 137.16 77.47 0)
+    (property "Value" "" (id 1) (at 137.16 74.93 0)
+      (effects (font (size 1 1)) hide)
+    )
+    (property "Footprint" "" (id 2) (at 137.16 77.47 0)
       (effects (font (size 1 1)) hide)
     )
@@
       (effects (font (size 1.15 1.15)))
     )
-    (property "Footprint" "" (id 2) (at 182.88 55.88 0)
+    (property "Footprint" "tronixio:RESISTOR-1206" (id 2) (at 182.88 55.88 0)
       (effects (font (size 1 1)) hide)
     )
@@
       (effects (font (size 1.15 1.15)) (justify right))
     )
-    (property "Value" "2K4" (id 1) (at 114.3 76.2 90)
-      (effects (font (size 1.15 1.15)))
-    )
-    (property "Footprint" "" (id 2) (at 114.3 88.9 0)
+    (property "Value" "" (id 1) (at 114.3 76.2 90)
+      (effects (font (size 1.15 1.15)))
+    )
+    (property "Footprint" "tronixio:RESISTOR-1206" (id 2) (at 114.3 88.9 0)
       (effects (font (size 1 1)) hide)
     )
@@
       (effects (font (size 1.15 1.15)))
     )
-    (property "Footprint" "" (id 2) (at 154.94 137.16 0)
+    (property "Footprint" "tronixio:RESISTOR-1206" (id 2) (at 154.94 137.16 0)
       (effects (font (size 1 1)) hide)
     )
@@
       (effects (font (size 1.15 1.15)))
     )
-    (property "Footprint" "" (id 2) (at 254 137.16 0)
+    (property "Footprint" "tronixio:RESISTOR-1206" (id 2) (at 254 137.16 0)
       (effects (font (size 1 1)) hide)
     )
@@
       (effects (font (size 1.15 1.15)))
     )
-    (property "Value" "" (id 1) (at 259.08 144.7799 0)
+    (property "Value" "HARWIN-254-F-1X06-VERTICAL" (id 1) (at 259.08 144.7799 0)
       (effects (font (size 1.15 1.15)) (justify left) hide)
     )
-    (property "Footprint" "" (id 2) (at 256.54 160.02 0)
+    (property "Footprint" "tronixio:zzHARWIN-M20-782064x" (id 2) (at 256.54 160.02 0)
       (effects (font (size 1 1)) hide)
     )
@@
       (effects (font (size 1.15 1.15)) (justify left))
     )
-    (property "Value" "" (id 1) (at 46.355 151.13 90)
+    (property "Value" "S1" (id 1) (at 46.355 151.13 90)
       (effects (font (size 1.15 1.15)) (justify left))
     )
@@
       (effects (font (size 1.15 1.15)) (justify left))
     )
-    (property "Value" "" (id 1) (at 67.31 64.77 90)
-      (effects (font (size 1.15 1.15)) (justify right))
-    )
-    (property "Footprint" "" (id 2) (at 76.2 63.5 0)
+    (property "Value" "1µ" (id 1) (at 67.31 64.77 90)
+      (effects (font (size 1.15 1.15)) (justify right))
+    )
+    (property "Footprint" "tronixio:CAPACITOR-1206" (id 2) (at 76.2 63.5 0)
       (effects (font (size 1 1)) hide)
     )
@@
       (effects (font (size 1.15 1.15)))
     )
-    (property "Footprint" "" (id 2) (at 185.42 137.16 0)
+    (property "Footprint" "tronixio:RESISTOR-1206" (id 2) (at 185.42 137.16 0)
       (effects (font (size 1 1)) hide)
     )
@@
       (effects (font (size 1.15 1.15)) (justify right))
     )
-    (property "Footprint" "" (id 2) (at 154.94 160.02 0)
+    (property "Footprint" "tronixio:CAPACITOR-1206" (id 2) (at 154.94 160.02 0)
       (effects (font (size 1 1)) hide)
     )
@@
       (effects (font (size 1.15 1.15)))
     )
-    (property "Footprint" "" (id 2) (at 68.58 137.16 0)
+    (property "Footprint" "tronixio:RESISTOR-1206" (id 2) (at 68.58 137.16 0)
       (effects (font (size 1 1)) hide)
     )
@@
       (effects (font (size 1.15 1.15)))
     )
-    (property "Footprint" "" (id 2) (at 48.26 142.24 0)
+    (property "Footprint" "tronixio:RESISTOR-1206" (id 2) (at 48.26 142.24 0)
       (effects (font (size 1 1)) hide)
     )
@@
       (effects (font (size 1.15 1.15)))
     )
-    (property "Footprint" "" (id 2) (at 160.02 137.16 0)
+    (property "Footprint" "tronixio:RESISTOR-1206" (id 2) (at 160.02 137.16 0)
       (effects (font (size 1 1)) hide)
     )
@@
       (effects (font (size 1.15 1.15)))
     )
-    (property "Footprint" "" (id 2) (at 86.36 139.7 0)
+    (property "Footprint" "tronixio:RESISTOR-1206" (id 2) (at 86.36 139.7 0)
       (effects (font (size 1 1)) hide)
     )
@@
       (effects (font (size 1.15 1.15)) (justify left))
     )
-    (property "Footprint" "" (id 2) (at 215.9 66.04 0)
+    (property "Footprint" "tronixio:LED-1206" (id 2) (at 215.9 66.04 0)
       (effects (font (size 1 1)) hide)
     )
@@
       (effects (font (size 1.15 1.15)))
     )
-    (property "Footprint" "" (id 2) (at 58.42 55.88 0)
+    (property "Footprint" "tronixio:RESISTOR-1206" (id 2) (at 58.42 55.88 0)
       (effects (font (size 1 1)) hide)
     )
@@
       (effects (font (size 1.15 1.15)))
     )
-    (property "Footprint" "" (id 2) (at 223.52 55.88 0)
+    (property "Footprint" "tronixio:RESISTOR-1206" (id 2) (at 223.52 55.88 0)
       (effects (font (size 1 1)) hide)
     )
@@
       (effects (font (size 1.15 1.15)) (justify right))
     )
-    (property "Footprint" "" (id 2) (at 63.5 86.36 0)
+    (property "Footprint" "tronixio:CAPACITOR-1206" (id 2) (at 63.5 86.36 0)
       (effects (font (size 1 1)) hide)
     )
@@
       (effects (font (size 1.15 1.15)))
     )
-    (property "Footprint" "" (id 2) (at 63.5 142.24 0)
+    (property "Footprint" "tronixio:RESISTOR-1206" (id 2) (at 63.5 142.24 0)
       (effects (font (size 1 1)) hide)
     )
@@
       (effects (font (size 1.15 1.15)))
     )
-    (property "Footprint" "" (id 2) (at 218.44 55.88 0)
+    (property "Footprint" "tronixio:RESISTOR-1206" (id 2) (at 218.44 55.88 0)
       (effects (font (size 1 1)) hide)
     )
@@
       (effects (font (size 1.15 1.15)) (justify right))
     )
-    (property "Footprint" "" (id 2) (at 210.82 66.04 0)
+    (property "Footprint" "tronixio:LED-1206" (id 2) (at 210.82 66.04 0)
       (effects (font (size 1 1)) hide)
     )
@@
       (effects (font (size 1.15 1.15)))
     )
-    (property "Footprint" "" (id 2) (at 213.36 55.88 0)
+    (property "Footprint" "tronixio:RESISTOR-1206" (id 2) (at 213.36 55.88 0)
       (effects (font (size 1 1)) hide)
     )
@@
       (effects (font (size 1.15 1.15)))
     )
-    (property "Footprint" "" (id 2) (at 208.28 55.88 0)
+    (property "Footprint" "tronixio:RESISTOR-1206" (id 2) (at 208.28 55.88 0)
       (effects (font (size 1 1)) hide)
     )
@@
       (effects (font (size 1.15 1.15)))
     )
-    (property "Footprint" "" (id 2) (at 147.32 88.9 0)
+    (property "Footprint" "tronixio:RESISTOR-1206" (id 2) (at 147.32 88.9 0)
       (effects (font (size 1 1)) hide)
     )
@@
       (effects (font (size 1.15 1.15)) (justify left))
     )
-    (property "Value" "" (id 1) (at 61.595 151.13 90)
+    (property "Value" "S2" (id 1) (at 61.595 151.13 90)
       (effects (font (size 1.15 1.15)) (justify left))
     )
@@
       (effects (font (size 1.15 1.15)))
     )
-    (property "Footprint" "" (id 2) (at 157.48 134.62 0)
+    (property "Footprint" "tronixio:RESISTOR-1206" (id 2) (at 157.48 134.62 0)
       (effects (font (size 1 1)) hide)
     )
@@
       (effects (font (size 1.15 1.15)))
     )
-    (property "Footprint" "" (id 2) (at 205.74 139.7 0)
+    (property "Footprint" "tronixio:RESISTOR-1206" (id 2) (at 205.74 139.7 0)
       (effects (font (size 1 1)) hide)
     )
@@
       (effects (font (size 1.15 1.15)) (justify right))
     )
-    (property "Footprint" "" (id 2) (at 177.8 86.36 0)
+    (property "Footprint" "tronixio:CAPACITOR-1206" (id 2) (at 177.8 86.36 0)
       (effects (font (size 1 1)) hide)
     )
@@
       (effects (font (size 1.15 1.15)) (justify right))
     )
-    (property "Footprint" "" (id 2) (at 58.42 86.36 0)
+    (property "Footprint" "tronixio:CAPACITOR-1206" (id 2) (at 58.42 86.36 0)
       (effects (font (size 1 1)) hide)
     )
@@
       (effects (font (size 1.15 1.15)))
     )
-    (property "Value" "MICROCHIP-MCP2221A-ISL" (id 1) (at 195.58 81.28 0)
-      (effects (font (size 1 1)) hide)
-    )
-    (property "Footprint" "tronixio:SOIC-SL-14" (id 2) (at 195.58 83.82 0)
+    (property "Value" "" (id 1) (at 195.58 81.28 0)
+      (effects (font (size 1 1)) hide)
+    )
+    (property "Footprint" "" (id 2) (at 195.58 83.82 0)
       (effects (font (size 1 1)) hide)
     )
@@
       (effects (font (size 1.15 1.15)))
     )
-    (property "Footprint" "" (id 2) (at 157.48 139.7 0)
-      (effects (font (size 1 1)) hide)
-    )
+    (property "Footprint" "tronixio:RESISTOR-1206" (id 2) (at 157.48 139.7 0)
+      (effects (font (size 1 1)) hide)
+    )

Commit message: Update Kicad
Parts:
- IC301: value (none) -> CAT4002A; footprint (none) -> tronixio:SOT-23-6
- IC302: value (none) -> MCP2221A; footprint (none) -> tronixio:SOIC-SL-14
- R307: value (none) -> 10K
Changed lines of the file:
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@@
       (effects (font (size 1.15 1.15)))
     )
-    (property "Value" "" (id 1) (at 137.16 74.93 0)
-      (effects (font (size 1 1)) hide)
-    )
-    (property "Footprint" "" (id 2) (at 137.16 77.47 0)
+    (property "Value" "CAT4002A" (id 1) (at 137.16 74.93 0)
+      (effects (font (size 1 1)) hide)
+    )
+    (property "Footprint" "tronixio:SOT-23-6" (id 2) (at 137.16 77.47 0)
       (effects (font (size 1 1)) hide)
     )
@@
       (effects (font (size 1.15 1.15)) (justify right))
     )
-    (property "Value" "" (id 1) (at 114.3 76.2 90)
+    (property "Value" "10K" (id 1) (at 114.3 76.2 90)
       (effects (font (size 1.15 1.15)))
     )
@@
       (effects (font (size 1.15 1.15)))
     )
-    (property "Value" "" (id 1) (at 195.58 81.28 0)
-      (effects (font (size 1 1)) hide)
-    )
-    (property "Footprint" "" (id 2) (at 195.58 83.82 0)
-      (effects (font (size 1 1)) hide)
-    )
+    (property "Value" "MCP2221A" (id 1) (at 195.58 81.28 0)
+      (effects (font (size 1 1)) hide)
+    )
+    (property "Footprint" "tronixio:SOIC-SL-14" (id 2) (at 195.58 83.82 0)
+      (effects (font (size 1 1)) hide)
+    )

Commit message: Update Kicad
Connections:
- net PGC/UTX/RB1 renamed PGC/URX/RB1
Changed lines of the file:
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@@
     (effects (font (size 1.2 1.2)) (justify right))
   )
-  (hierarchical_label "PGD{slash}UTX{slash}RB0" (shape output) (at 243.84 53.34 0)
+  (hierarchical_label "PGD{slash}UTX{slash}RB0" (shape input) (at 243.84 53.34 0)
     (effects (font (size 1.2 1.2)) (justify left))
   )
@@
     (effects (font (size 1.2 1.2)) (justify right))
   )
-  (hierarchical_label "PGC{slash}UTX{slash}RB1" (shape input) (at 243.84 55.88 0)
+  (hierarchical_label "PGC{slash}URX{slash}RB1" (shape output) (at 243.84 55.88 0)
     (effects (font (size 1.2 1.2)) (justify left))
   )

Commit message: Update
Other:
- moved on the sheet: R309, R310
Changed lines of the file:
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@@
     (stroke (width 0) (type solid) (color 0 0 0 0))
   )
-  (wire (pts (xy 149.86 139.7) (xy 154.94 139.7))
+  (wire (pts (xy 152.4 139.7) (xy 154.94 139.7))
     (stroke (width 0) (type solid) (color 0 0 0 0))
   )
@@
     (stroke (width 0) (type solid) (color 0 0 0 0))
   )
-  (wire (pts (xy 149.86 134.62) (xy 160.02 134.62))
+  (wire (pts (xy 152.4 134.62) (xy 160.02 134.62))
     (stroke (width 0) (type solid) (color 0 0 0 0))
   )
@@
     )
   )
-  (global_label "ROTARY_A" (shape output) (at 139.7 139.7 180) (fields_autoplaced)
+  (global_label "ROTARY_A" (shape output) (at 142.24 139.7 180) (fields_autoplaced)
     (effects (font (size 1.2 1.2)) (justify right))
-    (property "Intersheet References" "${INTERSHEET_REFS}" (id 0) (at 128.6686 139.625 0)
+    (property "Intersheet References" "${INTERSHEET_REFS}" (id 0) (at 131.2086 139.625 0)
       (effects (font (size 1.2 1.2)) (justify right) hide)
     )
@@
     )
   )
-  (global_label "ROTARY_S" (shape output) (at 139.7 134.62 180) (fields_autoplaced)
+  (global_label "ROTARY_S" (shape output) (at 142.24 134.62 180) (fields_autoplaced)
     (effects (font (size 1.2 1.2)) (justify right))
-    (property "Intersheet References" "${INTERSHEET_REFS}" (id 0) (at 128.5543 134.545 0)
+    (property "Intersheet References" "${INTERSHEET_REFS}" (id 0) (at 131.0943 134.545 0)
       (effects (font (size 1.2 1.2)) (justify right) hide)
     )
@@
     (pin "1")
   )
-  (symbol (lib_id "tronixio:R-0805") (at 144.78 134.62 90) (unit 1)
-    (in_bom yes) (on_board yes)
-    (property "Reference" "R309" (id 0) (at 144.78 132.08 90)
-      (effects (font (size 1.15 1.15)))
-    )
-    (property "Value" "1K" (id 1) (at 144.78 134.62 90)
-      (effects (font (size 1.15 1.15)))
-    )
-    (property "Footprint" "tronixio:RESISTOR-1206" (id 2) (at 157.48 134.62 0)
-      (effects (font (size 1 1)) hide)
-    )
-    (property "Datasheet" "" (id 3) (at 144.78 134.62 0)
+  (symbol (lib_id "tronixio:R-0805") (at 147.32 134.62 90) (unit 1)
+    (in_bom yes) (on_board yes)
+    (property "Reference" "R309" (id 0) (at 147.32 132.08 90)
+      (effects (font (size 1.15 1.15)))
+    )
+    (property "Value" "1K" (id 1) (at 147.32 134.62 90)
+      (effects (font (size 1.15 1.15)))
+    )
+    (property "Footprint" "tronixio:RESISTOR-1206" (id 2) (at 160.02 134.62 0)
+      (effects (font (size 1 1)) hide)
+    )
+    (property "Datasheet" "" (id 3) (at 147.32 134.62 0)
       (effects (font (size 1 1)) hide)
     )
@@
     (pin "9")
   )
-  (symbol (lib_id "tronixio:R-0805") (at 144.78 139.7 90) (unit 1)
-    (in_bom yes) (on_board yes)
-    (property "Reference" "R310" (id 0) (at 144.78 142.24 90)
-      (effects (font (size 1.15 1.15)))
-    )
-    (property "Value" "10K" (id 1) (at 144.78 139.7 90)
-      (effects (font (size 1.15 1.15)))
-    )
-    (property "Footprint" "tronixio:RESISTOR-1206" (id 2) (at 157.48 139.7 0)
-      (effects (font (size 1 1)) hide)
-    )
-    (property "Datasheet" "" (id 3) (at 144.78 139.7 0)
-      (effects (font (size 1 1)) hide)
-    )
+  (symbol (lib_id "tronixio:R-0805") (at 147.32 139.7 90) (unit 1)
+    (in_bom yes) (on_board yes)
+    (property "Reference" "R310" (id 0) (at 147.32 142.24 90)
+      (effects (font (size 1.15 1.15)))
+    )
+    (property "Value" "10K" (id 1) (at 147.32 139.7 90)
+      (effects (font (size 1.15 1.15)))
+    )
+    (property "Footprint" "tronixio:RESISTOR-1206" (id 2) (at 160.02 139.7 0)
+      (effects (font (size 1 1)) hide)
+    )
+    (property "Datasheet" "" (id 3) (at 147.32 139.7 0)
+      (effects (font (size 1 1)) hide)
+    )

Commit message: Update Mini
Parts:
- IC302: Name MCP2221A-ISL -> MCP2221A
- JP301: value EN BCKL -> BCKL
Other:
- note added: "EN"
Changed lines of the file:
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@@
     (effects (font (size 1.15 1.15)) (justify left bottom))
+  )
+  (text "EN" (at 112.395 59.69 180)
+    (effects (font (size 1.15 1.15)) (justify right bottom))
   )
   (text "ROTARY S" (at 259.08 146.05 0)
@@
       (effects (font (size 1.15 1.15)) (justify left))
     )
-    (property "Value" "EN BCKL" (id 1) (at 113.665 60.96 0)
+    (property "Value" "BCKL" (id 1) (at 113.665 60.96 0)
       (effects (font (size 1.15 1.15)) (justify left))
     )
@@
       (effects (font (size 1 1)) hide)
     )
-    (property "Name" "MCP2221A-ISL" (id 4) (at 195.58 77.47 0)
-      (effects (font (size 1.15 1.15)))
-    )
+    (property "Name" "MCP2221A" (id 4) (at 195.58 77.47 0)
+      (effects (font (size 1.15 1.15)))
+    )

Commit message: Update
Other:
- note added: "Ibckl ~30mA = (125 * 0.6) / 2400"
- moved on the sheet: BB301, C301, C302, C303, C304, C305, C306, C307, IC301, IC302, JP301, JP302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

Commit message: Updaet
Parts:
- K302: footprint tronixio:zzHARWIN-M20-782064x -> tronixio:HARWIN-M20-782064x
Changed lines of the file:
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@@
       (effects (font (size 1.15 1.15)) (justify left) hide)
     )
-    (property "Footprint" "tronixio:zzHARWIN-M20-782064x" (id 2) (at 251.46 160.02 0)
+    (property "Footprint" "tronixio:HARWIN-M20-782064x" (id 2) (at 251.46 160.02 0)
       (effects (font (size 1 1)) hide)
     )
