File: Kicad/mini/pic16bit-hid.kicad_sch (KiCad schematic)
At the start: 43 parts, among them IC301 CAT4002A, IC302 MCP2221A, K301 HARWIN-254-F-1X08-VERTICAL, K302 HARWIN-254-F-1X06-VERTICAL, P301 PIHER-PT10MV-10K, P302 PIHER-PT10MV-10K

Commit message: Update
Parts:
- U302: renamed from IC302; Name MCP2221A -> MCP2221A-ISL
- renumbered IC301 to U301
Changed lines of the file:
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@@
   (symbol (lib_id "tronixio:ONSEMI-CAT4002A-SOT-23") (at 132.08 66.04 0) (unit 1)
     (in_bom yes) (on_board yes)
-    (property "Reference" "IC301" (id 0) (at 132.08 59.69 0)
+    (property "Reference" "U301" (id 0) (at 132.08 59.69 0)
       (effects (font (size 1.15 1.15)))
     )
@@
   (symbol (lib_id "tronixio:MICROCHIP-MCP2221A-ISL") (at 190.5 63.5 0) (unit 1)
     (in_bom yes) (on_board yes)
-    (property "Reference" "IC302" (id 0) (at 190.5 49.53 0)
+    (property "Reference" "U302" (id 0) (at 190.5 49.53 0)
       (effects (font (size 1.15 1.15)))
     )
@@
       (effects (font (size 1 1)) hide)
     )
-    (property "Name" "MCP2221A" (id 4) (at 190.5 77.47 0)
-      (effects (font (size 1.15 1.15)))
-    )
+    (property "Name" "MCP2221A-ISL" (id 4) (at 190.5 77.47 0)
+      (effects (font (size 1.15 1.15)))
+    )

Commit message: Update
Parts:
- C301, C305, C307: value 10n -> CAPACITOR-0805-100N; footprint tronixio:CAPACITOR-1206 -> tronixio:CAPACITOR-0805; symbol tronixio:C-0805 -> tronixio:CAPACITOR-0805-100N; Mouser (none) -> 80-C0805C104M5R; Name (none) -> CAPACITOR-0805-100N; Tolerance (none) -> 20%; Voltage (none) -> 50V
- C302, C303, C304: value 1µ -> CAPACITOR-0805-100N; footprint tronixio:CAPACITOR-1206 -> tronixio:CAPACITOR-0805; symbol tronixio:C-0805 -> tronixio:CAPACITOR-0805-100N; Mouser (none) -> 80-C0805C104M5R; Name (none) -> CAPACITOR-0805-100N; Tolerance (none) -> 20%; Voltage (none) -> 50V
- C306: value 100n -> CAPACITOR-0805-100N; footprint tronixio:CAPACITOR-1206 -> tronixio:CAPACITOR-0805; symbol tronixio:C-0805 -> tronixio:CAPACITOR-0805-100N; Mouser (none) -> 80-C0805C104M5R; Name (none) -> CAPACITOR-0805-100N; Tolerance (none) -> 20%; Voltage (none) -> 50V
- JP301: value BCKL -> HARWIN-254-M-1X02-JUMPER-VERTICAL; Name (none) -> HARWIN-254-M-1X02-JUMPER-VERTICAL
- JP302: value UTX -> HARWIN-254-M-1X02-JUMPER-VERTICAL; Name (none) -> HARWIN-254-M-1X02-JUMPER-VERTICAL
- JP303: value URX -> HARWIN-254-M-1X02-JUMPER-VERTICAL; Name (none) -> HARWIN-254-M-1X02-JUMPER-VERTICAL
- K301, K302: Name (none) -> HARWIN-254-F-1X06-VERTICAL
- LED301: value URX -> KINGBRIGHT-LED-0805-BLUE; footprint tronixio:LED-1206 -> tronixio:LED-0805; symbol tronixio:LED-0805-ORANGE -> tronixio:KINGBRIGHT-LED-0805-BLUE; Mouser 604-APT2012LSECKJ4RV -> 604-APT2012LVBCD; Name (none) -> KINGBRIGHT-LED-0805-BLUE
- LED302: value UTX -> KINGBRIGHT-LED-0805-BLUE; footprint tronixio:LED-1206 -> tronixio:LED-0805; symbol tronixio:LED-0805-ORANGE -> tronixio:KINGBRIGHT-LED-0805-BLUE; Mouser 604-APT2012LSECKJ4RV -> 604-APT2012LVBCD; Name (none) -> KINGBRIGHT-LED-0805-BLUE
- P301, P302: Name 10K -> PIHER-PT10MV-10K; Tolerance (none) -> 20%
- R301, R303, R304, R307, R310, R311, R312, R313, R314, R315, R316, R317: value 10K -> RESISTOR-0805-1K; footprint tronixio:RESISTOR-1206 -> tronixio:RESISTOR-0805; symbol tronixio:R-0805 -> tronixio:RESISTOR-0805-1K; Mouser (none) -> 660-RK73B2ATTDD102J; Name (none) -> RESISTOR-0805-1K; Tolerance (none) -> 5%
- R302, R305, R306, R309, R320: value 1K -> RESISTOR-0805-1K; footprint tronixio:RESISTOR-1206 -> tronixio:RESISTOR-0805; symbol tronixio:R-0805 -> tronixio:RESISTOR-0805-1K; Mouser (none) -> 660-RK73B2ATTDD102J; Name (none) -> RESISTOR-0805-1K; Tolerance (none) -> 5%
- R308: value 2K4 -> RESISTOR-0805-1K; footprint tronixio:RESISTOR-1206 -> tronixio:RESISTOR-0805; symbol tronixio:R-0805 -> tronixio:RESISTOR-0805-1K; Mouser (none) -> 660-RK73B2ATTDD102J; Name (none) -> RESISTOR-0805-1K; Tolerance (none) -> 5%
- R318, R319: value 4K7 -> RESISTOR-0805-1K; footprint tronixio:RESISTOR-1206 -> tronixio:RESISTOR-0805; symbol tronixio:R-0805 -> tronixio:RESISTOR-0805-1K; Mouser (none) -> 660-RK73B2ATTDD102J; Name (none) -> RESISTOR-0805-1K; Tolerance (none) -> 5%
- S301: value S1 -> CK-KSA; Name (none) -> CK-KSA
- S302: value S2 -> CK-KSA; Name (none) -> CK-KSA
- S303: value BOURNS-PEC12R-24DENTS -> BOURNS-PEC12R-24DENTS-SWITCH; footprint tronixio:BOURNS-PEC12R -> tronixio:BOURNS-PEC12R-SWITCH; symbol tronixio:BOURNS-PEC12R-24DENTS -> tronixio:BOURNS-PEC12R-24DENTS-SWITCH; Name (none) -> BOURNS-PEC12R-24DENTS-SWITCH
- U301: value CAT4002A -> ONSEMI-CAT4002A-SOT-23; Name CAT4002A -> ONSEMI-CAT4002A-SOT-23
- U302: value MCP2221A -> MICROCHIP-MCP2221A-ISL; footprint tronixio:SOIC-SL-14 -> tronixio:SOIC-14; Name MCP2221A-ISL -> MICROCHIP-MCP2221A-ISL
Connections:
- net GND: no longer S301.1, S301.2, S302.1, S302.2
- net at R301.2, R302.1: no longer S301.3, S301.4
- net at R304.2, R305.1: no longer S302.3, S302.4
Other:
- moved on the sheet: S301, S302

Commit message: Update
Parts:
- C301, C305, C307: value CAPACITOR-0805-100N -> 10n; footprint tronixio:CAPACITOR-0805 -> tronixio:CAPACITOR-1206; symbol tronixio:CAPACITOR-0805-100N -> tronixio:CAPACITOR-1206-10N; Mouser 80-C0805C104M5R -> 80-C1206C103M5R; Name CAPACITOR-0805-100N -> CAPACITOR-1206-10N
- C302, C303, C304: value CAPACITOR-0805-100N -> 1µ; footprint tronixio:CAPACITOR-0805 -> tronixio:CAPACITOR-1206; symbol tronixio:CAPACITOR-0805-100N -> tronixio:CAPACITOR-1206-1U; Mouser 80-C0805C104M5R -> C1206C105M5RACTU; Name CAPACITOR-0805-100N -> CAPACITOR-1206-1U
- C306: value CAPACITOR-0805-100N -> 100n; footprint tronixio:CAPACITOR-0805 -> tronixio:CAPACITOR-1206; symbol tronixio:CAPACITOR-0805-100N -> tronixio:CAPACITOR-1206-100N; Mouser 80-C0805C104M5R -> 80-C1206C104M5R; Name CAPACITOR-0805-100N -> CAPACITOR-1206-100N
- JP301: value HARWIN-254-M-1X02-JUMPER-VERTICAL -> BCKL
- JP302: value HARWIN-254-M-1X02-JUMPER-VERTICAL -> UTX
- JP303: value HARWIN-254-M-1X02-JUMPER-VERTICAL -> URX
- LED301: value KINGBRIGHT-LED-0805-BLUE -> URX; footprint tronixio:LED-0805 -> tronixio:LED-1206; symbol tronixio:KINGBRIGHT-LED-0805-BLUE -> tronixio:KINGBRIGHT-LED-1206-BLUE; Mouser 604-APT2012LVBCD -> 604-APT3216LVBCD; Name KINGBRIGHT-LED-0805-BLUE -> KINGBRIGHT-LED-1206-BLUE
- LED302: value KINGBRIGHT-LED-0805-BLUE -> UTX; footprint tronixio:LED-0805 -> tronixio:LED-1206; symbol tronixio:KINGBRIGHT-LED-0805-BLUE -> tronixio:KINGBRIGHT-LED-1206-BLUE; Mouser 604-APT2012LVBCD -> 604-APT3216LVBCD; Name KINGBRIGHT-LED-0805-BLUE -> KINGBRIGHT-LED-1206-BLUE
- P301, P302: value PIHER-PT10MV-10K -> 10K
- R301, R303, R304, R307, R310, R311, R312, R313, R314, R316, R317: value RESISTOR-0805-1K -> 10K; footprint tronixio:RESISTOR-0805 -> tronixio:RESISTOR-1206; symbol tronixio:RESISTOR-0805-1K -> tronixio:RESISTOR-1206-10K; Mouser 660-RK73B2ATTDD102J -> 660-RK73B2BTTDD103J; Name RESISTOR-0805-1K -> RESISTOR-1206-10K
- R302, R305, R306, R309, R320: value RESISTOR-0805-1K -> 1K; footprint tronixio:RESISTOR-0805 -> tronixio:RESISTOR-1206; symbol tronixio:RESISTOR-0805-1K -> tronixio:RESISTOR-1206-1K; Mouser 660-RK73B2ATTDD102J -> 660-RK73B2BTTDD102J; Name RESISTOR-0805-1K -> RESISTOR-1206-1K
- R308: value RESISTOR-0805-1K -> 2K4; footprint tronixio:RESISTOR-0805 -> tronixio:RESISTOR-1206; symbol tronixio:RESISTOR-0805-1K -> tronixio:RESISTOR-1206-2K4; Mouser 660-RK73B2ATTDD102J -> 660-RK73B2BTTD242J; Name RESISTOR-0805-1K -> RESISTOR-1206-2K4
- R315: value RESISTOR-0805-1K -> 1K; footprint tronixio:RESISTOR-0805 -> tronixio:RESISTOR-1206; symbol tronixio:RESISTOR-0805-1K -> tronixio:RESISTOR-1206-10K; Mouser 660-RK73B2ATTDD102J -> 660-RK73B2BTTDD103J; Name RESISTOR-0805-1K -> RESISTOR-1206-10K
- R318, R319: value RESISTOR-0805-1K -> 4K7; footprint tronixio:RESISTOR-0805 -> tronixio:RESISTOR-1206; symbol tronixio:RESISTOR-0805-1K -> tronixio:RESISTOR-1206-4K7; Mouser 660-RK73B2ATTDD102J -> 660-RK73B2BTTDD472J; Name RESISTOR-0805-1K -> RESISTOR-1206-4K7
- S301: value CK-KSA -> S1
- S302: value CK-KSA -> S2
- U301: value ONSEMI-CAT4002A-SOT-23 -> CAT4002A
- U302: value MICROCHIP-MCP2221A-ISL -> MCP2221A-ISL
Connections:
- net GND: now also S301.1, S301.2, S302.1, S302.2
- net at S301.3: now also R301.2, R302.1, S301.4
- net at R304.2, R305.1: now also S302.3, S302.4
Other:
- moved on the sheet: S301, S302

Commit message: Update
Parts:
- C301, C302, C303, C304, C305, C306, C307: footprint tronixio:CAPACITOR-1206 -> tronixio:CAPACITOR-SMD-1206
- LED301, LED302: footprint tronixio:LED-1206 -> tronixio:LED-SMD-1206
- R301, R302, R303, R304, R305, R306, R307, R308, R309, R310, R311, R312, R313, R314, R315, R316, R317, R318, R319, R320: footprint tronixio:RESISTOR-1206 -> tronixio:RESISTOR-SMD-1206

Commit message: Update
Parts:
- U301: footprint tronixio:SOT-23-6 -> tronixioZZZ:SC-70-6; symbol tronixio:ONSEMI-CAT4002A-SOT-23 -> tronixio:ONSEMI-CAT4002A-SC-70; Mouser 863-CAT4002ATD-GT3 -> 863-CAT4002ASD-GT3; Name ONSEMI-CAT4002A-SOT-23 -> ONSEMI-CAT4002A-SC-70
- U302: value MCP2221A-ISL -> MCP2221A
Changed lines of the file:
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@@
     (effects (font (size 1.2 1.2)) (justify left))
   )
-  (hierarchical_label "SCL" (shape input) (at 48.26 55.88 180)
+  (hierarchical_label "SCL" (shape bidirectional) (at 48.26 55.88 180)
     (effects (font (size 1.2 1.2)) (justify right))
   )
@@
     (effects (font (size 1.2 1.2)) (justify right))
   )
-  (hierarchical_label "SCL" (shape output) (at 238.76 58.42 0)
+  (hierarchical_label "SCL" (shape bidirectional) (at 238.76 58.42 0)
     (effects (font (size 1.2 1.2)) (justify left))
   )
@@
     (pin "3")
   )
-  (symbol (lib_id "tronixio:ONSEMI-CAT4002A-SOT-23") (at 124.46 63.5 0) (unit 1)
+  (symbol (lib_id "tronixio:ONSEMI-CAT4002A-SC-70") (at 124.46 63.5 0) (unit 1)
     (in_bom yes) (on_board yes)
     (property "Reference" "U301" (id 0) (at 132.08 59.69 0)
@@
       (effects (font (size 1.15 1.15)))
     )
-    (property "Footprint" "tronixio:SOT-23-6" (id 2) (at 132.08 78.74 0)
+    (property "Footprint" "tronixioZZZ:SC-70-6" (id 2) (at 132.08 78.74 0)
       (effects (font (size 1 1)) hide)
     )
@@
       (effects (font (size 1 1)) hide)
     )
-    (property "Name" "ONSEMI-CAT4002A-SOT-23" (id 4) (at 132.08 76.2 0)
-      (effects (font (size 1 1)) hide)
-    )
-    (property "Mouser" "863-CAT4002ATD-GT3" (id 5) (at 132.08 83.82 0)
+    (property "Name" "ONSEMI-CAT4002A-SC-70" (id 4) (at 132.08 76.2 0)
+      (effects (font (size 1 1)) hide)
+    )
+    (property "Mouser" "863-CAT4002ASD-GT3" (id 5) (at 132.08 83.82 0)
       (effects (font (size 1 1)) hide)
     )
@@
       (effects (font (size 1.15 1.15)) (justify right))
     )
-    (property "Value" "10K" (id 1) (at 180.34 44.45 0)
+    (property "Value" "10K" (id 1) (at 177.8 43.18 90)
       (effects (font (size 1.15 1.15)))
     )
@@
       (effects (font (size 1.15 1.15)) (justify right))
     )
-    (property "Value" "10K" (id 1) (at 111.76 77.47 0)
+    (property "Value" "10K" (id 1) (at 109.22 76.2 90)
       (effects (font (size 1.15 1.15)))
     )
@@
       (effects (font (size 1.15 1.15)) (justify left))
     )
-    (property "Value" "4K7" (id 1) (at 220.98 44.45 0)
+    (property "Value" "4K7" (id 1) (at 218.44 43.18 90)
       (effects (font (size 1.15 1.15)))
     )
@@
       (effects (font (size 1.15 1.15)) (justify left))
     )
-    (property "Value" "4K7" (id 1) (at 215.9 44.45 0)
+    (property "Value" "4K7" (id 1) (at 213.36 43.18 90)
       (effects (font (size 1.15 1.15)))
     )
@@
       (effects (font (size 1.15 1.15)) (justify left))
     )
-    (property "Value" "10K" (id 1) (at 210.82 44.45 0)
+    (property "Value" "10K" (id 1) (at 208.28 43.18 90)
       (effects (font (size 1.15 1.15)))
     )
@@
       (effects (font (size 1.15 1.15)) (justify left))
     )
-    (property "Value" "10K" (id 1) (at 205.74 44.45 0)
+    (property "Value" "10K" (id 1) (at 203.2 43.18 90)
       (effects (font (size 1.15 1.15)))
     )
@@
       (effects (font (size 1.15 1.15)) (justify left))
     )
-    (property "Value" "2K4" (id 1) (at 144.78 77.47 0)
+    (property "Value" "2K4" (id 1) (at 142.24 76.2 90)
       (effects (font (size 1.15 1.15)))
     )
@@
   (symbol (lib_id "tronixio:MICROCHIP-MCP2221A-ISL") (at 180.34 53.34 0) (unit 1)
     (in_bom yes) (on_board yes)
-    (property "Reference" "U302" (id 0) (at 180.34 39.37 0)
-      (effects (font (size 1.15 1.15)))
-    )
-    (property "Value" "MCP2221A-ISL" (id 1) (at 190.5 77.47 0)
-      (effects (font (size 1.15 1.15)))
+    (property "Reference" "U302" (id 0) (at 182.88 49.53 0)
+      (effects (font (size 1.15 1.15)) (justify left))
+    )
+    (property "Value" "MCP2221A" (id 1) (at 198.12 49.53 0)
+      (effects (font (size 1.15 1.15)) (justify right))
     )
     (property "Footprint" "tronixio:SOIC-14" (id 2) (at 190.5 83.82 0)

Commit message: Update Mini
Parts:
- C301, C305, C307: symbol tronixio:CAPACITOR-1206-10N -> tronixio:KEMET-X7R-1206-10N-50V-20P; Name CAPACITOR-1206-10N -> (none)
- C302, C303, C304: symbol tronixio:CAPACITOR-1206-1U -> tronixio:KEMET-X7R-1206-1U-50V-20P; Mouser C1206C105M5RACTU -> 80-C1206C105M5R; Name CAPACITOR-1206-1U -> (none)
- C306: symbol tronixio:CAPACITOR-1206-100N -> tronixio:KEMET-X7R-1206-100N-50V-20P; Name CAPACITOR-1206-100N -> (none)
- JP301, JP302, JP303: Name HARWIN-254-M-1X02-JUMPER-VERTICAL -> (none)
- K301, K302: Name HARWIN-254-F-1X06-VERTICAL -> (none)
- LED301, LED302: Name KINGBRIGHT-LED-1206-BLUE -> (none)
- P301, P302: Name PIHER-PT10MV-10K -> (none)
- R301, R303, R304, R307, R310, R311, R312, R313, R314, R315, R316, R317: symbol tronixio:RESISTOR-1206-10K -> tronixio:KOASPEER-RK73B-1206-10K-5P; Name RESISTOR-1206-10K -> (none)
- R302, R305, R306, R309, R320: symbol tronixio:RESISTOR-1206-1K -> tronixio:KOASPEER-RK73B-1206-1K-5P; Name RESISTOR-1206-1K -> (none)
- R308: symbol tronixio:RESISTOR-1206-2K4 -> tronixio:KOASPEER-RK73B-1206-2K4-5P; Mouser 660-RK73B2BTTD242J -> 660-RK73B2BTTDD242J; Name RESISTOR-1206-2K4 -> (none)
- R318, R319: symbol tronixio:RESISTOR-1206-4K7 -> tronixio:KOASPEER-RK73B-1206-4K7-5P; Name RESISTOR-1206-4K7 -> (none)
- S301, S302: Name CK-KSA -> (none)
- S303: Name BOURNS-PEC12R-24DENTS-SWITCH -> (none)
- U301: footprint tronixioZZZ:SC-70-6 -> tronixio:SC-70-6; Name ONSEMI-CAT4002A-SC-70 -> (none)
- U302: Name MICROCHIP-MCP2221A-ISL -> (none)
Other:
- moved on the sheet: JP301, JP302, JP303

Commit message: Update Mini
Parts:
- C302, C303, C304: symbol tronixio:KEMET-X7R-1206-1U-50V-20P -> tronixio:KEMET-X7R-1206-1U-16V-20P; Mouser 80-C1206C105M5R -> 80-C1206C105M4R; Voltage 50V -> 16V
Changed lines of the file:
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@@
     (pin "5")
   )
-  (symbol (lib_id "tronixio:KEMET-X7R-1206-1U-50V-20P") (at 116.84 76.2 0) (unit 1)
+  (symbol (lib_id "tronixio:KEMET-X7R-1206-1U-16V-20P") (at 116.84 76.2 0) (unit 1)
     (in_bom yes) (on_board yes)
     (property "Reference" "C304" (id 0) (at 116.205 73.66 0)
@@
       (effects (font (size 1 1)) hide)
     )
-    (property "Voltage" "50V" (id 4) (at 118.11 81.28 0)
+    (property "Voltage" "16V" (id 4) (at 118.11 81.28 0)
       (effects (font (size 1.15 1.15)) (justify left) hide)
     )
@@
       (effects (font (size 1.15 1.15)) (justify left) hide)
     )
-    (property "Mouser" "80-C1206C105M5R" (id 6) (at 116.84 91.44 0)
+    (property "Mouser" "80-C1206C105M4R" (id 6) (at 116.84 91.44 0)
       (effects (font (size 1 1)) hide)
     )
@@
     (pin "1")
   )
-  (symbol (lib_id "tronixio:KEMET-X7R-1206-1U-50V-20P") (at 60.96 63.5 90) (unit 1)
+  (symbol (lib_id "tronixio:KEMET-X7R-1206-1U-16V-20P") (at 60.96 63.5 90) (unit 1)
     (in_bom yes) (on_board yes)
     (property "Reference" "C303" (id 0) (at 59.69 64.77 90)
@@
       (effects (font (size 1 1)) hide)
     )
-    (property "Voltage" "50V" (id 4) (at 66.04 62.23 0)
+    (property "Voltage" "16V" (id 4) (at 66.04 62.23 0)
       (effects (font (size 1.15 1.15)) (justify left) hide)
     )
@@
       (effects (font (size 1.15 1.15)) (justify left) hide)
     )
-    (property "Mouser" "80-C1206C105M5R" (id 6) (at 76.2 63.5 0)
+    (property "Mouser" "80-C1206C105M4R" (id 6) (at 76.2 63.5 0)
       (effects (font (size 1 1)) hide)
     )
@@
     (pin "2")
   )
-  (symbol (lib_id "tronixio:KEMET-X7R-1206-1U-50V-20P") (at 58.42 76.2 0) (unit 1)
+  (symbol (lib_id "tronixio:KEMET-X7R-1206-1U-16V-20P") (at 58.42 76.2 0) (unit 1)
     (in_bom yes) (on_board yes)
     (property "Reference" "C302" (id 0) (at 58.42 73.66 0)
@@
       (effects (font (size 1 1)) hide)
     )
-    (property "Voltage" "50V" (id 4) (at 59.69 81.28 0)
+    (property "Voltage" "16V" (id 4) (at 59.69 81.28 0)
       (effects (font (size 1.15 1.15)) (justify left) hide)
     )
@@
       (effects (font (size 1.15 1.15)) (justify left) hide)
     )
-    (property "Mouser" "80-C1206C105M5R" (id 6) (at 58.42 91.44 0)
-      (effects (font (size 1 1)) hide)
-    )
+    (property "Mouser" "80-C1206C105M4R" (id 6) (at 58.42 91.44 0)
+      (effects (font (size 1 1)) hide)
+    )

Commit message: Up
Parts:
- C301, C305, C307: symbol tronixio:KEMET-X7R-1206-10N-50V-20P -> tronixio:CAPACITOR-1206-10N-20P-X7R
- C302, C303, C304: symbol tronixio:KEMET-X7R-1206-1U-16V-20P -> tronixio:CAPACITOR-1206-1U-10P-X7R; Mouser 80-C1206C105M4R -> 80-C1206C105K5R; Tolerance 20% -> 10%; Voltage 16V -> 50V
- C306: symbol tronixio:KEMET-X7R-1206-100N-50V-20P -> tronixio:CAPACITOR-1206-100N-10P-X7R; Mouser 80-C1206C104M5R -> 80-C1206C104K5R; Tolerance 20% -> 10%
- R301, R303, R304, R307, R310, R311, R312, R313, R314, R315, R316, R317: symbol tronixio:KOASPEER-RK73B-1206-10K-5P -> tronixio:RESISTOR-1206-10K-5P
- R302, R305, R306, R309, R320: symbol tronixio:KOASPEER-RK73B-1206-1K-5P -> tronixio:RESISTOR-1206-1K-5P
- R308: symbol tronixio:KOASPEER-RK73B-1206-2K4-5P -> tronixio:RESISTOR-1206-2K4-5P
- R318, R319: symbol tronixio:KOASPEER-RK73B-1206-4K7-5P -> tronixio:RESISTOR-1206-4K7-5P
