File: Kicad/mini/pic16bit-hid.kicad_sch (KiCad schematic)
At the start: 43 parts, among them K301 HARWIN-254-F-1X08-VERTICAL, K302 HARWIN-254-F-1X06-VERTICAL, P301 10K, P302 10K, U301 CAT4002A, U302 MCP2221A

Commit message: Update
Parts:
- C302, C303, C304: Mouser 80-C1206C105K5R -> 80-C1206C105K4R; Voltage 50V -> 16V
- C306: Mouser 80-C1206C104K5R -> 187-CL31B106KAHNFNE
- S303: symbol tronixio:BOURNS-PEC12R-24DENTS-SWITCH -> tronixio:BOURNS-PEC12R-24-DENTS-SWITCH
Changed lines of the file:
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@@
     )
   )
-  (symbol (lib_id "tronixio:BOURNS-PEC12R-24DENTS-SWITCH") (at 165.1 139.7 0) (unit 1)
+  (symbol (lib_id "tronixio:BOURNS-PEC12R-24-DENTS-SWITCH") (at 165.1 139.7 0) (unit 1)
     (in_bom yes) (on_board yes) (dnp no)
     (property "Reference" "S303" (at 165.1 128.27 0)
@@
       (effects (font (size 1 1)) hide)
     )
-    (property "Voltage" "50V" (at 121.84 81.28 0) (do_not_autoplace)
+    (property "Voltage" "16V" (at 121.84 81.28 0) (do_not_autoplace)
       (effects (font (size 1.15 1.15)) (justify left) hide)
     )
@@
       (effects (font (size 1.15 1.15)) (justify left) hide)
     )
-    (property "Mouser" "80-C1206C105K5R" (at 116.84 88.9 0)
+    (property "Mouser" "80-C1206C105K4R" (at 116.84 88.9 0)
       (effects (font (size 1 1)) hide)
     )
@@
       (effects (font (size 1 1)) hide)
     )
-    (property "Voltage" "50V" (at 66.04 58.5 0) (do_not_autoplace)
+    (property "Voltage" "16V" (at 66.04 58.5 0) (do_not_autoplace)
       (effects (font (size 1.15 1.15)) (justify left) hide)
     )
@@
       (effects (font (size 1.15 1.15)) (justify left) hide)
     )
-    (property "Mouser" "80-C1206C105K5R" (at 73.66 63.5 0)
+    (property "Mouser" "80-C1206C105K4R" (at 73.66 63.5 0)
       (effects (font (size 1 1)) hide)
     )
@@
       (effects (font (size 1 1)) hide)
     )
-    (property "Voltage" "50V" (at 63.42 81.28 0) (do_not_autoplace)
+    (property "Voltage" "16V" (at 63.42 81.28 0) (do_not_autoplace)
       (effects (font (size 1.15 1.15)) (justify left) hide)
     )
@@
       (effects (font (size 1.15 1.15)) (justify left) hide)
     )
-    (property "Mouser" "80-C1206C105K5R" (at 58.42 88.9 0)
+    (property "Mouser" "80-C1206C105K4R" (at 58.42 88.9 0)
       (effects (font (size 1 1)) hide)
     )
@@
       (effects (font (size 1.15 1.15)) (justify left) hide)
     )
-    (property "Mouser" "80-C1206C104K5R" (at 172.72 88.9 0)
-      (effects (font (size 1 1)) hide)
-    )
+    (property "Mouser" "187-CL31B106KAHNFNE" (at 172.72 88.9 0)
+      (effects (font (size 1 1)) hide)
+    )

Commit message: Up
Parts:
- C301, C305, C307: symbol tronixio:CAPACITOR-1206-10N-20P-X7R -> tronixio:CAPACITOR-1206-10N-100V-5P-X7R; Mouser 80-C1206C103M5R -> 80-C1206C103J1R; Tolerance 20% -> 5%; Voltage 50V -> 100V
- C302, C303, C304: symbol tronixio:CAPACITOR-1206-1U-10P-X7R -> tronixio:CAPACITOR-1206-1U-16V-10P-X7R
- C306: symbol tronixio:CAPACITOR-1206-100N-10P-X7R -> tronixio:CAPACITOR-1206-100N-50V-5P-X7R; Mouser 187-CL31B106KAHNFNE -> 80-C1206C104J5R; Tolerance 10% -> 5%
- K301: Mouser 855-M20-999084 -> 855-M20-782084
Connections:
- net GND: now also S303.5; no longer S303.4
- net at R309.2, R312.2: now also S303.4; no longer S303.5
Other:
- moved on the sheet: C301, C306, C307, JP302, JP303, LED301, LED302, R303, R312, R314, R315, R317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

Commit message: Update Mini Kicad 8
Connections:
- net +3V3 renamed POWER-+3V3
- net +5V renamed POWER-+5V
- net GND renamed POWER-GND

Commit message: Update Mini
Other:
- moved on the sheet: JP302, JP303
