File: Kicad/mini/pic16bit.kicad_sch (KiCad schematic)
At the start: 12 parts, among them K101 PE-450-4X6X-BLACK

Commit message: Update Mini
Parts:
- H101, H102, H103, H104: MOUSER 534-9055 -> (none); Mouser (none) -> 534-9055
- JP101, JP102, JP103, JP104, JP105, JP106, JP107: MOUSER 855-M7582 -> (none); Mouser (none) -> 855-M7582
- K101: MOUSER 450-476 -> (none); Mouser (none) -> 450-476

Commit message: Update Kicad
Other:
- sheet HID ports: added PGC/URX/RB1; removed PGC/UTX/RB1
- sheet MCU ports: added PGC/URX/RB1; removed PGC/UTX/RB1
Changed lines of the file:
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@@
       (effects (font (size 1.27 1.27)) (justify right))
     )
-    (pin "PGD{slash}UTX{slash}RB0" input (at 124.46 104.14 0)
+    (pin "PGD{slash}UTX{slash}RB0" output (at 124.46 104.14 0)
       (effects (font (size 1.27 1.27)) (justify right))
     )
-    (pin "PGC{slash}UTX{slash}RB1" output (at 124.46 106.68 0)
+    (pin "PGC{slash}URX{slash}RB1" input (at 124.46 106.68 0)
       (effects (font (size 1.27 1.27)) (justify right))
     )
@@
       (effects (font (size 1.27 1.27)) (justify left))
     )
-    (pin "PGD{slash}UTX{slash}RB0" output (at 165.1 104.14 180)
+    (pin "PGC{slash}URX{slash}RB1" output (at 165.1 106.68 180)
       (effects (font (size 1.27 1.27)) (justify left))
     )
-    (pin "PGC{slash}UTX{slash}RB1" input (at 165.1 106.68 180)
+    (pin "PGD{slash}UTX{slash}RB0" input (at 165.1 104.14 180)
       (effects (font (size 1.27 1.27)) (justify left))
     )

Commit message: Update
Changed lines of the file:
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@@
-      (effects (font (size 1.27 1.27)) (justify right))
-    )
-    (pin "SCL" input (at 124.46 96.52 0)
       (effects (font (size 1.27 1.27)) (justify right))
     )
@@
       (effects (font (size 1.27 1.27)) (justify right))
     )
+    (pin "SCL" output (at 124.46 96.52 0)
+      (effects (font (size 1.27 1.27)) (justify right))
+    )

Commit message: Update
Other:
- title: Diagram -> Connections
