File: Kicad/mini/pic16bit.kicad_sch (KiCad schematic)
At the start: 12 parts, among them K101 PE-450-4X6X-BLACK

Commit message: Update
Changed lines of the file:
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@@
-      (effects (font (size 1.27 1.27)) (justify left))
-    )
-    (pin "SCL" input (at 165.1 96.52 180)
       (effects (font (size 1.27 1.27)) (justify left))
     )
@@
     )
     (pin "PGC{slash}URX{slash}RB1" bidirectional (at 165.1 106.68 180)
+      (effects (font (size 1.27 1.27)) (justify left))
+    )
+    (pin "SCL" bidirectional (at 165.1 96.52 180)
       (effects (font (size 1.27 1.27)) (justify left))
     )
@@
     )
     (path "/64edc06d-d6ae-4dac-9759-3f1fbed6457d/2259c208-8ca0-4ca4-9675-2e8cdca370a7"
-      (reference "JP205") (unit 1) (value "VCA") (footprint "tronixio:HARWIN-M20-999024x")
+      (reference "JP205") (unit 1) (value "VCAP") (footprint "tronixio:HARWIN-M20-999024x")
     )
     (path "/8cdf8b92-b881-481d-a85a-c0055e9a856b/decd714e-c32f-40e5-b629-c0d4257717ea"
@@
     )
     (path "/8cdf8b92-b881-481d-a85a-c0055e9a856b/2a18c81a-56c3-4e70-b384-8772ef4752eb"
-      (reference "U301") (unit 1) (value "CAT4002A") (footprint "tronixio:SOT-23-6")
+      (reference "U301") (unit 1) (value "CAT4002A") (footprint "tronixioZZZ:SC-70-6")
     )
     (path "/8cdf8b92-b881-481d-a85a-c0055e9a856b/ff1657d3-e3fc-4778-bbec-5be8aca2417b"
-      (reference "U302") (unit 1) (value "MCP2221A-ISL") (footprint "tronixio:SOIC-14")
+      (reference "U302") (unit 1) (value "MCP2221A") (footprint "tronixio:SOIC-14")
     )
   )

Commit message: Up
Other:
- title: Connections -> Root
