File: Kicad/mini/pic16bit-mcu.kicad_sch (KiCad schematic)
At the start: 31 parts, among them IC201 TLV1117-33, IC202 dsPIC33/PIC24F, K201 *Power & UART, K202 MCU 1, K203 MCU 1, K204 ICSP, K205 MCU 2, K206 MCU 2

Commit message: Update Mini
Parts:
- removed IC202: dsPIC33/PIC24F, tronixio:DIP-28-W762, symbol tronixio:MICROCHIP-PIC24FJxxGA002-ISP
- added IC202: MICROCHIP-PIC24FJ64GA102-ISP, tronixio:DIP-28-W762, symbol tronixio:MICROCHIP-PIC24FJ64GA102-ISP
- C201, C202, C203, C204, C205: footprint tronixio:CAPACITOR-1206 -> (none)
- C206: footprint tronixio:KEMET-C322 -> (none)
- D201, D202: value PMEG3030 -> (none); footprint tronixio:SOD-128 -> (none); symbol tronixio:PMEG3030 -> tronixio:NEXPERIA-PMEG3030; MOUSER 771-PMEG3030EP115 -> (none); Mouser (none) -> 771-PMEG3030EP115; Name (none) -> PMEG3030
- F201: value F050 -> (none); footprint tronixio:FUSE-1206 -> (none); MOUSER 652-MF-NSMF050-2 -> (none); Mouser (none) -> 652-MF-NSMF050-2; Name (none) -> 500mA
- IC201: symbol tronixio:TLV1117-33-SOT -> tronixio:TI-TLV1117-33-SOT; MOUSER 595-TLV1117-33CDC -> (none); Mouser (none) -> 595-TLV1117-33CDC; Name (none) -> TLV1117-33
- JP201: value *Power IN -> (none); MOUSER 855-M20-999024 -> (none); Mouser (none) -> 855-M20-999024
- JP202, JP203, JP205: MOUSER 855-M20-999024 -> (none); Mouser (none) -> 855-M20-999024
- JP204: MOUSER 855-M20-999024 -> (none); Mouser (none) -> 855-M20-999034
- K201: MOUSER 649-10118193-0001LF -> (none); Mouser (none) -> 649-10118193-0001LF
- K202, K205: MOUSER 855-M20-999144 -> (none); Mouser (none) -> 855-M20-999144
- K203: value MCU 1 -> (none); footprint tronixio:zzHARWIN-M20-782144x -> (none); MOUSER 855-M20-782144 -> (none); Mouser (none) -> 855-M20-782144
- K204: MOUSER 200-SSW10602TSRA -> (none); Mouser (none) -> 200-SSW10602TSRA
- K206: value MCU 2 -> (none); footprint tronixio:zzHARWIN-M20-782144x -> (none); MOUSER 855-M20-782144 -> (none); Mouser (none) -> 855-M20-782144
- LED201: MOUSER 604-APT3216LVBCD -> (none); Mouser (none) -> 604-APT3216LVBCD
- R201, R202, R203, R204, R205: footprint tronixio:RESISTOR-1206 -> (none)
- S201: value Reset -> (none); MOUSER 688-SKRPACE010 -> (none); Mouser (none) -> 688-SKRPACE010
- TP201, TP202: MOUSER 534-5006 -> (none); Mouser (none) -> 534-5006
Connections:
- net +3V3: now also IC202.13 (VDD), IC202.28 (VDD)
- net GND: now also IC202.27 (VSS), IC202.8 (VSS)
- net PGC/UTX/RB1: now also IC202.5 (RB1/PGC1)
- net PGD/UTX/RB0: now also IC202.4 (RB0/PGD1)
- net ~{MCLR}: now also IC202.1 (~{MCLR})
- net at JP205.1, K205.9 (Pin_9), K206.9 (Pin_9): now also IC202.20 (VCAP/VDDCORE)
- net at K202.10 (Pin_10), K203.10 (Pin_10): now also IC202.10 (RA3/CLKO)
- net at K202.11 (Pin_11), K203.11 (Pin_11): now also IC202.11 (RB4)
- net at K202.12 (Pin_12), K203.12 (Pin_12): now also IC202.12 (RA4)
- net at K202.14 (Pin_14), K203.14 (Pin_14): now also IC202.14 (RB5)
- net at K202.2 (Pin_2), K203.2 (Pin_2): now also IC202.2 (RA0)
- net at K202.3 (Pin_3), K203.3 (Pin_3): now also IC202.3 (RA1)
- net at K202.6 (Pin_6), K203.6 (Pin_6): now also IC202.6 (RB2)
- net at K202.7 (Pin_7), K203.7 (Pin_7): now also IC202.7 (RB3)
- net at K202.9 (Pin_9), K203.9 (Pin_9): now also IC202.9 (RA2/CLKI)
- net at JP204.2, K205.10 (Pin_10), K206.10 (Pin_10): now also IC202.19 (DISVREG)
- net at JP202.2, K205.12 (Pin_12), K206.12 (Pin_12): now also IC202.17 (RB8)
- net at K205.14 (Pin_14), K206.14 (Pin_14): now also IC202.15 (RB6)
- net at K205.13 (Pin_13), K206.13 (Pin_13): now also IC202.16 (RB7)
- net at JP203.2, K205.11 (Pin_11), K206.11 (Pin_11): now also IC202.18 (RB9)
- net at K205.8 (Pin_8), K206.8 (Pin_8): now also IC202.21 (RB10)
- net at K205.7 (Pin_7), K206.7 (Pin_7): now also IC202.22 (RB11)
- net at K205.6 (Pin_6), K206.6 (Pin_6): now also IC202.23 (RB12)
- net at K205.5 (Pin_5), K206.5 (Pin_5): now also IC202.24 (RB13)
- net at K205.4 (Pin_4), K206.4 (Pin_4): now also IC202.25 (RB14)
- net at K205.3 (Pin_3), K206.3 (Pin_3): now also IC202.26 (RB15)

Commit message: Update
Parts:
- C201, C202, C203, C204, C205: footprint (none) -> tronixio:CAPACITOR-1206
- C206: footprint (none) -> tronixio:KEMET-C322
- D201, D202: value (none) -> PMEG3030; footprint (none) -> tronixio:SOD-128
- F201: value (none) -> F050; footprint (none) -> tronixio:FUSE-1206
- JP201: value (none) -> *Power IN
- K203: value (none) -> MCU 1; footprint (none) -> tronixio:zzHARWIN-M20-782144x
- K206: value (none) -> MCU 2; footprint (none) -> tronixio:zzHARWIN-M20-782144x
- R201, R202, R203, R204, R205: footprint (none) -> tronixio:RESISTOR-1206
- S201: value (none) -> Reset
Changed lines of the file:
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@@
       (effects (font (size 1.15 1.15)))
     )
-    (property "Value" "" (id 1) (at 68.58 177.8 0)
-      (effects (font (size 1 1)) hide)
-    )
-    (property "Footprint" "" (id 2) (at 68.58 167.64 0)
+    (property "Value" "PMEG3030" (id 1) (at 68.58 177.8 0)
+      (effects (font (size 1 1)) hide)
+    )
+    (property "Footprint" "tronixio:SOD-128" (id 2) (at 68.58 167.64 0)
       (effects (font (size 1 1)) hide)
     )
@@
       (effects (font (size 1.15 1.15)))
     )
-    (property "Value" "" (id 1) (at 68.58 137.16 0)
-      (effects (font (size 1.15 1.15)))
-    )
-    (property "Footprint" "" (id 2) (at 68.58 139.7 0)
+    (property "Value" "MCU 1" (id 1) (at 68.58 137.16 0)
+      (effects (font (size 1.15 1.15)))
+    )
+    (property "Footprint" "tronixio:zzHARWIN-M20-782144x" (id 2) (at 68.58 139.7 0)
       (effects (font (size 1 1)) hide)
     )
@@
       (effects (font (size 1.15 1.15)) (justify right))
     )
-    (property "Footprint" "" (id 2) (at 81.28 190.5 0)
+    (property "Footprint" "tronixio:CAPACITOR-1206" (id 2) (at 81.28 190.5 0)
       (effects (font (size 1 1)) hide)
     )
@@
       (effects (font (size 1.15 1.15)) (justify left))
     )
-    (property "Footprint" "" (id 2) (at 167.64 106.68 0)
+    (property "Footprint" "tronixio:CAPACITOR-1206" (id 2) (at 167.64 106.68 0)
       (effects (font (size 1 1)) hide)
     )
@@
       (effects (font (size 1.15 1.15)) (justify left))
     )
-    (property "Value" "" (id 1) (at 57.785 185.42 0)
+    (property "Value" "*Power IN" (id 1) (at 57.785 185.42 0)
       (effects (font (size 1.15 1.15)) (justify left))
     )
@@
       (effects (font (size 1.15 1.15)) (justify left))
     )
-    (property "Footprint" "" (id 2) (at 193.04 157.48 0)
+    (property "Footprint" "tronixio:KEMET-C322" (id 2) (at 193.04 157.48 0)
       (effects (font (size 1 1)) hide)
     )
@@
       (effects (font (size 1.15 1.15)) (justify left))
     )
-    (property "Footprint" "" (id 2) (at 109.22 190.5 0)
+    (property "Footprint" "tronixio:CAPACITOR-1206" (id 2) (at 109.22 190.5 0)
       (effects (font (size 1 1)) hide)
     )
@@
       (effects (font (size 1.15 1.15)))
     )
-    (property "Footprint" "" (id 2) (at 78.74 38.1 0)
+    (property "Footprint" "tronixio:RESISTOR-1206" (id 2) (at 78.74 38.1 0)
       (effects (font (size 1 1)) hide)
     )
@@
       (effects (font (size 1.15 1.15)) (justify right))
     )
-    (property "Footprint" "" (id 2) (at 121.92 106.68 0)
+    (property "Footprint" "tronixio:CAPACITOR-1206" (id 2) (at 121.92 106.68 0)
       (effects (font (size 1 1)) hide)
     )
@@
       (effects (font (size 1.15 1.15)))
     )
-    (property "Value" "" (id 1) (at 68.58 167.64 0)
-      (effects (font (size 1 1)) hide)
-    )
-    (property "Footprint" "" (id 2) (at 68.58 162.56 0)
+    (property "Value" "PMEG3030" (id 1) (at 68.58 167.64 0)
+      (effects (font (size 1 1)) hide)
+    )
+    (property "Footprint" "tronixio:SOD-128" (id 2) (at 68.58 162.56 0)
       (effects (font (size 1 1)) hide)
     )
@@
       (effects (font (size 1.15 1.15)))
     )
-    (property "Footprint" "" (id 2) (at 187.96 48.26 0)
+    (property "Footprint" "tronixio:RESISTOR-1206" (id 2) (at 187.96 48.26 0)
       (effects (font (size 1 1)) hide)
     )
@@
       (effects (font (size 1.15 1.15)) (justify left))
     )
-    (property "Footprint" "" (id 2) (at 83.82 53.34 0)
+    (property "Footprint" "tronixio:CAPACITOR-1206" (id 2) (at 83.82 53.34 0)
       (effects (font (size 1 1)) hide)
     )
@@
       (effects (font (size 1.15 1.15)))
     )
-    (property "Footprint" "" (id 2) (at 177.8 48.26 0)
+    (property "Footprint" "tronixio:RESISTOR-1206" (id 2) (at 177.8 48.26 0)
       (effects (font (size 1 1)) hide)
     )
@@
       (effects (font (size 1.15 1.15)))
     )
-    (property "Value" "" (id 1) (at 58.42 167.64 0)
-      (effects (font (size 1 1)) hide)
-    )
-    (property "Footprint" "" (id 2) (at 58.42 177.8 0)
+    (property "Value" "F050" (id 1) (at 58.42 167.64 0)
+      (effects (font (size 1 1)) hide)
+    )
+    (property "Footprint" "tronixio:FUSE-1206" (id 2) (at 58.42 177.8 0)
       (effects (font (size 1 1)) hide)
     )
@@
       (effects (font (size 1.15 1.15)))
     )
-    (property "Footprint" "" (id 2) (at 76.2 45.72 0)
+    (property "Footprint" "tronixio:RESISTOR-1206" (id 2) (at 76.2 45.72 0)
       (effects (font (size 1 1)) hide)
     )
@@
       (effects (font (size 1.15 1.15)))
     )
-    (property "Footprint" "" (id 2) (at 127 182.88 0)
+    (property "Footprint" "tronixio:RESISTOR-1206" (id 2) (at 127 182.88 0)
       (effects (font (size 1 1)) hide)
     )
@@
       (effects (font (size 1.15 1.15)) (justify left))
     )
-    (property "Value" "" (id 1) (at 74.295 46.99 90)
+    (property "Value" "Reset" (id 1) (at 74.295 46.99 90)
       (effects (font (size 1.15 1.15)) (justify left))
     )
@@
       (effects (font (size 1.15 1.15)))
     )
-    (property "Value" "" (id 1) (at 220.98 137.16 0)
-      (effects (font (size 1.15 1.15)))
-    )
-    (property "Footprint" "" (id 2) (at 220.98 139.7 0)
-      (effects (font (size 1 1)) hide)
-    )
+    (property "Value" "MCU 2" (id 1) (at 220.98 137.16 0)
+      (effects (font (size 1.15 1.15)))
+    )
+    (property "Footprint" "tronixio:zzHARWIN-M20-782144x" (id 2) (at 220.98 139.7 0)
+      (effects (font (size 1 1)) hide)
+    )

Commit message: Update Kicad
Parts:
- added TP203: KEYSTONE-2000-3, tronixio:KEYSTONE-2000-3, symbol tronixio:KEYSTONE-2000-3
- IC202: value MICROCHIP-PIC24FJ64GA102-ISP -> (none); footprint tronixio:DIP-28-W762 -> (none)
Connections:
- net GND: now also TP203.1
Other:
- moved on the sheet: C203, LED201, R203, TP201, TP202

Commit message: Update Kicad
Parts:
- IC202: value (none) -> MICROCHIP-PIC24FJ64GA102-ISP; footprint (none) -> tronixio:DIP-28-W762-SOCKET
Connections:
- net PGC/UTX/RB1: no longer IC202.5 (RB1/PGC1), K202.5 (Pin_5), K203.5 (Pin_5)
- new net PGC/URX/RB1: IC202.5 (RB1/PGC1), K202.5 (Pin_5), K203.5 (Pin_5)
Changed lines of the file:
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@@
     (effects (font (size 1.15 1.15)) (justify left))
   )
-  (hierarchical_label "PGD{slash}UTX{slash}RB0" (shape input) (at 71.12 144.78 180)
+  (hierarchical_label "PGD{slash}UTX{slash}RB0" (shape output) (at 71.12 144.78 180)
     (effects (font (size 1.2 1.2)) (justify right))
   )
-  (hierarchical_label "PGC{slash}UTX{slash}RB1" (shape output) (at 71.12 147.32 180)
+  (hierarchical_label "PGC{slash}URX{slash}RB1" (shape input) (at 71.12 147.32 180)
     (effects (font (size 1.2 1.2)) (justify right))
   )
@@
       (effects (font (size 1.15 1.15)) (justify left))
     )
-    (property "Value" "" (id 1) (at 144.78 92.71 0)
+    (property "Value" "MICROCHIP-PIC24FJ64GA102-ISP" (id 1) (at 144.78 92.71 0)
       (effects (font (size 1.15 1.15)) hide)
     )
-    (property "Footprint" "" (id 2) (at 144.78 95.25 0)
-      (effects (font (size 1 1)) hide)
-    )
+    (property "Footprint" "tronixio:DIP-28-W762-SOCKET" (id 2) (at 144.78 95.25 0)
+      (effects (font (size 1 1)) hide)
+    )

Commit message: Update
Connections:
- net PGC/UTX/RB1 is gone; now on net PGC/URX/RB1: K204.2
Changed lines of the file:
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@@
     )
   )
-  (global_label "PGC{slash}UTX{slash}RB1" (shape input) (at 142.24 123.19 180) (fields_autoplaced)
+  (global_label "PGC{slash}URX{slash}RB1" (shape input) (at 142.24 123.19 180) (fields_autoplaced)
     (effects (font (size 1.2 1.2)) (justify right))
-    (property "Intersheet References" "${INTERSHEET_REFS}" (id 0) (at 126.8086 123.115 0)
+    (property "Intersheet References" "${INTERSHEET_REFS}" (id 0) (at 126.5229 123.115 0)
       (effects (font (size 1.2 1.2)) (justify right) hide)
     )
@@
     )
   )
-  (hierarchical_label "SCL" (shape input) (at 180.34 40.64 0)
+  (hierarchical_label "SCL" (shape output) (at 180.34 40.64 0)
     (effects (font (size 1.15 1.15)) (justify left))
   )

Commit message: Update
Parts:
- K203, K206: footprint tronixio:zzHARWIN-M20-782144x -> tronixio:HARWIN-M20-782144x
Other:
- moved on the sheet: F201
Changed lines of the file:
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@@
     (stroke (width 0) (type solid) (color 0 0 0 0))
   )
-  (wire (pts (xy 182.88 182.88) (xy 182.88 190.5))
+  (wire (pts (xy 177.8 182.88) (xy 177.8 190.5))
     (stroke (width 0) (type solid) (color 0 0 0 0))
   )
@@
     (stroke (width 0) (type solid) (color 0 0 0 0))
   )
-  (wire (pts (xy 63.5 170.18) (xy 66.04 170.18))
+  (wire (pts (xy 60.96 170.18) (xy 66.04 170.18))
     (stroke (width 0) (type default) (color 0 0 0 0))
   )
@@
     (stroke (width 0) (type solid) (color 0 0 0 0))
   )
-  (wire (pts (xy 43.18 170.18) (xy 53.34 170.18))
+  (wire (pts (xy 43.18 170.18) (xy 50.8 170.18))
     (stroke (width 0) (type default) (color 0 0 0 0))
   )
@@
   )
   (text "IC202: Check the pinout for the desired MCU family"
-    (at 185.42 173.99 0)
+    (at 181.61 173.99 0)
     (effects (font (size 1.27 1.27)) (justify left bottom))
   )
@@
     (effects (font (size 1.15 1.15)) (justify right bottom))
   )
-  (text "Power & UART OR Header Power IN" (at 185.42 171.45 0)
+  (text "Power & UART OR Header Power IN" (at 181.61 171.45 0)
     (effects (font (size 1.27 1.27)) (justify left bottom))
   )
@@
     (effects (font (size 1.15 1.15)) (justify right bottom))
   )
-  (global_label "~{MCLR}" (shape input) (at 142.24 113.03 180) (fields_autoplaced)
+  (global_label "~{MCLR}" (shape output) (at 142.24 113.03 180) (fields_autoplaced)
     (effects (font (size 1.2 1.2)) (justify right))
-    (property "Intersheet References" "${INTERSHEET_REFS}" (id 0) (at 135.2171 112.955 0)
+    (property "Intersheet References" "${INTERSHEET_REFS}" (id 0) (at 135.0371 112.955 0)
       (effects (font (size 1.2 1.2)) (justify right) hide)
     )
@@
     )
   )
-  (global_label "PGC{slash}URX{slash}RB1" (shape input) (at 142.24 123.19 180) (fields_autoplaced)
+  (global_label "PGC{slash}URX{slash}RB1" (shape bidirectional) (at 142.24 123.19 180) (fields_autoplaced)
     (effects (font (size 1.2 1.2)) (justify right))
     (property "Intersheet References" "${INTERSHEET_REFS}" (id 0) (at 126.5229 123.115 0)
@@
     )
   )
-  (global_label "PGD{slash}UTX{slash}RB0" (shape input) (at 142.24 120.65 180) (fields_autoplaced)
+  (global_label "PGD{slash}UTX{slash}RB0" (shape bidirectional) (at 142.24 120.65 180) (fields_autoplaced)
     (effects (font (size 1.2 1.2)) (justify right))
     (property "Intersheet References" "${INTERSHEET_REFS}" (id 0) (at 126.8086 120.575 0)
@@
     )
   )
-  (hierarchical_label "SCL" (shape output) (at 180.34 40.64 0)
+  (hierarchical_label "SCL" (shape bidirectional) (at 180.34 40.64 0)
     (effects (font (size 1.15 1.15)) (justify left))
   )
-  (hierarchical_label "PGD{slash}UTX{slash}RB0" (shape output) (at 71.12 144.78 180)
+  (hierarchical_label "PGD{slash}UTX{slash}RB0" (shape bidirectional) (at 71.12 144.78 180)
     (effects (font (size 1.2 1.2)) (justify right))
   )
-  (hierarchical_label "PGC{slash}URX{slash}RB1" (shape input) (at 71.12 147.32 180)
+  (hierarchical_label "PGC{slash}URX{slash}RB1" (shape bidirectional) (at 71.12 147.32 180)
     (effects (font (size 1.2 1.2)) (justify right))
   )
@@
     (pin "1")
   )
-  (symbol (lib_id "tronixio:KEYSTONE-5006") (at 137.16 162.56 0) (unit 1)
+  (symbol (lib_name "KEYSTONE-5006_1") (lib_id "tronixio:KEYSTONE-5006") (at 137.16 162.56 0) (unit 1)
     (in_bom yes) (on_board yes)
     (property "Reference" "TP201" (id 0) (at 137.16 157.48 0)
@@
       (effects (font (size 1.15 1.15)))
     )
-    (property "Footprint" "tronixio:zzHARWIN-M20-782144x" (id 2) (at 68.58 139.7 0)
+    (property "Footprint" "tronixio:HARWIN-M20-782144x" (id 2) (at 68.58 139.7 0)
       (effects (font (size 1 1)) hide)
     )
@@
     (pin "2")
   )
-  (symbol (lib_id "tronixio:PWR_FLAG") (at 182.88 190.5 180) (unit 1)
-    (in_bom yes) (on_board yes) (fields_autoplaced)
-    (property "Reference" "#FLG0201" (id 0) (at 182.88 188.595 0)
+  (symbol (lib_id "tronixio:PWR_FLAG") (at 177.8 190.5 180) (unit 1)
+    (in_bom yes) (on_board yes) (fields_autoplaced)
+    (property "Reference" "#FLG0201" (id 0) (at 177.8 188.595 0)
       (effects (font (size 1.27 1.27)) hide)
     )
-    (property "Value" "PWR_FLAG" (id 1) (at 182.88 186.69 0)
+    (property "Value" "PWR_FLAG" (id 1) (at 177.8 186.69 0)
       (effects (font (size 1.27 1.27)) hide)
     )
-    (property "Footprint" "" (id 2) (at 182.88 190.5 0)
+    (property "Footprint" "" (id 2) (at 177.8 190.5 0)
       (effects (font (size 1.27 1.27)) hide)
     )
-    (property "Datasheet" "~" (id 3) (at 182.88 190.5 0)
+    (property "Datasheet" "~" (id 3) (at 177.8 190.5 0)
       (effects (font (size 1.27 1.27)) hide)
     )
@@
     (pin "2")
   )
-  (symbol (lib_id "tronixio:BOURNS-FUSE-MF-NSMF050") (at 58.42 170.18 0) (unit 1)
-    (in_bom yes) (on_board yes)
-    (property "Reference" "F201" (id 0) (at 58.42 165.1 0)
-      (effects (font (size 1.15 1.15)))
-    )
-    (property "Value" "F050" (id 1) (at 58.42 167.64 0)
-      (effects (font (size 1 1)) hide)
-    )
-    (property "Footprint" "tronixio:FUSE-1206" (id 2) (at 58.42 177.8 0)
-      (effects (font (size 1 1)) hide)
-    )
-    (property "Datasheet" "https://www.bourns.com/pdfs/mfnsmf.pdf" (id 3) (at 58.42 180.34 0)
-      (effects (font (size 1 1)) hide)
-    )
-    (property "Name" "500mA" (id 4) (at 58.42 167.64 0)
-      (effects (font (size 1.15 1.15)))
-    )
-    (property "Mouser" "652-MF-NSMF050-2" (id 5) (at 58.42 182.88 0)
+  (symbol (lib_id "tronixio:BOURNS-FUSE-MF-NSMF050") (at 55.88 170.18 0) (unit 1)
+    (in_bom yes) (on_board yes)
+    (property "Reference" "F201" (id 0) (at 55.88 165.1 0)
+      (effects (font (size 1.15 1.15)))
+    )
+    (property "Value" "F050" (id 1) (at 55.88 167.64 0)
+      (effects (font (size 1 1)) hide)
+    )
+    (property "Footprint" "tronixio:FUSE-1206" (id 2) (at 55.88 177.8 0)
+      (effects (font (size 1 1)) hide)
+    )
+    (property "Datasheet" "https://www.bourns.com/pdfs/mfnsmf.pdf" (id 3) (at 55.88 180.34 0)
+      (effects (font (size 1 1)) hide)
+    )
+    (property "Name" "500mA" (id 4) (at 55.88 167.64 0)
+      (effects (font (size 1.15 1.15)))
+    )
+    (property "Mouser" "652-MF-NSMF050-2" (id 5) (at 55.88 182.88 0)
       (effects (font (size 1 1)) hide)
     )
@@
   (symbol (lib_id "tronixio:LED-1206-BLUE") (at 121.92 180.34 270) (mirror x) (unit 1)
     (in_bom yes) (on_board yes)
-    (property "Reference" "LED201" (id 0) (at 122.555 177.8 90)
-      (effects (font (size 1.15 1.15)) (justify left))
-    )
-    (property "Value" "Power" (id 1) (at 122.555 182.88 90)
+    (property "Reference" "LED201" (id 0) (at 122.555 177.165 90)
+      (effects (font (size 1.15 1.15)) (justify left))
+    )
+    (property "Value" "Power" (id 1) (at 122.555 183.515 90)
       (effects (font (size 1.15 1.15)) (justify left))
     )
@@
     (pin "1")
   )
-  (symbol (lib_id "tronixio:POWER-+5V") (at 182.88 182.88 0) (unit 1)
-    (in_bom yes) (on_board yes) (fields_autoplaced)
-    (property "Reference" "#PWR0107" (id 0) (at 182.88 193.04 0)
-      (effects (font (size 1 1)) hide)
-    )
-    (property "Value" "POWER-+5V" (id 1) (at 182.88 195.58 0)
-      (effects (font (size 1 1)) hide)
-    )
-    (property "Footprint" "" (id 2) (at 182.88 182.88 0)
-      (effects (font (size 1 1)) hide)
-    )
-    (property "Datasheet" "" (id 3) (at 182.88 182.88 0)
-      (effects (font (size 1 1)) hide)
-    )
-    (property "Name" "+5V" (id 4) (at 182.88 177.8 0)
+  (symbol (lib_id "tronixio:POWER-+5V") (at 177.8 182.88 0) (unit 1)
+    (in_bom yes) (on_board yes) (fields_autoplaced)
+    (property "Reference" "#PWR0107" (id 0) (at 177.8 193.04 0)
+      (effects (font (size 1 1)) hide)
+    )
+    (property "Value" "POWER-+5V" (id 1) (at 177.8 195.58 0)
+      (effects (font (size 1 1)) hide)
+    )
+    (property "Footprint" "" (id 2) (at 177.8 182.88 0)
+      (effects (font (size 1 1)) hide)
+    )
+    (property "Datasheet" "" (id 3) (at 177.8 182.88 0)
+      (effects (font (size 1 1)) hide)
+    )
+    (property "Name" "+5V" (id 4) (at 177.8 177.8 0)
       (effects (font (size 1.15 1.15)))
     )
@@
       (effects (font (size 1.15 1.15)))
     )
-    (property "Footprint" "tronixio:zzHARWIN-M20-782144x" (id 2) (at 220.98 139.7 0)
-      (effects (font (size 1 1)) hide)
-    )
+    (property "Footprint" "tronixio:HARWIN-M20-782144x" (id 2) (at 220.98 139.7 0)
+      (effects (font (size 1 1)) hide)
+    )

Commit message: Update
Parts:
- U202: renamed from IC202; footprint tronixio:DIP-28-W762-SOCKET -> tronixio:DIP-28-W762; Name PIC24F/dsPIC33 -> PIC24FJ64GA102-ISP
- renumbered IC201 to U201
Changed lines of the file:
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@@
   (symbol (lib_id "tronixio:TI-TLV1117-33-SOT") (at 93.98 170.18 0) (unit 1)
     (in_bom yes) (on_board yes)
-    (property "Reference" "IC201" (id 0) (at 93.98 163.83 0)
+    (property "Reference" "U201" (id 0) (at 93.98 163.83 0)
       (effects (font (size 1.15 1.15)))
     )
@@
   (symbol (lib_id "tronixio:MICROCHIP-PIC24FJ64GA102-ISP") (at 144.78 72.39 0) (unit 1)
     (in_bom yes) (on_board yes)
-    (property "Reference" "IC202" (id 0) (at 132.08 52.07 0)
+    (property "Reference" "U202" (id 0) (at 132.08 52.07 0)
       (effects (font (size 1.15 1.15)) (justify left))
     )
@@
       (effects (font (size 1.15 1.15)) hide)
     )
-    (property "Footprint" "tronixio:DIP-28-W762-SOCKET" (id 2) (at 144.78 95.25 0)
+    (property "Footprint" "tronixio:DIP-28-W762" (id 2) (at 144.78 95.25 0)
       (effects (font (size 1 1)) hide)
     )
@@
       (effects (font (size 1 1)) hide)
     )
-    (property "Name" "PIC24F/dsPIC33" (id 4) (at 157.48 52.07 0)
+    (property "Name" "PIC24FJ64GA102-ISP" (id 4) (at 157.48 52.07 0)
       (effects (font (size 1.15 1.15)) (justify right))
     )
