File: Kicad/mini/pic16bit-mcu.kicad_sch (KiCad schematic)
At the start: 32 parts, among them K201 *Power & UART, K202 MCU 1, K203 MCU 1, K204 ICSP, K205 MCU 2, K206 MCU 2, U201 TLV1117-33, U202 MICROCHIP-PIC24FJ64GA102-ISP

Commit message: Update
Parts:
- C201, C203: footprint tronixio:CAPACITOR-1206 -> tronixio:CAPACITOR-0805; symbol tronixio:C-0805 -> tronixio:CAPACITOR-0805-10U; Mouser (none) -> 80-C0805C106M3P; Name (none) -> CAPACITOR-0805-10U; Tolerance (none) -> 20%; Voltage (none) -> 25V
- C202, C204, C205: footprint tronixio:CAPACITOR-1206 -> tronixio:CAPACITOR-0805; symbol tronixio:C-0805 -> tronixio:CAPACITOR-0805-100N; Mouser (none) -> 80-C0805C104M5R; Name (none) -> CAPACITOR-0805-100N; Tolerance (none) -> 20%; Voltage (none) -> 50V
- C206: symbol tronixio:C-0805 -> tronixio:KEMET-C322-10U-508; Mouser (none) -> 80-C322C106K3R; Name (none) -> KEMET-C32210U-508; Tolerance (none) -> 10%
- D201, D202: Name PMEG3030 -> NEXPERIA-PMEG3030
- F201: value F050 -> 500mA; footprint tronixio:FUSE-1206 -> tronixio:FUSE-0805; Name 500mA -> BOURNS-FUSE-MF-NSMF050
- JP201: value *Power IN -> Power IN; Name (none) -> HARWIN-254-M-1X02-JUMPER-VERTICAL
- JP202, JP203: Name (none) -> HARWIN-254-M-1X02-JUMPER-VERTICAL
- JP204: Name (none) -> HARWIN-254-M-1X03-VERTICAL
- JP205: value VCAP -> VCA; Name (none) -> HARWIN-254-M-1X02-JUMPER-VERTICAL
- K201: Name (none) -> FCI-USB-TYPE-B-MICRO-THT
- K202, K205: Name (none) -> HARWIN-254-M-1X14-VERTICAL
- K203, K206: Name (none) -> HARWIN-254-F-1X14-VERTICAL
- K204: Name ICSP -> MICROCHIP-ICSP-F-1X06
- LED201: footprint tronixio:LED-1206 -> tronixio:LED-0805; symbol tronixio:LED-1206-BLUE -> tronixio:KINGBRIGHT-LED-0805-BLUE; Mouser 604-APT3216LVBCD -> 604-APT2012LVBCD; Name (none) -> KINGBRIGHT-LED-0805-BLUE
- R201: footprint tronixio:RESISTOR-1206 -> tronixio:RESISTOR-0805; symbol tronixio:R-0805 -> tronixio:RESISTOR-0805-10K; Mouser (none) -> 660-RK73B2ATTDD103J; Name (none) -> RESISTOR-0805-10K; Tolerance (none) -> 5%
- R202: footprint tronixio:RESISTOR-1206 -> tronixio:RESISTOR-0805; symbol tronixio:R-0805 -> tronixio:RESISTOR-0805-1K; Mouser (none) -> 660-RK73B2ATTDD102J; Name (none) -> RESISTOR-0805-1K; Tolerance (none) -> 5%
- R203, R204, R205: footprint tronixio:RESISTOR-1206 -> tronixio:RESISTOR-0805; symbol tronixio:R-0805 -> tronixio:RESISTOR-0805-4K7; Mouser (none) -> 660-RK73B2ATTDD472J; Name (none) -> RESISTOR-0805-4K7; Tolerance (none) -> 5%
- S201: Name (none) -> ALPS-SKRPAC
- TP201, TP202: Name (none) -> KEYSTONE-5006
- TP203: Name (none) -> KEYSTONE-2000-3
- U201: symbol tronixio:TI-TLV1117-33-SOT -> tronixio:TI-TLV1117-33-SOT-223; Name TLV1117-33 -> TI-TLV1117-33-SOT-223
- U202: value MICROCHIP-PIC24FJ64GA102-ISP -> PIC24/dsPIC32; footprint tronixio:DIP-28-W762 -> tronixio:DIP-28-W762-SOCKET; Name PIC24FJ64GA102-ISP -> MICROCHIP-PIC24FJ64GA102-ISP
