File: Kicad/mini/pic16bit-mcu.kicad_sch (KiCad schematic)
At the start: 32 parts, among them K201 *Power & UART, K202 MCU 1, K203 MCU 1, K204 ICSP, K205 MCU 2, K206 MCU 2, U201 TLV1117-33, U202 PIC24/dsPIC32

Commit message: Update
Parts:
- C201, C203: footprint tronixio:CAPACITOR-0805 -> tronixio:CAPACITOR-1206; symbol tronixio:CAPACITOR-0805-10U -> tronixio:CAPACITOR-1206-10U; Mouser 80-C0805C106M3P -> 80-C1206C106M3R; Name CAPACITOR-0805-10U -> CAPACITOR-1206-10U
- C202, C204, C205: footprint tronixio:CAPACITOR-0805 -> tronixio:CAPACITOR-1206; symbol tronixio:CAPACITOR-0805-100N -> tronixio:CAPACITOR-1206-100N; Mouser 80-C0805C104M5R -> 80-C1206C104M5R; Name CAPACITOR-0805-100N -> CAPACITOR-1206-100N
- F201: footprint tronixio:FUSE-0805 -> tronixio:FUSE-1206
- LED201: footprint tronixio:LED-0805 -> tronixio:LED-1206; symbol tronixio:KINGBRIGHT-LED-0805-BLUE -> tronixio:KINGBRIGHT-LED-1206-BLUE; Mouser 604-APT2012LVBCD -> 604-APT3216LVBCD; Name KINGBRIGHT-LED-0805-BLUE -> KINGBRIGHT-LED-1206-BLUE
- R201: footprint tronixio:RESISTOR-0805 -> tronixio:RESISTOR-1206; symbol tronixio:RESISTOR-0805-10K -> tronixio:RESISTOR-1206-10K; Mouser 660-RK73B2ATTDD103J -> 660-RK73B2BTTDD103J; Name RESISTOR-0805-10K -> RESISTOR-1206-10K
- R202: footprint tronixio:RESISTOR-0805 -> tronixio:RESISTOR-1206; symbol tronixio:RESISTOR-0805-1K -> tronixio:RESISTOR-1206-1K; Mouser 660-RK73B2ATTDD102J -> 660-RK73B2BTTDD102J; Name RESISTOR-0805-1K -> RESISTOR-1206-1K
- R203, R204, R205: footprint tronixio:RESISTOR-0805 -> tronixio:RESISTOR-1206; symbol tronixio:RESISTOR-0805-4K7 -> tronixio:RESISTOR-1206-4K7; Mouser 660-RK73B2ATTDD472J -> 660-RK73B2BTTDD472J; Name RESISTOR-0805-4K7 -> RESISTOR-1206-4K7
Other:
- note added: "U202: Check the pinout for the desired MCU family"
- note removed: "IC202: Check the pinout for the desired MCU family"

Commit message: Update
Parts:
- C201, C202, C203, C204, C205: footprint tronixio:CAPACITOR-1206 -> tronixio:CAPACITOR-SMD-1206
- F201: footprint tronixio:FUSE-1206 -> tronixio:FUSE-SMD-1206
- LED201: footprint tronixio:LED-1206 -> tronixio:LED-SMD-1206
- R201, R202, R203, R204, R205: footprint tronixio:RESISTOR-1206 -> tronixio:RESISTOR-SMD-1206
- U202: footprint tronixio:DIP-28-W762-SOCKET -> tronixio:DIP-28-W762
Changed lines of the file:
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@@
       (effects (font (size 1.15 1.15)) (justify right))
     )
-    (property "Footprint" "tronixio:CAPACITOR-1206" (id 2) (at 81.28 193.04 0)
+    (property "Footprint" "tronixio:CAPACITOR-SMD-1206" (id 2) (at 81.28 193.04 0)
       (effects (font (size 1 1)) hide)
     )
@@
     (pin "1")
   )
-  (symbol (lib_id "tronixio:CAPACITOR-1206-100N") (at 167.64 96.52 0) (unit 1)
+  (symbol (lib_name "CAPACITOR-1206-100N_1") (lib_id "tronixio:CAPACITOR-1206-100N") (at 167.64 96.52 0) (unit 1)
     (in_bom yes) (on_board yes)
     (property "Reference" "C205" (id 0) (at 168.275 93.98 0)
@@
       (effects (font (size 1.15 1.15)) (justify left))
     )
-    (property "Footprint" "tronixio:CAPACITOR-1206" (id 2) (at 167.64 109.22 0)
+    (property "Footprint" "tronixio:CAPACITOR-SMD-1206" (id 2) (at 167.64 109.22 0)
       (effects (font (size 1 1)) hide)
     )
@@
     )
     (property "Footprint" "" (id 2) (at 177.8 190.5 0)
-      (effects (font (size 1.27 1.27)) hide)
-    )
-    (property "Datasheet" "~" (id 3) (at 177.8 190.5 0)
-      (effects (font (size 1.27 1.27)) hide)
+      (effects (font (size 1 1)) hide)
+    )
+    (property "Datasheet" "" (id 3) (at 177.8 190.5 0)
+      (effects (font (size 1 1)) hide)
     )
     (pin "1")
@@
     (pin "2")
   )
-  (symbol (lib_id "tronixio:CAPACITOR-1206-10U") (at 106.68 180.34 0) (unit 1)
+  (symbol (lib_name "CAPACITOR-1206-10U_1") (lib_id "tronixio:CAPACITOR-1206-10U") (at 106.68 180.34 0) (unit 1)
     (in_bom yes) (on_board yes)
     (property "Reference" "C203" (id 0) (at 107.315 177.8 0)
@@
       (effects (font (size 1.15 1.15)) (justify left))
     )
-    (property "Footprint" "tronixio:CAPACITOR-1206" (id 2) (at 106.68 193.04 0)
+    (property "Footprint" "tronixio:CAPACITOR-SMD-1206" (id 2) (at 106.68 193.04 0)
       (effects (font (size 1 1)) hide)
     )
@@
       (effects (font (size 1.15 1.15)))
     )
-    (property "Footprint" "tronixio:RESISTOR-1206" (id 2) (at 76.2 38.1 0)
-      (effects (font (size 1 1)) hide)
-    )
-    (property "Datasheet" "https://www.koaspeer.com/pdfs/RK73B.pdf" (id 3) (at 73.66 38.1 0)
+    (property "Footprint" "tronixio:RESISTOR-SMD-1206" (id 2) (at 76.2 38.1 0)
+      (effects (font (size 1 1)) hide)
+    )
+    (property "Datasheet" "https://www.koaspeer.com/products/resistors/general-purpose/rk73b/" (id 3) (at 73.66 38.1 0)
       (effects (font (size 1 1)) hide)
     )
@@
       (effects (font (size 1.15 1.15)) (justify right))
     )
-    (property "Footprint" "tronixio:CAPACITOR-1206" (id 2) (at 121.92 109.22 0)
+    (property "Footprint" "tronixio:CAPACITOR-SMD-1206" (id 2) (at 121.92 109.22 0)
       (effects (font (size 1 1)) hide)
     )
@@
     (pin "2")
   )
-  (symbol (lib_id "tronixio:RESISTOR-1206-4K7") (at 187.96 35.56 0) (unit 1)
+  (symbol (lib_name "RESISTOR-1206-4K7_2") (lib_id "tronixio:RESISTOR-1206-4K7") (at 187.96 35.56 0) (unit 1)
     (in_bom yes) (on_board yes)
     (property "Reference" "R205" (id 0) (at 188.595 31.75 0)
@@
       (effects (font (size 1.15 1.15)))
     )
-    (property "Footprint" "tronixio:RESISTOR-1206" (id 2) (at 187.96 50.8 0)
-      (effects (font (size 1 1)) hide)
-    )
-    (property "Datasheet" "https://www.koaspeer.com/pdfs/RK73B.pdf" (id 3) (at 187.96 53.34 0)
+    (property "Footprint" "tronixio:RESISTOR-SMD-1206" (id 2) (at 187.96 50.8 0)
+      (effects (font (size 1 1)) hide)
+    )
+    (property "Datasheet" "https://www.koaspeer.com/products/resistors/general-purpose/rk73b/" (id 3) (at 187.96 53.34 0)
       (effects (font (size 1 1)) hide)
     )
@@
     (pin "2")
   )
-  (symbol (lib_id "tronixio:CAPACITOR-1206-100N") (at 83.82 43.18 0) (unit 1)
+  (symbol (lib_name "CAPACITOR-1206-100N_2") (lib_id "tronixio:CAPACITOR-1206-100N") (at 83.82 43.18 0) (unit 1)
     (in_bom yes) (on_board yes)
     (property "Reference" "C202" (id 0) (at 84.455 45.72 0)
@@
       (effects (font (size 1.15 1.15)) (justify left))
     )
-    (property "Footprint" "tronixio:CAPACITOR-1206" (id 2) (at 83.82 55.88 0)
+    (property "Footprint" "tronixio:CAPACITOR-SMD-1206" (id 2) (at 83.82 55.88 0)
       (effects (font (size 1 1)) hide)
     )
@@
     (pin "2")
   )
-  (symbol (lib_id "tronixio:MICROCHIP-PIC24FJ64GA102-ISP") (at 144.78 72.39 0) (unit 1)
+  (symbol (lib_id "tronixio:MICROCHIP-PIC24FJ64GA102-ISP") (at 129.54 55.88 0) (unit 1)
     (in_bom yes) (on_board yes)
     (property "Reference" "U202" (id 0) (at 132.08 52.07 0)
@@
       (effects (font (size 1.15 1.15)) (justify right))
     )
-    (property "Footprint" "tronixio:DIP-28-W762-SOCKET" (id 2) (at 144.78 100.33 0)
-      (effects (font (size 1 1)) hide)
-    )
-    (property "Datasheet" "https://www.microchip.com/en-us/product/PIC24FJ64GA102" (id 3) (at 144.78 102.87 0)
-      (effects (font (size 1 1)) hide)
-    )
-    (property "Name" "MICROCHIP-PIC24FJ64GA102-ISP" (id 4) (at 144.78 97.79 0)
-      (effects (font (size 1 1)) hide)
-    )
-    (property "Mouser" "579-P24FJ64GA102ISP" (id 5) (at 144.78 105.41 0)
+    (property "Footprint" "tronixio:DIP-28-W762" (id 2) (at 144.78 99.06 0)
+      (effects (font (size 1 1)) hide)
+    )
+    (property "Datasheet" "https://www.microchip.com/en-us/product/PIC24FJ64GA102" (id 3) (at 144.78 101.6 0)
+      (effects (font (size 1 1)) hide)
+    )
+    (property "Name" "MICROCHIP-PIC24FJ64GA102-ISP" (id 4) (at 144.78 96.52 0)
+      (effects (font (size 1 1)) hide)
+    )
+    (property "Mouser" "579-P24FJ64GA102ISP" (id 5) (at 144.78 104.14 0)
       (effects (font (size 1 1)) hide)
     )
@@
     (pin "9")
   )
-  (symbol (lib_id "tronixio:RESISTOR-1206-4K7") (at 177.8 35.56 0) (unit 1)
+  (symbol (lib_name "RESISTOR-1206-4K7_1") (lib_id "tronixio:RESISTOR-1206-4K7") (at 177.8 35.56 0) (unit 1)
     (in_bom yes) (on_board yes)
     (property "Reference" "R204" (id 0) (at 177.165 31.75 0)
@@
       (effects (font (size 1.15 1.15)))
     )
-    (property "Footprint" "tronixio:RESISTOR-1206" (id 2) (at 177.8 50.8 0)
-      (effects (font (size 1 1)) hide)
-    )
-    (property "Datasheet" "https://www.koaspeer.com/pdfs/RK73B.pdf" (id 3) (at 177.8 53.34 0)
+    (property "Footprint" "tronixio:RESISTOR-SMD-1206" (id 2) (at 177.8 50.8 0)
+      (effects (font (size 1 1)) hide)
+    )
+    (property "Datasheet" "https://www.koaspeer.com/products/resistors/general-purpose/rk73b/" (id 3) (at 177.8 53.34 0)
       (effects (font (size 1 1)) hide)
     )
@@
       (effects (font (size 1.15 1.15)))
     )
-    (property "Footprint" "tronixio:FUSE-1206" (id 2) (at 55.88 177.8 0)
+    (property "Footprint" "tronixio:FUSE-SMD-1206" (id 2) (at 55.88 177.8 0)
       (effects (font (size 1 1)) hide)
     )
@@
       (effects (font (size 1.15 1.15)))
     )
-    (property "Footprint" "tronixio:RESISTOR-1206" (id 2) (at 76.2 48.26 0)
-      (effects (font (size 1 1)) hide)
-    )
-    (property "Datasheet" "https://www.koaspeer.com/pdfs/RK73B.pdf" (id 3) (at 76.2 50.8 0)
+    (property "Footprint" "tronixio:RESISTOR-SMD-1206" (id 2) (at 76.2 48.26 0)
+      (effects (font (size 1 1)) hide)
+    )
+    (property "Datasheet" "https://www.koaspeer.com/products/resistors/general-purpose/rk73b/" (id 3) (at 76.2 50.8 0)
       (effects (font (size 1 1)) hide)
     )
@@
       (effects (font (size 1.15 1.15)))
     )
-    (property "Footprint" "tronixio:RESISTOR-1206" (id 2) (at 121.92 185.42 0)
-      (effects (font (size 1 1)) hide)
-    )
-    (property "Datasheet" "https://www.koaspeer.com/pdfs/RK73B.pdf" (id 3) (at 121.92 187.96 0)
+    (property "Footprint" "tronixio:RESISTOR-SMD-1206" (id 2) (at 121.92 185.42 0)
+      (effects (font (size 1 1)) hide)
+    )
+    (property "Datasheet" "https://www.koaspeer.com/products/resistors/general-purpose/rk73b/" (id 3) (at 121.92 187.96 0)
       (effects (font (size 1 1)) hide)
     )
@@
       (effects (font (size 1.15 1.15)) (justify left))
     )
-    (property "Footprint" "tronixio:LED-1206" (id 2) (at 111.76 180.34 0)
-      (effects (font (size 1 1)) hide)
-    )
+    (property "Footprint" "tronixio:LED-SMD-1206" (id 2) (at 111.76 180.34 0)
+      (effects (font (size 1 1)) hide)
+    )

Commit message: Update
Parts:
- JP205: value VCA -> VCAP
Other:
- note added: "*"
- note added: "*Power & UART OR Header Power IN"
- note added: "*U202: Check the pinout for the desired MCU family"
- note removed: "Power & UART OR Header Power IN"
- note removed: "U202: Check the pinout for the desired MCU family"
Changed lines of the file:
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@@
     (effects (font (size 1.15 1.15)) (justify left bottom))
   )
-  (text "U202: Check the pinout for the desired MCU family" (at 181.61 173.99 0)
+  (text "*U202: Check the pinout for the desired MCU family"
+    (at 181.61 173.99 0)
     (effects (font (size 1.27 1.27)) (justify left bottom))
   )
@@
     (effects (font (size 1.15 1.15)) (justify right bottom))
   )
-  (text "Power & UART OR Header Power IN" (at 181.61 171.45 0)
+  (text "*Power & UART OR Header Power IN" (at 181.61 171.45 0)
     (effects (font (size 1.27 1.27)) (justify left bottom))
   )
@@
   (text "GND" (at 66.04 74.93 180)
     (effects (font (size 1.15 1.15)) (justify right bottom))
+  )
+  (text "*" (at 132.08 53.34 0)
+    (effects (font (size 1.27 1.27)) (justify left bottom))
   )
   (text "RB3" (at 66.04 72.39 180)
@@
       (effects (font (size 1.15 1.15)) (justify right))
     )
-    (property "Value" "VCA" (id 1) (at 194.945 142.24 0)
+    (property "Value" "VCAP" (id 1) (at 194.945 142.24 0)
       (effects (font (size 1.15 1.15)) (justify right))
     )
@@
   (symbol (lib_id "tronixio:MICROCHIP-PIC24FJ64GA102-ISP") (at 129.54 55.88 0) (unit 1)
     (in_bom yes) (on_board yes)
-    (property "Reference" "U202" (id 0) (at 132.08 52.07 0)
-      (effects (font (size 1.15 1.15)) (justify left))
-    )
+    (property "Reference" "U202" (id 0) (at 133.35 52.07 0)
+      (effects (font (size 1.15 1.15)) (justify left))
+    )

Commit message: Update Mini
Parts:
- C201, C203: symbol tronixio:CAPACITOR-1206-10U -> tronixio:KEMET-X5R-1206-10U-25V-20P; Mouser 80-C1206C106M3R -> 80-C1206C106M3P; Name CAPACITOR-1206-10U -> (none)
- C202, C204, C205: symbol tronixio:CAPACITOR-1206-100N -> tronixio:KEMET-X7R-1206-100N-50V-20P; Name CAPACITOR-1206-100N -> (none)
- C206: symbol tronixio:KEMET-C322-10U-508 -> tronixio:KEMET-C322-0508-10U-25V-10P; Name KEMET-C32210U-508 -> (none); Voltage (none) -> 25V
- D201, D202: Name NEXPERIA-PMEG3030 -> (none)
- F201: Name BOURNS-FUSE-MF-NSMF050 -> (none)
- JP201, JP202, JP203, JP205: Name HARWIN-254-M-1X02-JUMPER-VERTICAL -> (none)
- JP204: Name HARWIN-254-M-1X03-VERTICAL -> (none)
- K201: Name FCI-USB-TYPE-B-MICRO-THT -> (none)
- K202, K205: Name HARWIN-254-M-1X14-VERTICAL -> (none)
- K203, K206: Name HARWIN-254-F-1X14-VERTICAL -> (none)
- K204: Name MICROCHIP-ICSP-F-1X06 -> (none)
- LED201: Name KINGBRIGHT-LED-1206-BLUE -> (none)
- R201: symbol tronixio:RESISTOR-1206-10K -> tronixio:KOASPEER-RK73B-1206-10K-5P; Name RESISTOR-1206-10K -> (none)
- R202: symbol tronixio:RESISTOR-1206-1K -> tronixio:KOASPEER-RK73B-1206-1K-5P; Name RESISTOR-1206-1K -> (none)
- R203, R204, R205: symbol tronixio:RESISTOR-1206-4K7 -> tronixio:KOASPEER-RK73B-1206-4K7-5P; Name RESISTOR-1206-4K7 -> (none)
- S201: Name ALPS-SKRPAC -> (none)
- TP201, TP202: Name KEYSTONE-5006 -> (none)
- TP203: Name KEYSTONE-2000-3 -> (none)
- U201: Name TI-TLV1117-33-SOT-223 -> (none)
- U202: Name MICROCHIP-PIC24FJ64GA102-ISP -> (none)
Other:
- moved on the sheet: C206, JP201, JP202, JP203, JP205

Commit message: Up
Parts:
- C201, C203: symbol tronixio:KEMET-X5R-1206-10U-25V-20P -> tronixio:CAPACITOR-1206-10U-20P-X7R; Mouser 80-C1206C106M3P -> 80-C1206C106M9P; Voltage 25V -> 6V3
- C202, C204, C205: symbol tronixio:KEMET-X7R-1206-100N-50V-20P -> tronixio:CAPACITOR-1206-100N-10P-X7R; Mouser 80-C1206C104M5R -> 80-C1206C104K5R; Tolerance 20% -> 10%
- R201: symbol tronixio:KOASPEER-RK73B-1206-10K-5P -> tronixio:RESISTOR-1206-10K-5P
- R202: symbol tronixio:KOASPEER-RK73B-1206-1K-5P -> tronixio:RESISTOR-1206-1K-5P
- R203, R204, R205: symbol tronixio:KOASPEER-RK73B-1206-4K7-5P -> tronixio:RESISTOR-1206-4K7-5P
Other:
- moved on the sheet: K204

Commit message: Update
Parts:
- C201, C203: symbol tronixio:CAPACITOR-1206-10U-20P-X7R -> tronixio:CAPACITOR-1206-10U-10P-X7R; Mouser 80-C1206C106M9P -> 80-C1206C106K3R; Tolerance 20% -> 10%; Voltage 6V3 -> 25V
- C202, C204, C205: Mouser 80-C1206C104K5R -> 187-CL31B106KAHNFNE
Changed lines of the file:
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@@
     )
   )
-  (symbol (lib_id "tronixio:CAPACITOR-1206-10U-20P-X7R") (at 81.28 180.34 0) (unit 1)
+  (symbol (lib_id "tronixio:CAPACITOR-1206-10U-10P-X7R") (at 81.28 180.34 0) (unit 1)
     (in_bom yes) (on_board yes) (dnp no)
     (property "Reference" "C201" (at 80.645 177.8 0)
@@
       (effects (font (size 1 1)) hide)
     )
-    (property "Voltage" "6V3" (at 86.28 185.42 0) (do_not_autoplace)
-      (effects (font (size 1.15 1.15)) (justify left) hide)
-    )
-    (property "Tolerance" "20%" (at 82.28 185.42 0) (do_not_autoplace)
-      (effects (font (size 1.15 1.15)) (justify left) hide)
-    )
-    (property "Mouser" "80-C1206C106M9P" (at 81.28 193.04 0)
+    (property "Voltage" "25V" (at 86.28 185.42 0) (do_not_autoplace)
+      (effects (font (size 1.15 1.15)) (justify left) hide)
+    )
+    (property "Tolerance" "10%" (at 82.28 185.42 0) (do_not_autoplace)
+      (effects (font (size 1.15 1.15)) (justify left) hide)
+    )
+    (property "Mouser" "80-C1206C106K3R" (at 81.28 193.04 0)
       (effects (font (size 1 1)) hide)
     )
@@
       (effects (font (size 1.15 1.15)) (justify left) hide)
     )
-    (property "Mouser" "80-C1206C104K5R" (at 167.64 109.22 0)
+    (property "Mouser" "187-CL31B106KAHNFNE" (at 167.64 109.22 0)
       (effects (font (size 1 1)) hide)
     )
@@
     )
   )
-  (symbol (lib_id "tronixio:CAPACITOR-1206-10U-20P-X7R") (at 106.68 180.34 0) (unit 1)
+  (symbol (lib_id "tronixio:CAPACITOR-1206-10U-10P-X7R") (at 106.68 180.34 0) (unit 1)
     (in_bom yes) (on_board yes) (dnp no)
     (property "Reference" "C203" (at 107.315 177.8 0)
@@
       (effects (font (size 1 1)) hide)
     )
-    (property "Voltage" "6V3" (at 111.68 185.42 0) (do_not_autoplace)
-      (effects (font (size 1.15 1.15)) (justify left) hide)
-    )
-    (property "Tolerance" "20%" (at 107.68 185.42 0) (do_not_autoplace)
-      (effects (font (size 1.15 1.15)) (justify left) hide)
-    )
-    (property "Mouser" "80-C1206C106M9P" (at 106.68 193.04 0)
+    (property "Voltage" "25V" (at 111.68 185.42 0) (do_not_autoplace)
+      (effects (font (size 1.15 1.15)) (justify left) hide)
+    )
+    (property "Tolerance" "10%" (at 107.68 185.42 0) (do_not_autoplace)
+      (effects (font (size 1.15 1.15)) (justify left) hide)
+    )
+    (property "Mouser" "80-C1206C106K3R" (at 106.68 193.04 0)
       (effects (font (size 1 1)) hide)
     )
@@
       (effects (font (size 1.15 1.15)) (justify left) hide)
     )
-    (property "Mouser" "80-C1206C104K5R" (at 121.92 109.22 0)
+    (property "Mouser" "187-CL31B106KAHNFNE" (at 121.92 109.22 0)
       (effects (font (size 1 1)) hide)
     )
@@
       (effects (font (size 1.15 1.15)) (justify left) hide)
     )
-    (property "Mouser" "80-C1206C104K5R" (at 83.82 55.88 0)
-      (effects (font (size 1 1)) hide)
-    )
+    (property "Mouser" "187-CL31B106KAHNFNE" (at 83.82 55.88 0)
+      (effects (font (size 1 1)) hide)
+    )

Commit message: Up
Parts:
- removed C206: 10µ, tronixio:KEMET-C322, symbol tronixio:KEMET-C322-0508-10U-25V-10P
- added C206: 10µ, tronixio:CAPACITOR-SMD-1206, symbol tronixio:CAPACITOR-1206-10U-25V-5P-X7R
- C201, C203: symbol tronixio:CAPACITOR-1206-10U-10P-X7R -> tronixio:CAPACITOR-1206-10U-25V-5P-X7R; Mouser 80-C1206C106K3R -> 791-1206X106J250CT; Tolerance 10% -> 5%
- C202, C204, C205: symbol tronixio:CAPACITOR-1206-100N-10P-X7R -> tronixio:CAPACITOR-1206-100N-50V-5P-X7R; Mouser 187-CL31B106KAHNFNE -> 80-C1206C104J5R; Tolerance 10% -> 5%
- K201: footprint tronixio:FCI-USB-TYPE-B-MICRO-THT -> tronixio:USB-TYPE-B-MICRO-TH
- U202: footprint tronixio:DIP-28-W762 -> tronixio:DIP-28-W762-SOCKET
Connections:
- net GND: now also K201.SH (SHIELD), C206.2; no longer K201.6 (SHIELD)
- net at JP205.2: now also C206.1
