File: Kicad/mini/pic16bit-mcu.kicad_sch (KiCad schematic)
At the start: 32 parts, among them K201 *Power & UART, K202 MCU 1, K203 MCU 1, K204 ICSP, K205 MCU 2, K206 MCU 2, U201 TLV1117-33, U202 PIC24/dsPIC32

Commit message: Up
Parts:
- K201: symbol tronixio:FCI-USB-TYPE-B-MICRO-THT -> tronixio:FCI-USB-TYPE-B-MICRO-TH
Changed lines of the file:
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@@
     )
   )
-  (symbol (lib_id "tronixio:FCI-USB-TYPE-B-MICRO-THT") (at 38.1 175.26 0) (unit 1)
+  (symbol (lib_id "tronixio:FCI-USB-TYPE-B-MICRO-TH") (at 38.1 175.26 0) (unit 1)
     (in_bom yes) (on_board yes) (dnp no)
     (property "Reference" "K201" (at 38.1 162.56 0)

Commit message: Up
Parts:
- K204: symbol tronixio:MICROCHIP-ICSP-F-1X06 -> tronixio:MICROCHIP-ICSP-F-RIGHT-ANGLE-TH
- U202: footprint tronixio:DIP-28-W762-SOCKET -> tronixio:DIP-28-W762
Changed lines of the file:
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@@
       (effects (font (size 1.15 1.15)) (justify right))
     )
-    (property "Footprint" "tronixio:DIP-28-W762-SOCKET" (at 144.78 96.52 0) (do_not_autoplace)
+    (property "Footprint" "tronixio:DIP-28-W762" (at 144.78 96.52 0) (do_not_autoplace)
       (effects (font (size 1 1)) hide)
     )
@@
     )
   )
-  (symbol (lib_id "tronixio:MICROCHIP-ICSP-F-1X06") (at 149.86 111.76 0) (unit 1)
+  (symbol (lib_id "tronixio:MICROCHIP-ICSP-F-RIGHT-ANGLE-TH") (at 149.86 111.76 0) (unit 1)
     (in_bom yes) (on_board yes) (dnp no)
     (property "Reference" "K204" (at 149.86 109.22 0)

Commit message: Update
Parts:
- C201, C203, C206: Mouser 791-1206X106J250CT -> 80-C1206C106J3R
- D201, D202: symbol tronixio:NEXPERIA-PMEG3030 -> tronixio:NEXPERIA-PMEG3030-SOD
Changed lines of the file:
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@@
       (effects (font (size 1.15 1.15)) (justify left) hide)
     )
-    (property "Mouser" "791-1206X106J250CT" (at 193.04 162.56 0) (do_not_autoplace)
+    (property "Mouser" "80-C1206C106J3R" (at 193.04 162.56 0) (do_not_autoplace)
       (effects (font (size 1 1)) hide)
     )
@@
     )
   )
-  (symbol (lib_id "tronixio:NEXPERIA-PMEG3030") (at 68.58 175.26 180) (unit 1)
+  (symbol (lib_id "tronixio:NEXPERIA-PMEG3030-SOD") (at 68.58 175.26 180) (unit 1)
     (in_bom yes) (on_board yes) (dnp no)
     (property "Reference" "D202" (at 68.58 179.705 0)
@@
       (effects (font (size 1.15 1.15)) (justify left) hide)
     )
-    (property "Mouser" "791-1206X106J250CT" (at 81.28 193.04 0) (do_not_autoplace)
+    (property "Mouser" "80-C1206C106J3R" (at 81.28 193.04 0) (do_not_autoplace)
       (effects (font (size 1 1)) hide)
     )
@@
       (effects (font (size 1.15 1.15)) (justify left) hide)
     )
-    (property "Mouser" "791-1206X106J250CT" (at 106.68 193.04 0) (do_not_autoplace)
+    (property "Mouser" "80-C1206C106J3R" (at 106.68 193.04 0) (do_not_autoplace)
       (effects (font (size 1 1)) hide)
     )
@@
     )
   )
-  (symbol (lib_id "tronixio:NEXPERIA-PMEG3030") (at 68.58 170.18 180) (unit 1)
+  (symbol (lib_id "tronixio:NEXPERIA-PMEG3030-SOD") (at 68.58 170.18 180) (unit 1)
     (in_bom yes) (on_board yes) (dnp no)
     (property "Reference" "D201" (at 68.58 165.1 0)

Commit message: Update Mini Kicad 8
Parts:
- U201: footprint tronixio:SOT-223-3 -> tronixio:SOT-223-3-TABPIN2
Connections:
- net +3V3 renamed POWER-+3V3
- net +5V renamed POWER-+5V
- net GND renamed POWER-GND

Commit message: Update Mini
Changed lines of the file:
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@@
 	)
 	(junction
+		(at 86.36 170.18)
+		(diameter 0)
+		(color 0 0 0 0)
+	)
+	(junction
 		(at 45.72 185.42)
 		(diameter 0)
@@
 	(wire
 		(pts
-			(xy 177.8 182.88) (xy 177.8 190.5)
-		)
-		(stroke
-			(width 0)
-			(type solid)
-		)
-	)
-	(wire
-		(pts
 			(xy 93.98 175.26) (xy 93.98 187.96)
 		)
@@
 	(wire
 		(pts
-			(xy 81.28 170.18) (xy 88.9 170.18)
+			(xy 81.28 170.18) (xy 86.36 170.18)
 		)
 		(stroke
@@
 	(wire
 		(pts
+			(xy 86.36 170.18) (xy 88.9 170.18)
+		)
+		(stroke
+			(width 0)
+			(type solid)
+		)
+	)
+	(wire
+		(pts
 			(xy 167.64 99.06) (xy 167.64 101.6)
 		)
@@
 	(text "5V MAX"
 		(exclude_from_sim no)
-		(at 57.785 188.595 0)
+		(at 57.785 187.96 0)
 		(effects
 			(font
@@
 		(on_board yes)
 		(dnp no)
-		(fields_autoplaced yes)
 		(property "Reference" "#PWR0123"
 			(at 121.92 175.26 0)
@@
 			)
 		)
-		(property "Description" ""
-			(at 121.92 162.56 0)
-			(effects
-				(font
-					(size 1.27 1.27)
-				)
-				(hide yes)
-			)
-		)
-		(property "Name" "3V3"
+		(property "Description" "3V3"
 			(at 121.92 157.48 0)
-			(do_not_autoplace yes)
 			(effects
 				(font
-					(size 1.15 1.15)
+					(size 1.27 1.27)
 				)
 			)
@@
 		(on_board yes)
 		(dnp no)
-		(fields_autoplaced yes)
 		(property "Reference" "#PWR0165"
 			(at 175.26 144.78 0)
@@
 			)
 		)
-		(property "Description" ""
-			(at 175.26 132.08 0)
-			(effects
-				(font
-					(size 1.27 1.27)
-				)
-				(hide yes)
-			)
-		)
-		(property "Name" "3V3"
+		(property "Description" "3V3"
 			(at 175.26 127 0)
-			(do_not_autoplace yes)
 			(effects
 				(font
-					(size 1.15 1.15)
+					(size 1.27 1.27)
 				)
 			)
@@
 		(on_board yes)
 		(dnp no)
-		(fields_autoplaced yes)
 		(property "Reference" "#PWR0164"
 			(at 121.92 40.64 0)
@@
 			)
 		)
-		(property "Description" ""
-			(at 121.92 27.94 0)
-			(effects
-				(font
-					(size 1.27 1.27)
-				)
-				(hide yes)
-			)
-		)
-		(property "Name" "3V3"
+		(property "Description" "3V3"
 			(at 121.92 22.86 0)
-			(do_not_autoplace yes)
 			(effects
 				(font
-					(size 1.15 1.15)
+					(size 1.27 1.27)
 				)
 			)
@@
 		(on_board yes)
 		(dnp no)
-		(fields_autoplaced yes)
 		(property "Reference" "#PWR0101"
 			(at 167.64 40.64 0)
@@
 			)
 		)
-		(property "Description" ""
-			(at 167.64 27.94 0)
-			(effects
-				(font
-					(size 1.27 1.27)
-				)
-				(hide yes)
-			)
-		)
-		(property "Name" "3V3"
+		(property "Description" "3V3"
 			(at 167.64 22.86 0)
-			(do_not_autoplace yes)
 			(effects
 				(font
-					(size 1.15 1.15)
+					(size 1.27 1.27)
 				)
 			)
@@
 		(on_board yes)
 		(dnp no)
-		(fields_autoplaced yes)
 		(property "Reference" "#PWR0103"
 			(at 144.78 121.92 0)
@@
 			)
 		)
-		(property "Description" ""
-			(at 144.78 109.22 0)
-			(effects
-				(font
-					(size 1.27 1.27)
-				)
-				(hide yes)
-			)
-		)
-		(property "Name" "3V3"
+		(property "Description" "3V3"
 			(at 144.78 104.14 0)
-			(do_not_autoplace yes)
 			(effects
 				(font
-					(size 1.15 1.15)
+					(size 1.27 1.27)
 				)
 			)
@@
 	(symbol
 		(lib_id "tronixio:POWER-FLAG")
-		(at 177.8 190.5 180)
+		(at 86.36 170.18 0)
 		(unit 1)
 		(exclude_from_sim no)
@@
 		(fields_autoplaced yes)
 		(property "Reference" "#FLG0201"
-			(at 177.8 188.595 0)
+			(at 86.36 172.085 0)
 			(effects
 				(font
@@
 		)
 		(property "Value" "PWR_FLAG"
-			(at 177.8 186.69 0)
+			(at 86.36 173.99 0)
 			(effects
 				(font
@@
 		)
 		(property "Footprint" ""
-			(at 177.8 190.5 0)
+			(at 86.36 170.18 0)
 			(effects
 				(font
@@
 		)
 		(property "Datasheet" ""
-			(at 177.8 190.5 0)
+			(at 86.36 170.18 0)
 			(effects
 				(font
@@
 		)
 		(property "Description" "Special symbol for telling ERC where power comes from"
-			(at 177.8 190.5 0)
+			(at 86.36 170.18 0)
 			(effects
 				(font
@@
 		)
 		(property "Value" "Power IN"
-			(at 57.785 185.42 0)
+			(at 57.785 184.785 0)
 			(effects
 				(font
@@
 		(on_board yes)
 		(dnp no)
-		(fields_autoplaced yes)
 		(property "Reference" "#PWR0113"
 			(at 187.96 40.64 0)
@@
 			)
 		)
-		(property "Description" ""
-			(at 187.96 27.94 0)
-			(effects
-				(font
-					(size 1.27 1.27)
-				)
-				(hide yes)
-			)
-		)
-		(property "Name" "3V3"
+		(property "Description" "3V3"
 			(at 187.96 22.86 0)
-			(do_not_autoplace yes)
 			(effects
 				(font
-					(size 1.15 1.15)
+					(size 1.27 1.27)
 				)
 			)
@@
 		(on_board yes)
 		(dnp no)
-		(fields_autoplaced yes)
 		(property "Reference" "#PWR0110"
 			(at 76.2 40.64 0)
@@
 			)
 		)
-		(property "Description" ""
-			(at 76.2 27.94 0)
-			(effects
-				(font
-					(size 1.27 1.27)
-				)
-				(hide yes)
-			)
-		)
-		(property "Name" "3V3"
+		(property "Description" "3V3"
 			(at 76.2 22.86 0)
-			(do_not_autoplace yes)
 			(effects
 				(font
-					(size 1.15 1.15)
+					(size 1.27 1.27)
 				)
 			)
@@
 		(on_board yes)
 		(dnp no)
-		(fields_autoplaced yes)
 		(property "Reference" "#PWR0102"
 			(at 177.8 40.64 0)
@@
 			)
 		)
-		(property "Description" ""
-			(at 177.8 27.94 0)
-			(effects
-				(font
-					(size 1.27 1.27)
-				)
-				(hide yes)
-			)
-		)
-		(property "Name" "3V3"
+		(property "Description" "3V3"
 			(at 177.8 22.86 0)
-			(do_not_autoplace yes)
 			(effects
 				(font
-					(size 1.15 1.15)
+					(size 1.27 1.27)
 				)
 			)
@@
 		(on_board yes)
 		(dnp no)
-		(fields_autoplaced yes)
 		(property "Reference" "#PWR0124"
 			(at 106.68 175.26 0)
@@
 			)
 		)
-		(property "Description" ""
-			(at 106.68 162.56 0)
-			(effects
-				(font
-					(size 1.27 1.27)
-				)
-				(hide yes)
-			)
-		)
-		(property "Name" "3V3"
+		(property "Description" "3V3"
 			(at 106.68 157.48 0)
-			(do_not_autoplace yes)
 			(effects
 				(font
-					(size 1.15 1.15)
+					(size 1.27 1.27)
 				)
 			)
@@
 	)
 	(symbol
-		(lib_id "tronixio:POWER-+5V")
-		(at 177.8 182.88 0)
-		(unit 1)
-		(exclude_from_sim no)
-		(in_bom yes)
-		(on_board yes)
-		(dnp no)
-		(fields_autoplaced yes)
-		(property "Reference" "#PWR0107"
-			(at 177.8 193.04 0)
-			(effects
-				(font
-					(size 1 1)
-				)
-				(hide yes)
-			)
-		)
-		(property "Value" "POWER-+5V"
-			(at 177.8 195.58 0)
-			(effects
-				(font
-					(size 1 1)
-				)
-				(hide yes)
-			)
-		)
-		(property "Footprint" ""
-			(at 177.8 182.88 0)
-			(effects
-				(font
-					(size 1 1)
-				)
-				(hide yes)
-			)
-		)
-		(property "Datasheet" ""
-			(at 177.8 182.88 0)
-			(effects
-				(font
-					(size 1 1)
-				)
-				(hide yes)
-			)
-		)
-		(property "Description" ""
-			(at 177.8 182.88 0)
-			(effects
-				(font
-					(size 1.27 1.27)
-				)
-				(hide yes)
-			)
-		)
-		(property "Name" "5V"
-			(at 177.8 177.8 0)
-			(do_not_autoplace yes)
-			(effects
-				(font
-					(size 1.15 1.15)
-				)
-			)
-		)
-		(pin "1"
-		)
-		(instances
-			(project "pic16bit"
-				(path "/d431d485-8cd8-4e00-afcd-f39218d614ca/64edc06d-d6ae-4dac-9759-3f1fbed6457d"
-					(reference "#PWR0107")
-					(unit 1)
-				)
-			)
-		)
-	)
-	(symbol
 		(lib_id "tronixio:MICROCHIP-ICSP-F-RIGHT-ANGLE-TH")
 		(at 149.86 111.76 0)
@@
 		(on_board yes)
 		(dnp no)
-		(fields_autoplaced yes)
 		(property "Reference" "#PWR0118"
 			(at 81.28 172.72 0)
@@
 			)
 		)
-		(property "Description" ""
-			(at 81.28 162.56 0)
-			(effects
-				(font
-					(size 1.27 1.27)
-				)
-				(hide yes)
-			)
-		)
-		(property "Name" "5V"
+		(property "Description" "5V"
 			(at 81.28 157.48 0)
-			(do_not_autoplace yes)
 			(effects
 				(font
-					(size 1.15 1.15)
+					(size 1.27 1.27)
 				)
 			)

Commit message: Up
Parts:
- U202: value PIC24/dsPIC32 -> PIC24/dsPIC33
Changed lines of the file:
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@@
 			)
 		)
-		(property "Value" "PIC24/dsPIC32"
+		(property "Value" "PIC24/dsPIC33"
 			(at 157.48 52.07 0)
 			(effects
