File: Kicad/nano/pic16bit.kicad_sch (KiCad schematic)
At the start: 35 parts, among them K1 MCU 1, K2 MCU 2, K3 ICSP, K4 POWER & UART, U1 PIC24/dsPIC32, U2 MCP2221A-IST, U3 BU33SD5WG

Commit message: Update
Parts:
- U2: value MCP2221A-IST -> MCP2221A
Other:
- note added: "*R4/*R5/*JP3/*JP4: I2C Optional components."
- note added: "*U2/*R3/*R6/*R7/*LED2/*LED3: EUSART Optional components."
- note removed: "*R1/*R4/*R5/*LED2/*LED3/*U2: EUSART Optional components."
- note removed: "*R2/*R3/*JP3/*JP4: I2C Optional components."
Changed lines of the file:
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@@
     (effects (font (size 1.27 1.27)) (justify right bottom))
   )
-  (text "*R1/*R4/*R5/*LED2/*LED3/*U2: EUSART Optional components."
+  (text "*U2/*R3/*R6/*R7/*LED2/*LED3: EUSART Optional components."
     (at 181.61 179.07 0)
     (effects (font (size 1.27 1.27)) (justify left bottom))
@@
     (effects (font (size 1.15 1.15)) (justify right bottom))
   )
-  (text "*R2/*R3/*JP3/*JP4: I2C Optional components." (at 181.61 176.53 0)
+  (text "*R4/*R5/*JP3/*JP4: I2C Optional components." (at 181.61 176.53 0)
     (effects (font (size 1.27 1.27)) (justify left bottom))
   )
@@
     (effects (font (size 1.15 1.15)) (justify right bottom))
   )
-  (text "*" (at 118.745 129.54 180)
-    (effects (font (size 1.15 1.15)) (justify right bottom))
+  (text "*" (at 111.76 129.54 0)
+    (effects (font (size 1.15 1.15)) (justify left bottom))
   )
   (label "RA0" (at 58.42 83.82 180)
@@
   (symbol (lib_id "tronixio:MICROCHIP-MCP2221A-IST") (at 109.22 132.08 0) (unit 1)
     (in_bom yes) (on_board yes)
-    (property "Reference" "U2" (id 0) (at 120.015 128.27 0)
-      (effects (font (size 1.15 1.15)))
-    )
-    (property "Value" "MCP2221A-IST" (id 1) (at 119.38 156.21 0)
-      (effects (font (size 1.15 1.15)))
+    (property "Reference" "U2" (id 0) (at 113.03 128.27 0)
+      (effects (font (size 1.15 1.15)) (justify left))
+    )
+    (property "Value" "MCP2221A" (id 1) (at 127 128.27 0)
+      (effects (font (size 1.15 1.15)) (justify right))
     )
     (property "Footprint" "tronixio:TSSOP-14" (id 2) (at 119.38 162.56 0)
@@
     )
     (path "/15b76320-9a6e-4ed9-be26-15ea028b6641"
-      (reference "U2") (unit 1) (value "MCP2221A-IST") (footprint "tronixio:TSSOP-14")
+      (reference "U2") (unit 1) (value "MCP2221A") (footprint "tronixio:TSSOP-14")
     )
     (path "/ef27345a-c7c1-44c7-b4de-dc92b9c6de34"

Commit message: Update
Parts:
- C1, C2, C3, C4, C5: symbol tronixio:CAPACITOR-0805-100N -> tronixio:KEMET-X7R-0805-100N-50V-20P; Name CAPACITOR-0805-100N -> (none)
- C6: symbol tronixio:CAPACITOR-0805-10U -> tronixio:KEMET-X7R-0805-10U-25V-20P; Name CAPACITOR-0805-10U -> (none)
- C7, C8: symbol tronixio:CAPACITOR-0805-1U -> tronixio:KEMET-X7R-0805-1U-50V-20P; Name CAPACITOR-0805-1U -> (none)
- F1: Name BOURNS-FUSE-MF-PSMF050X -> (none)
- JP1, JP2: symbol tronixio:RESISTOR-0805-0 -> tronixio:KOASPEER-RK73B-0805-0; Name RESISTOR-0805-0 -> (none); Tolerance (none) -> 5%
- JP3, JP4: Name HARWIN-200-M-1X02-JUMPER-TH-VERTICAL -> (none)
- K1, K2: Name SAMTEC-254-M-TSW-1X20-22-T-S_1 -> (none)
- K3: Name MICROCHIP-ICSP-M-2X03 -> (none)
- K4: Name FCI-USB-TYPE-B-MICRO-THT -> (none)
- LED1, LED2, LED3: Name KINGBRIGHT-LED-0805-BLUE -> (none)
- MEMS1: Name MICROCHIP-DSC1001C-245760-CDFN -> (none)
- R1, R3: symbol tronixio:RESISTOR-0805-10K -> tronixio:KOASPEER-RK73B-0805-10K-5P; Name RESISTOR-0805-10K -> (none)
- R2: symbol tronixio:RESISTOR-0805-1K -> tronixio:KOASPEER-RK73B-0805-1K-5P; Name RESISTOR-0805-1K -> (none)
- R4, R5, R6, R7, R8: symbol tronixio:RESISTOR-0805-4K7 -> tronixio:KOASPEER-RK73B-0805-4K7-5P; Name RESISTOR-0805-4K7 -> (none)
- S1: Name ALPS-SKRPAC -> (none)
- U1: Name MICROCHIP-PIC24FJ64GA104-IPT -> (none)
- U2: Name MICROCHIP-MCP2221A-IST -> (none)
- U3: Name ROHM-BU33SD5WG-500-SOT-23 -> (none)
Other:
- moved on the sheet: JP3, JP4

Commit message: Update Nano
Parts:
- C6: symbol tronixio:KEMET-X7R-0805-10U-25V-20P -> tronixio:KEMET-X5R-0805-10U-25V-20P
Changed lines of the file:
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@@
       (effects (font (size 1 1)) hide)
     )
-    (property "Datasheet" "https://www.bourns.com/pdfs/mfnsmf.pdf" (id 3) (at 91.44 147.32 0)
+    (property "Datasheet" "https://www.bourns.com/pdfs/mfpsmf.pdf" (id 3) (at 91.44 147.32 0)
       (effects (font (size 1 1)) hide)
     )
@@
     (pin "1")
   )
-  (symbol (lib_id "tronixio:KEMET-X7R-0805-10U-25V-20P") (at 149.86 93.98 0) (unit 1)
+  (symbol (lib_id "tronixio:KEMET-X5R-0805-10U-25V-20P") (at 149.86 93.98 0) (unit 1)
     (in_bom yes) (on_board yes)
     (property "Reference" "C6" (id 0) (at 149.225 91.44 0)

Commit message: Update Nano
Parts:
- C6: symbol tronixio:KEMET-X5R-0805-10U-25V-20P -> tronixio:KEMET-X5R-0805-10U-6V3-20P; Mouser 80-C0805C106M3P -> 80-C0805C106M9P; Voltage 25V -> 6V3
- C7, C8: symbol tronixio:KEMET-X7R-0805-1U-50V-20P -> tronixio:KEMET-X7R-0805-1U-16V-20P; Mouser 80-C0805C105M5R -> 80-C0805C105M4R; Voltage 50V -> 16V
Connections:
- net +3V3: no longer U3.5 (VOUT)

Commit message: Up
Parts:
- C1, C2, C3, C4, C5: symbol tronixio:KEMET-X7R-0805-100N-50V-20P -> tronixio:CAPACITOR-0805-100N-20P-X7R
- C6: symbol tronixio:KEMET-X5R-0805-10U-6V3-20P -> tronixio:CAPACITOR-0805-10U-20P-X7R
- C7, C8: symbol tronixio:KEMET-X7R-0805-1U-16V-20P -> tronixio:CAPACITOR-0805-1U-20P-X7R
- JP1, JP2: symbol tronixio:KOASPEER-RK73B-0805-0 -> tronixio:RESISTOR-0805; Mouser 660-RK73Z2ATTD -> (none); Tolerance 5% -> ~%
- R1, R3: symbol tronixio:KOASPEER-RK73B-0805-10K-5P -> tronixio:RESISTOR-0805-10K-5P
- R2: symbol tronixio:KOASPEER-RK73B-0805-1K-5P -> tronixio:RESISTOR-0805-1K-5P
- R4, R5, R6, R7, R8: symbol tronixio:KOASPEER-RK73B-0805-4K7-5P -> tronixio:RESISTOR-0805-4K7-5P
Connections:
- net +3V3: now also U3.5 (VOUT)

Commit message: Up
Parts:
- K4: footprint tronixio:FCI-USB-TYPE-B-MICRO-THT -> tronixio:USB-TYPE-B-MICRO-TH; symbol tronixio:FCI-USB-TYPE-B-MICRO-THT -> tronixio:FCI-USB-TYPE-B-MICRO-TH
Connections:
- net GND: now also K4.SH (SHIELD); no longer K4.6 (SHIELD)
Changed lines of the file:
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@@
     )
   )
-  (symbol (lib_id "tronixio:FCI-USB-TYPE-B-MICRO-THT") (at 81.28 144.78 0) (unit 1)
+  (symbol (lib_id "tronixio:FCI-USB-TYPE-B-MICRO-TH") (at 81.28 144.78 0) (unit 1)
     (in_bom yes) (on_board yes) (dnp no)
     (property "Reference" "K4" (at 81.3705 132.08 0)
@@
       (effects (font (size 1.15 1.15)))
     )
-    (property "Footprint" "tronixio:FCI-USB-TYPE-B-MICRO-THT" (at 81.28 162.56 0)
+    (property "Footprint" "tronixio:USB-TYPE-B-MICRO-TH" (at 81.28 162.56 0) (do_not_autoplace)
       (effects (font (size 1 1)) hide)
     )
-    (property "Datasheet" "https://cdn.amphenol-icc.com/media/wysiwyg/files/drawing/10118193.pdf" (at 81.28 165.1 0)
+    (property "Datasheet" "https://cdn.amphenol-icc.com/media/wysiwyg/files/drawing/10118193.pdf" (at 81.28 165.1 0) (do_not_autoplace)
       (effects (font (size 1 1)) hide)
     )
-    (property "Mouser" "649-10118193-0001LF" (at 81.28 167.64 0)
+    (property "Mouser" "649-10118193-0001LF" (at 81.28 167.64 0) (do_not_autoplace)
       (effects (font (size 1 1)) hide)
     )
@@
     (pin "4")
     (pin "5")
-    (pin "6")
+    (pin "SH")
     (instances
       (project "pic16bit"

Commit message: Up
Parts:
- C1, C2, C3, C4, C5: symbol tronixio:CAPACITOR-0805-100N-20P-X7R -> tronixio:CAPACITOR-0805-100N-50V-5P-X7R; Mouser 80-C0805C104M5R -> 80-C0805C104J5; Tolerance 20% -> 5%
- C6: symbol tronixio:CAPACITOR-0805-10U-20P-X7R -> tronixio:CAPACITOR-0805-10U-25V-10P-X7R; Mouser 80-C0805C106M9P -> 81-GRM21BZ71E106KE5L; Tolerance 20% -> 10%; Voltage 6V3 -> 25V
- C7, C8: symbol tronixio:CAPACITOR-0805-1U-20P-X7R -> tronixio:CAPACITOR-0805-1U-50V-10P-X7R; Mouser 80-C0805C105M4R -> 187-CL21B105KBFNNNE; Tolerance 20% -> 10%; Voltage 16V -> 50V
- JP1, JP2: symbol tronixio:RESISTOR-0805 -> tronixio:RESISTOR-0805-0R; Mouser (none) -> 660-RK73Z2ATTD; Tolerance ~% -> (none)
- JP3, JP4: symbol tronixio:HARWIN-200-M-1X02-JUMPER-TH-VERTICAL -> tronixio:HARWIN-200-M-1X02-JUMPER-VERTICAL
- K3: Mouser 855-M20-9980346 -> 855-M20-998034
Connections:
- no-connect marks 4 -> 5
Other:
- moved on the sheet: C2, MEMS1
