File: Kicad/nano/pic16bit.kicad_sch (KiCad schematic)
At the start: 35 parts, among them K1 MCU 1, K2 MCU 2, K3 ICSP, K4 POWER & UART, U1 PIC24/dsPIC32, U2 MCP2221A, U3 BU33SD5WG

Commit message: Update Nano
Connections:
- net +3V3 renamed POWER-+3V3
- net +5V renamed POWER-+5V
- net GND renamed POWER-GND

Commit message: Update Nano
Connections:
- net POWER-+3V3 renamed +3V3
- net POWER-GND renamed GND
- no-connect marks 5 -> 4
Other:
- moved on the sheet: JP3, JP4

Commit message: Up
Parts:
- U1: value PIC24/dsPIC32 -> PIC24/dsPIC33
Changed lines of the file:
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@@
 			)
 		)
-		(property "Value" "PIC24/dsPIC32"
+		(property "Value" "PIC24/dsPIC33"
 			(at 190.5 63.5 0)
 			(effects

Commit message: Up
Parts:
- K1, K2: symbol tronixio:SAMTEC-254-M-TSW-1X20-22-T-S -> tronixio:SAMTEC-254-M-1X20-VERTICAL
Changed lines of the file:
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@@
 	)
 	(symbol
-		(lib_id "tronixio:SAMTEC-254-M-TSW-1X20-22-T-S")
+		(lib_id "tronixio:SAMTEC-254-M-1X20-VERTICAL")
 		(at 45.72 111.76 0)
 		(mirror y)
@@
 	)
 	(symbol
-		(lib_id "tronixio:SAMTEC-254-M-TSW-1X20-22-T-S")
+		(lib_id "tronixio:SAMTEC-254-M-1X20-VERTICAL")
 		(at 45.72 43.18 0)
 		(mirror y)

Commit message: Up
Parts:
- H1, H2: footprint tronixio:HARWIN-M22-190-193 -> tronixio:HARWIN-M22-190-19X; now left out of the parts list
Changed lines of the file:
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@@
 	(wire
 		(pts
-			(xy 226.06 66.04) (xy 236.22 66.04)
-		)
-		(stroke
-			(width 0)
-			(type default)
-		)
-	)
-	(wire
-		(pts
 			(xy 48.26 71.12) (xy 58.42 71.12)
 		)
@@
 	(wire
 		(pts
+			(xy 226.06 66.04) (xy 233.68 66.04)
+		)
+		(stroke
+			(width 0)
+			(type default)
+		)
+	)
+	(wire
+		(pts
 			(xy 195.58 35.56) (xy 195.58 45.72)
 		)
@@
 			)
 		)
-		(property "Description" "Resistor"
+		(property "Description" ""
 			(at 142.24 91.44 0)
 			(effects
@@
 			)
 		)
-		(property "Description" "Resistor"
+		(property "Description" ""
 			(at 142.24 76.2 0)
 			(effects
@@
 		(unit 1)
 		(exclude_from_sim no)
-		(in_bom yes)
+		(in_bom no)
 		(on_board yes)
 		(dnp no)
@@
 			)
 		)
-		(property "Footprint" "tronixio:HARWIN-M22-190-193"
+		(property "Footprint" "tronixio:HARWIN-M22-190-19X"
 			(at 269.24 182.88 0)
 			(do_not_autoplace yes)
@@
 			)
 		)
-		(property "Description" "Resistor"
+		(property "Description" ""
 			(at 101.6 124.46 0)
 			(effects
@@
 			)
 		)
-		(property "Description" "Resistor"
+		(property "Description" ""
 			(at 254 33.02 0)
 			(effects
@@
 		(unit 1)
 		(exclude_from_sim no)
-		(in_bom yes)
+		(in_bom no)
 		(on_board yes)
 		(dnp no)
@@
 			)
 		)
-		(property "Footprint" "tronixio:HARWIN-M22-190-193"
+		(property "Footprint" "tronixio:HARWIN-M22-190-19X"
 			(at 274.32 182.88 0)
 			(do_not_autoplace yes)

Commit message: Up
Parts:
- C6: Mouser 81-GRM21BZ71E106KE5L -> 81-GRM21BZ71E106
- U2: symbol tronixio:MICROCHIP-MCP2221A-IST -> tronixio:MICROCHIP-MCP2221A-TSSOP
- U3: symbol tronixio:ROHM-BU33SD5WG-500-SOT-23 -> tronixio:ROHM-BU33SD5WG-500-SOT
