File: Kicad/nano/pic16bit.kicad_sch (KiCad schematic)
At the start: 35 parts, among them K1 MCU 1, K2 MCU 2, K3 ICSP, K4 POWER & UART, U1 PIC24/dsPIC33, U2 MCP2221A, U3 BU33SD5WG

Commit message: Up
Parts:
- H1, H2: now in the parts list
- JP3, JP4: symbol tronixio:HARWIN-200-M-1X02-JUMPER-VERTICAL -> tronixio:HARWIN-200-M-1X02-JUMPER-VERTICAL-TH
- K3: symbol tronixio:MICROCHIP-ICSP-M-2X03 -> tronixio:MICROCHIP-ICSP-M-2X03-254-TH
Other:
- note added: "*U1: Check the pinout for the desired MCU family. *C6: Optional check MCU datasheet. *JP1/*JP2: Check MCU datasheet for Selection. *MEMS1/*C2: Optional check MCU datasheet for values. *R4/*R5/*JP3/*JP4: I2C Optional components. *U2/*R3/*R6/*R7/*LED2/*LED3: EUSART Optional components."
- note removed: "*C6: Optional check MCU datasheet."
- note removed: "*JP1/*JP2: Check MCU datasheet for Selection."
- note removed: "*MEMS1/*C2: Optional check MCU datasheet for values."
- note removed: "*R4/*R5/*JP3/*JP4: I2C Optional components."
- note removed: "*U1: Check the pinout for the desired MCU family."
- note removed: "*U2/*R3/*R6/*R7/*LED2/*LED3: EUSART Optional components."
