File: Kicad/nano/pic16bit.kicad_pcb (KiCad board)
At the start: 2 copper layers, 21 x 52 mm, 37 parts, among them IC3 ROHM-BU33SD5WG-500-SOT, K1 MCU 1, K2 MCU 2, K3 ICSP, K4 POWER & UART

Commit message: Update Nano
Routing:
- net GND: track 88.2 -> 87.0 mm

Commit message: Update
Parts:
- added kibuzzard-6288ACA8: G***, kibuzzard-6288ACA8, F.Cu at (104.9, 85.4)
- added kibuzzard-6288ACB7: G***, kibuzzard-6288ACB7, F.Cu at (104.6, 82.9)
- added kibuzzard-6288ACD9: G***, kibuzzard-6288ACD9, F.Cu at (116.4, 82.9)
- added kibuzzard-6288ACE7: G***, kibuzzard-6288ACE7, F.Cu at (116.1, 85.4)

Commit message: Up
Parts:
- removed *IC1: PIC24/dsPIC33, tronixio:TQFP-44
- removed *IC2: MCP2221A, tronixio:TSSOP-14
- removed IC3: ROHM-BU33SD5WG-500-SOT, tronixio:SOT-23-5
- added U1: PIC24/dsPIC33, tronixio:TQFP-44, F.Cu at (110.5, 75.2)
- added U2: MCP2221A, tronixio:TSSOP-14, B.Cu at (110.5, 59.5)
- added U3: ROHM-BU33SD5WG-500-SOT, tronixio:SOT-23-5, B.Cu at (110.5, 50.1)

Commit message: Update
Parts:
- F1: value F050 -> 500mA
- JP1: renamed from *JP1; value 0R -> 0
- JP2: renamed from *JP2; value 0R -> 0
- MEMS1: renamed from *MEMS1; value MICROCHIP-DSC1001C-245760-CDFN -> DSC1001C
- U2: value MCP2221A -> MCP2221A-IST
- U3: value ROHM-BU33SD5WG-500-SOT -> BU33SD5WG
- renumbered *C2 to C2, *C6 to C6, *JP3 to JP3, *JP4 to JP4, *LED2 to LED2, *LED3 to LED3, *R3 to R3, *R4 to R4, *R5 to R5, *R6 to R6, *R7 to R7

Commit message: Update
Parts:
- U1: value PIC24/dsPIC33 -> PIC24/dsPIC32
Changed lines of the file:
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@@
       (effects (font (size 1 1) (thickness 0.15)))
     )
-    (fp_text value "PIC24/dsPIC33" (at 0 1.270001 135) (layer "F.Fab")
+    (fp_text value "PIC24/dsPIC32" (at 0 1.270001 135) (layer "F.Fab")
       (effects (font (size 1 1) (thickness 0.15)))
     )
@@
   (footprint "tronixio:FUSE-0805" (layer "B.Cu")
     (at 112.75 53.25 180)
-    (property "Mouser" "652-MF-NSMF050-2")
-    (property "Name" "BOURNS-FUSE-MF-NSMF050")
-    (property "Sheetfile" "pic16bit.kicad_sch")
-    (property "Sheetname" "")
+    (property "Mouser" "652-MF-PSMF050X-2")
+    (property "Name" "BOURNS-FUSE-MF-PSMF050X")
+    (property "Sheetfile" "pic16bit.kicad_sch")
+    (property "Sheetname" "")

Commit message: Update
Parts:
- C1, C2, C3, C4, C5, C6, C7, C8: footprint tronixio:CAPACITOR-0805 -> tronixio:CAPACITOR-SMD-0805
- F1: footprint tronixio:FUSE-0805 -> tronixio:FUSE-SMD-0805
- JP1, JP2, R1, R2, R3, R4, R5, R6, R7, R8: footprint tronixio:RESISTOR-0805 -> tronixio:RESISTOR-SMD-0805
- LED1, LED2, LED3: footprint tronixio:LED-0805 -> tronixio:LED-SMD-0805

Commit message: Update
Parts:
- U2: value MCP2221A-IST -> MCP2221A
Changed lines of the file:
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@@
     (at 109.5 65.25 90)
     (property "Mouser" "855-M22-25102")
-    (property "Name" "HARWIN-200-M-1X02-JUMPER-TH-VERTICAL")
     (property "Sheetfile" "pic16bit.kicad_sch")
     (property "Sheetname" "")
@@
     (at 116.25 97.25 -90)
     (property "Mouser" "604-APT2012LVBCD")
-    (property "Name" "KINGBRIGHT-LED-0805-BLUE")
     (property "Sheetfile" "pic16bit.kicad_sch")
     (property "Sheetname" "")
@@
     (at 107.96 98.5 90)
     (property "Mouser" "855-M20-9980346")
-    (property "Name" "MICROCHIP-ICSP-M-2X03")
     (property "Sheetfile" "pic16bit.kicad_sch")
     (property "Sheetname" "")
@@
     (at 110.5 75.235 -45)
     (property "Mouser" "579-FJ64GA104-I/PT")
-    (property "Name" "MICROCHIP-PIC24FJ64GA104-IPT")
     (property "Sheetfile" "pic16bit.kicad_sch")
     (property "Sheetname" "")
@@
     (at 109.5 63.25 90)
     (property "Mouser" "855-M22-25102")
-    (property "Name" "HARWIN-200-M-1X02-JUMPER-TH-VERTICAL")
     (property "Sheetfile" "pic16bit.kicad_sch")
     (property "Sheetname" "")
@@
     (at 110.5 50.65 -90)
     (property "Mouser" "649-10118193-0001LF")
-    (property "Name" "FCI-USB-TYPE-B-MICRO-THT")
     (property "Sheetfile" "pic16bit.kicad_sch")
     (property "Sheetname" "")
@@
     (at 116.5 50.5 90)
     (property "Mouser" "604-APT2012LVBCD")
-    (property "Name" "KINGBRIGHT-LED-0805-BLUE")
     (property "Sheetfile" "pic16bit.kicad_sch")
     (property "Sheetname" "")
@@
     (at 104.75 97.25 90)
     (property "Mouser" "660-RK73B2ATTDD103J")
-    (property "Name" "RESISTOR-0805-10K")
     (property "Sheetfile" "pic16bit.kicad_sch")
     (property "Sheetname" "")
@@
     (at 110.5 90.75)
     (property "Mouser" "688-SKRPACE010")
-    (property "Name" "ALPS-SKRPAC")
     (property "Sheetfile" "pic16bit.kicad_sch")
     (property "Sheetname" "")
@@
     (at 104.5 50.5 90)
     (property "Mouser" "604-APT2012LVBCD")
-    (property "Name" "KINGBRIGHT-LED-0805-BLUE")
     (property "Sheetfile" "pic16bit.kicad_sch")
     (property "Sheetname" "")
@@
     (at 112.75 70 180)
     (property "Mouser" "660-RK73Z2ATTD")
-    (property "Name" "RESISTOR-0805-0")
-    (property "Sheetfile" "pic16bit.kicad_sch")
-    (property "Sheetname" "")
-    (property "Tolerance" "~")
+    (property "Sheetfile" "pic16bit.kicad_sch")
+    (property "Sheetname" "")
+    (property "Tolerance" "5%")
     (zone_connect 2)
     (attr smd)
@@
     (at 108.25 78.5 180)
     (property "Mouser" "80-C0805C104M5R")
-    (property "Name" "CAPACITOR-0805-100N")
     (property "Sheetfile" "pic16bit.kicad_sch")
     (property "Sheetname" "")
@@
     (at 116.5 50.5 90)
     (property "Mouser" "660-RK73B2ATTDD472J")
-    (property "Name" "RESISTOR-0805-4K7")
     (property "Sheetfile" "pic16bit.kicad_sch")
     (property "Sheetname" "")
@@
     (at 119.39 49.835 180)
     (property "Mouser" "200-TSW12022TS")
-    (property "Name" "SAMTEC-254-M-TSW-1X20-22-T-S_1")
     (property "Sheetfile" "pic16bit.kicad_sch")
     (property "Sheetname" "")
@@
     (at 110.5 50.1)
     (property "Mouser" "755-BU33SD5WG-TR")
-    (property "Name" "ROHM-BU33SD5WG-500-SOT-23")
     (property "Sheetfile" "pic16bit.kicad_sch")
     (property "Sheetname" "")
@@
     (at 110.5 59.5 180)
     (property "Mouser" "579-MCP2221A-I/ST")
-    (property "Name" "MICROCHIP-MCP2221A-IST")
     (property "Sheetfile" "pic16bit.kicad_sch")
     (property "Sheetname" "")
@@
       (effects (font (size 1 1) (thickness 0.15)) (justify mirror))
     )
-    (fp_text value "MCP2221A-IST" (at 0 -4) (layer "B.Fab")
+    (fp_text value "MCP2221A" (at 0 -4) (layer "B.Fab")
       (effects (font (size 1 1) (thickness 0.15)) (justify mirror))
     )
@@
     (at 108.25 81 180)
     (property "Mouser" "80-C0805C104M5R")
-    (property "Name" "CAPACITOR-0805-100N")
     (property "Sheetfile" "pic16bit.kicad_sch")
     (property "Sheetname" "")
@@
     (at 115.75 58 -90)
     (property "Mouser" "660-RK73B2ATTDD103J")
-    (property "Name" "RESISTOR-0805-10K")
     (property "Sheetfile" "pic16bit.kicad_sch")
     (property "Sheetname" "")
@@
     (at 108.25 73.5)
     (property "Mouser" "80-C0805C106M3P")
-    (property "Name" "CAPACITOR-0805-10U")
     (property "Sheetfile" "pic16bit.kicad_sch")
     (property "Sheetname" "")
@@
     (at 104.5 50.5 90)
     (property "Mouser" "660-RK73B2ATTDD472J")
-    (property "Name" "RESISTOR-0805-4K7")
     (property "Sheetfile" "pic16bit.kicad_sch")
     (property "Sheetname" "")
@@
     (at 112.75 77.75 -90)
     (property "Mouser" "998-1001CI2-024.5760")
-    (property "Name" "MICROCHIP-DSC1001C-245760-CDFN")
     (property "Sheetfile" "pic16bit.kicad_sch")
     (property "Sheetname" "")
@@
     (at 104.75 97.25 -90)
     (property "Mouser" "660-RK73B2ATTDD102J")
-    (property "Name" "RESISTOR-0805-1K")
     (property "Sheetfile" "pic16bit.kicad_sch")
     (property "Sheetname" "")
@@
     (at 112.75 81)
     (property "Mouser" "80-C0805C104M5R")
-    (property "Name" "CAPACITOR-0805-100N")
     (property "Sheetfile" "pic16bit.kicad_sch")
     (property "Sheetname" "")
@@
     (at 101.61 49.835 180)
     (property "Mouser" "200-TSW12022TS")
-    (property "Name" "SAMTEC-254-M-TSW-1X20-22-T-S_1")
     (property "Sheetfile" "pic16bit.kicad_sch")
     (property "Sheetname" "")
@@
     (at 108.25 67.5)
     (property "Mouser" "660-RK73B2ATTDD472J")
-    (property "Name" "RESISTOR-0805-4K7")
     (property "Sheetfile" "pic16bit.kicad_sch")
     (property "Sheetname" "")
@@
     (at 112.75 67.5 180)
     (property "Mouser" "660-RK73B2ATTDD472J")
-    (property "Name" "RESISTOR-0805-4K7")
     (property "Sheetfile" "pic16bit.kicad_sch")
     (property "Sheetname" "")
@@
     (at 112.75 55.5)
     (property "Mouser" "80-C0805C105M5R")
-    (property "Name" "CAPACITOR-0805-1U")
     (property "Sheetfile" "pic16bit.kicad_sch")
     (property "Sheetname" "")
@@
     (at 112.75 73.5 180)
     (property "Mouser" "80-C0805C104M5R")
-    (property "Name" "CAPACITOR-0805-100N")
     (property "Sheetfile" "pic16bit.kicad_sch")
     (property "Sheetname" "")
@@
     (at 108.25 70 180)
     (property "Mouser" "660-RK73Z2ATTD")
-    (property "Name" "RESISTOR-0805-0")
-    (property "Sheetfile" "pic16bit.kicad_sch")
-    (property "Sheetname" "")
-    (property "Tolerance" "~")
+    (property "Sheetfile" "pic16bit.kicad_sch")
+    (property "Sheetname" "")
+    (property "Tolerance" "5%")
     (zone_connect 2)
     (attr smd)
@@
     (at 108.25 53.25 180)
     (property "Mouser" "80-C0805C105M5R")
-    (property "Name" "CAPACITOR-0805-1U")
     (property "Sheetfile" "pic16bit.kicad_sch")
     (property "Sheetname" "")
@@
     (at 112.75 53.25 180)
     (property "Mouser" "652-MF-PSMF050X-2")
-    (property "Name" "BOURNS-FUSE-MF-PSMF050X")
     (property "Sheetfile" "pic16bit.kicad_sch")
     (property "Sheetname" "")
@@
     (at 108.25 76 180)
     (property "Mouser" "80-C0805C104M5R")
-    (property "Name" "CAPACITOR-0805-100N")
     (property "Sheetfile" "pic16bit.kicad_sch")
     (property "Sheetname" "")
@@
     (at 116.25 97.25 -90)
     (property "Mouser" "660-RK73B2ATTDD472J")
-    (property "Name" "RESISTOR-0805-4K7")
-    (property "Sheetfile" "pic16bit.kicad_sch")
-    (property "Sheetname" "")
+    (property "Sheetfile" "pic16bit.kicad_sch")
+    (property "Sheetname" "")
