File: Kicad/nano/pic16bit.kicad_pcb (KiCad board)
At the start: 2 copper layers, 21 x 52 mm, 45 parts, among them K1 MCU 1, K2 MCU 2, K3 ICSP, K4 POWER & UART, U1 PIC24/dsPIC32, U2 MCP2221A, U3 BU33SD5WG

Commit message: Up
Parts:
- K4: footprint tronixio:FCI-USB-TYPE-B-MICRO-THT -> tronixio:USB-TYPE-B-MICRO-TH

Commit message: Up
Changed lines of the file:
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@@
     (pad_to_mask_clearance 0)
     (aux_axis_origin 100 100)
-    (grid_origin 100 100)
     (pcbplotparams
       (layerselection 0x00011fc_ffffffff)
@@
   (net 43 "Net-(U2-SCL)")
   (net 44 "Net-(U2-SDA)")
-  (net 45 "unconnected-(K3-NC-Pad6)")
+  (net 45 "unconnected-(K3-Pad6)")
   (net 46 "Net-(K4-D-)")
   (net 47 "Net-(K4-D+)")
@@
   (footprint "tronixio:HARWIN-M20-998034x" (layer "F.Cu")
     (at 107.96 98.5 90)
-    (property "Mouser" "855-M20-9980346")
+    (property "Mouser" "855-M20-998034")
     (property "Sheetfile" "pic16bit.kicad_sch")
     (property "Sheetname" "")
+    (property "ki_description" "M20 Series - 2.54mm Pitch PCB Connector")
+    (property "ki_keywords" "200-TSW10308TD")
     (attr through_hole)
     (fp_text reference "K3" (at 0 0 90) (layer "F.SilkS") hide
@@
       (stroke (width 0.1) (type solid)) (layer "F.Fab"))
     (pad "1" thru_hole roundrect (at 0 0 90) (size 1.6 1.6) (drill 0.8) (layers "*.Cu" "*.Mask") (roundrect_rratio 0.1)
-      (net 11 "/~{MCLR}") (pinfunction "~{MCLR}") (pintype "input"))
+      (net 11 "/~{MCLR}") (pinfunction "1") (pintype "passive"))
     (pad "2" thru_hole roundrect (at 2.54 0 90) (size 1.6 1.6) (drill 0.8) (layers "*.Cu" "*.Mask") (roundrect_rratio 0.1)
-      (net 1 "+3V3") (pinfunction "VDD") (pintype "power_in"))
+      (net 1 "+3V3") (pinfunction "2") (pintype "passive"))
     (pad "3" thru_hole roundrect (at 0 2.54 90) (size 1.6 1.6) (drill 0.8) (layers "*.Cu" "*.Mask") (roundrect_rratio 0.1)
-      (net 2 "GND") (pinfunction "GND") (pintype "passive"))
+      (net 2 "GND") (pinfunction "3") (pintype "passive"))
     (pad "4" thru_hole roundrect (at 2.54 2.54 90) (size 1.6 1.6) (drill 0.8) (layers "*.Cu" "*.Mask") (roundrect_rratio 0.1)
-      (net 32 "/RB0{slash}PGD") (pinfunction "PGD") (pintype "bidirectional"))
+      (net 32 "/RB0{slash}PGD") (pinfunction "4") (pintype "passive"))
     (pad "5" thru_hole roundrect (at 0 5.08 90) (size 1.6 1.6) (drill 0.8) (layers "*.Cu" "*.Mask") (roundrect_rratio 0.1)
-      (net 33 "/RB1{slash}PGC") (pinfunction "PGC") (pintype "input"))
+      (net 33 "/RB1{slash}PGC") (pinfunction "5") (pintype "passive"))
     (pad "6" thru_hole roundrect (at 2.54 5.08 90) (size 1.6 1.6) (drill 0.8) (layers "*.Cu" "*.Mask") (roundrect_rratio 0.1)
-      (net 45 "unconnected-(K3-NC-Pad6)") (pinfunction "NC") (pintype "no_connect"))
+      (net 45 "unconnected-(K3-Pad6)") (pinfunction "6") (pintype "passive+no_connect"))
     (model "${KICAD_USER_3DMODEL_DIR}/Header/HARWIN-M20-998034x.wrl"
       (offset (xyz 0 0 0))
@@
   (footprint "tronixio:RESISTOR-SMD-0805" (layer "B.Cu")
     (at 112.75 70 180)
-    (property "Mouser" "")
+    (property "Mouser" "660-RK73Z2ATTD")
     (property "Sheetfile" "pic16bit.kicad_sch")
     (property "Sheetname" "")
-    (property "Tolerance" "~%")
+    (property "Tolerance" "")
     (property "ki_description" "Resistor")
     (zone_connect 2)
@@
   (footprint "tronixio:CAPACITOR-SMD-0805" (layer "B.Cu")
     (at 108.25 78.5 180)
-    (property "Mouser" "80-C0805C104M5R")
+    (property "Mouser" "80-C0805C104J5")
     (property "Sheetfile" "pic16bit.kicad_sch")
     (property "Sheetname" "")
-    (property "Tolerance" "20%")
+    (property "Tolerance" "5%")
     (property "Voltage" "50V")
     (property "ki_description" "Unpolarized Capacitor")
@@
   (footprint "tronixio:CAPACITOR-SMD-0805" (layer "B.Cu")
     (at 108.25 81 180)
-    (property "Mouser" "80-C0805C104M5R")
+    (property "Mouser" "80-C0805C104J5")
     (property "Sheetfile" "pic16bit.kicad_sch")
     (property "Sheetname" "")
-    (property "Tolerance" "20%")
+    (property "Tolerance" "5%")
     (property "Voltage" "50V")
     (property "ki_description" "Unpolarized Capacitor")
@@
   (footprint "tronixio:CAPACITOR-SMD-0805" (layer "B.Cu")
     (at 108.25 73.5)
-    (property "Mouser" "80-C0805C106M9P")
+    (property "Mouser" "81-GRM21BZ71E106KE5L")
     (property "Sheetfile" "pic16bit.kicad_sch")
     (property "Sheetname" "")
-    (property "Tolerance" "20%")
-    (property "Voltage" "6V3")
+    (property "Tolerance" "10%")
+    (property "Voltage" "25V")
     (property "ki_description" "Unpolarized Capacitor")
     (attr smd)
@@
   (footprint "tronixio:CAPACITOR-SMD-0805" (layer "B.Cu")
     (at 112.75 81)
-    (property "Mouser" "80-C0805C104M5R")
+    (property "Mouser" "80-C0805C104J5")
     (property "Sheetfile" "pic16bit.kicad_sch")
     (property "Sheetname" "")
-    (property "Tolerance" "20%")
+    (property "Tolerance" "5%")
     (property "Voltage" "50V")
     (property "ki_description" "Unpolarized Capacitor")
@@
   (footprint "tronixio:CAPACITOR-SMD-0805" (layer "B.Cu")
     (at 112.75 55.5)
-    (property "Mouser" "80-C0805C105M4R")
+    (property "Mouser" "187-CL21B105KBFNNNE")
     (property "Sheetfile" "pic16bit.kicad_sch")
     (property "Sheetname" "")
-    (property "Tolerance" "20%")
-    (property "Voltage" "16V")
+    (property "Tolerance" "10%")
+    (property "Voltage" "50V")
     (property "ki_description" "Unpolarized Capacitor")
     (attr smd)
@@
   (footprint "tronixio:CAPACITOR-SMD-0805" (layer "B.Cu")
     (at 112.75 73.5 180)
-    (property "Mouser" "80-C0805C104M5R")
+    (property "Mouser" "80-C0805C104J5")
     (property "Sheetfile" "pic16bit.kicad_sch")
     (property "Sheetname" "")
-    (property "Tolerance" "20%")
+    (property "Tolerance" "5%")
     (property "Voltage" "50V")
     (property "ki_description" "Unpolarized Capacitor")
@@
   (footprint "tronixio:RESISTOR-SMD-0805" (layer "B.Cu")
     (at 108.25 70 180)
-    (property "Mouser" "")
+    (property "Mouser" "660-RK73Z2ATTD")
     (property "Sheetfile" "pic16bit.kicad_sch")
     (property "Sheetname" "")
-    (property "Tolerance" "~%")
+    (property "Tolerance" "")
     (property "ki_description" "Resistor")
     (zone_connect 2)
@@
   (footprint "tronixio:CAPACITOR-SMD-0805" (layer "B.Cu")
     (at 108.25 53.25 180)
-    (property "Mouser" "80-C0805C105M4R")
+    (property "Mouser" "187-CL21B105KBFNNNE")
     (property "Sheetfile" "pic16bit.kicad_sch")
     (property "Sheetname" "")
-    (property "Tolerance" "20%")
-    (property "Voltage" "16V")
+    (property "Tolerance" "10%")
+    (property "Voltage" "50V")
     (property "ki_description" "Unpolarized Capacitor")
     (attr smd)
@@
     (property "Sheetfile" "pic16bit.kicad_sch")
     (property "Sheetname" "")
-    (property "ki_description" "MF-NSMF Series - PTC Resettable Fuses")
     (zone_connect 2)
     (attr smd)
@@
   (footprint "tronixio:CAPACITOR-SMD-0805" (layer "B.Cu")
     (at 108.25 76 180)
-    (property "Mouser" "80-C0805C104M5R")
+    (property "Mouser" "80-C0805C104J5")
     (property "Sheetfile" "pic16bit.kicad_sch")
     (property "Sheetname" "")
-    (property "Tolerance" "20%")
+    (property "Tolerance" "5%")
     (property "Voltage" "50V")
     (property "ki_description" "Unpolarized Capacitor")
@@
   (gr_circle (center 110.5 76.75) (end 110.7 76.75)
     (stroke (width 0.1) (type solid)) (fill solid) (layer "B.SilkS"))
-  (gr_circle (center 109.1 52) (end 109.35 52)
-    (stroke (width 0.1) (type solid)) (fill solid) (layer "B.SilkS"))
   (gr_circle (center 113.5 56.75) (end 113.75 56.75)
     (stroke (width 0.1) (type solid)) (fill solid) (layer "B.SilkS"))
@@
     )
     (stroke (width 0.1) (type solid)) (fill solid) (layer "B.SilkS"))
+  (gr_circle (center 111.5 67.5) (end 111.25 67.5)
+    (stroke (width 0.1) (type solid)) (fill solid) (layer "F.SilkS"))
   (gr_poly
     (pts
