File: Kicad/nano/pic16bit.kicad_pcb (KiCad board)
At the start: 2 copper layers, 21 x 52 mm, 45 parts, among them K1 MCU 1, K2 MCU 2, K3 ICSP, K4 POWER & UART, U1 PIC24/dsPIC32, U2 MCP2221A, U3 BU33SD5WG

Commit message: Update Nano
Connections:
- net POWER-+3V3 renamed +3V3
- net POWER-GND renamed GND
Routing:
- net /RB1/PGC: track 32.0 -> 32.5 mm
- net /RB0/PGD: track 26.0 -> 26.5 mm

Commit message: Up
Parts:
- U1: value PIC24/dsPIC32 -> PIC24/dsPIC33

Commit message: Up
Parts:
- H1, H2: footprint tronixio:HARWIN-M22-190-193 -> tronixio:HARWIN-M22-190-19X
