File: Kicad/nano/pic16bit.kicad_pcb (KiCad board)
At the start: 2 copper layers, 21 x 52 mm, 45 parts, among them K1 MCU 1, K2 MCU 2, K3 ICSP, K4 POWER & UART, U1 PIC24/dsPIC33, U2 MCP2221A, U3 BU33SD5WG

Commit message: Up
Parts:
- moved K1 35.0 mm to (136.6, 49.8)
- moved K3 35.0 mm to (143.0, 98.5)
- moved C1 35.0 mm to (143.2, 81.0)
- moved C2 35.0 mm to (147.8, 81.0)
- moved C3 35.0 mm to (143.2, 78.5)
- moved C4 35.0 mm to (147.8, 73.5)
- moved C5 35.0 mm to (143.2, 76.0)
- moved C6 35.0 mm to (143.2, 73.5)
- moved C7 35.0 mm to (143.2, 53.2)
- moved C8 35.0 mm to (147.8, 55.5)
- moved F1 35.0 mm to (147.8, 53.2)
- moved GB 35.0 mm to (145.5, 92.8)
- moved GT 35.0 mm to (145.5, 85.0)
- moved H1 35.0 mm to (149.0, 104.2)
- moved H2 35.0 mm to (154.1, 104.2)
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