File: Kicad/trainer/pic16bit.kicad_pcb (KiCad board)
At the start: 2 copper layers, 160 x 100 mm, 119 parts, among them K101 AC/DC 9-12V, K102 AC/DC 9-12V, K103 PE-450-4X6X-BLACK, K201 MCU 1, K202 MCU 2, K203 ICSP, K204 VIN, K205 VIN, K206 VDD, K207 GND, K208 VDD, K209 GND, K210 HARWIN-254-F-1X10-VERTICAL, K301 I2C/GPIO, K302 I2C/SPI, K303 SPI/GPIO, K304 EUSART/TTL, K401 HARWIN-254-F-1X10-VERTICAL, K402 HARWIN-254-F-1X10-VERTICAL, K409 HARWIN-254-F-1X16-VERTICAL, P401 AN1, P402 AN2, U101 KEYSTONE-24283, U102 KEYSTONE-24283, U103 KEYSTONE-24283, U104 KEYSTONE-24283, U105 NCP5662-ADJ, U201 PIC16F/18F, X1 XTAL-DIL08, X101 3M-SJ5376, X102 3M-SJ5376, X103 3M-SJ5376, X104 3M-SJ5376, X105 3M-SJ5376

Commit message: Update
Parts:
- removed K302: I2C/SPI, tronixio:HARWIN-M20-974034x
- removed X1: XTAL-DIL08, tronixio:DIP-08-W762-SOCKET
- added C204: 100n, tronixio:KEMET-C315, F.Cu at (162.9, 89.8)
- added JP204: VREG, tronixio:HARWIN-M20-975034x, F.Cu at (140.7, 110.0)
- added X201: XTAL-DIL08, tronixio:DIP-08-W762-SOCKET, F.Cu at (168.5, 77.0)
- U201: value PIC16F/18F -> PIC24/dsPIC33; footprint tronixio:DIP-28-W762 -> tronixio:DIP-28-W762-SOCKET
Connections:
- net /MCU/RA0/SPI_SC3 renamed /MCU/RA0/SPI_CS3
- net ~{MCLR} renamed Net-(K201-Pad1)
- JP202 pad 2: /MCU/RC3/SCL/SCK -> /MCU/RB8/I2C_SCL
- JP203 pad 2: /MCU/RC4/SDA/MISO -> /MCU/RB9/I2C_SDA
- K201 pad 11: Net-(K201-Pad11) -> /MCU/RB4/URTS
- K201 pad 12: /MCU/RC1/I2C_INT -> /MCU/RA4/UCTS
- K201 pad 13: /MCU/RC2/I2C_RESET -> VDD
- K201 pad 14: /MCU/RC3/SCL/SCK -> /MCU/RB5/I2C_RESET
- K201 pad 4: /MCU/RA2/SPI_RESET -> /MCU/RB0/UTX
- K201 pad 5: /MCU/RA3/SPI_INT -> /MCU/RB1/URX
- K201 pad 6: Net-(JP201-Pad1) -> /MCU/RB2/SPI_RESET
- K201 pad 7: /MCU/RA5/SPI_CS -> Net-(K201-Pad7)
- K202 pad 1: PGD -> VDD
- K202 pad 10: GND -> Net-(JP204-Pad2)
- K202 pad 11: /MCU/RC7/URX -> /MCU/RB9/I2C_SDA
- K202 pad 12: /MCU/RC6/UTX -> /MCU/RB8/I2C_SCL
- K202 pad 13: /MCU/RC5/MOSI -> /MCU/RB7/INT
- K202 pad 14: /MCU/RC4/SDA/MISO -> Net-(K202-Pad14)
- K202 pad 2: PGC -> GND
- K202 pad 3: /MCU/RB5/UCTS -> /MCU/RB15/SPI_CS
- K202 pad 4: /MCU/RB4/URTS -> Net-(K202-Pad4)
- K202 pad 5: Net-(K202-Pad5) -> /MCU/RB13/SPI_MISO
- K202 pad 7: Net-(K202-Pad7) -> /MCU/RB11/SPI_SCK
- K202 pad 8: Net-(K202-Pad8) -> /MCU/RB10/SPI_MOSI
- K202 pad 9: VDD -> Net-(JP201-Pad1)
- K203 pad 2: PGC -> /MCU/RB1/URX
- K203 pad 3: PGD -> /MCU/RB0/UTX
- R301 pad 1: /MCU/RC1/I2C_INT -> /MCU/RB7/INT
- R302 pad 1: /MCU/RC2/I2C_RESET -> /MCU/RB5/I2C_RESET
- R303 pad 1: RC3/SCL -> /MCU/RB8/I2C_SCL
- R304 pad 1: RC4/SDA -> /MCU/RB9/I2C_SDA
- R305 pad 1: /MCU/RA5/SPI_CS -> /MCU/RB15/SPI_CS
- R306 pad 1: /MCU/RC5/MOSI -> /MCU/RB10/SPI_MOSI
- R307 pad 1: RC4/MISO -> /MCU/RB13/SPI_MISO
- R308 pad 1: RC3/SCK -> /MCU/RB11/SPI_SCK
- R309 pad 2: /MCU/RA3/SPI_INT -> /MCU/RB7/INT
- R310 pad 2: /MCU/RA2/SPI_RESET -> /MCU/RB2/SPI_RESET
- R313 pad 1: /MCU/RB5/UCTS -> /MCU/RA4/UCTS
- R314 pad 1: /MCU/RC6/UTX -> /MCU/RB0/UTX
- R315 pad 1: /MCU/RC7/URX -> /MCU/RB1/URX
- U201 pad 11: Net-(K201-Pad11) -> /MCU/RB4/URTS
- U201 pad 12: /MCU/RC1/I2C_INT -> /MCU/RA4/UCTS
- U201 pad 13: /MCU/RC2/I2C_RESET -> VDD
- U201 pad 14: /MCU/RC3/SCL/SCK -> /MCU/RB5/I2C_RESET
- U201 pad 15: /MCU/RC4/SDA/MISO -> Net-(K202-Pad14)
- U201 pad 16: /MCU/RC5/MOSI -> /MCU/RB7/INT
- U201 pad 17: /MCU/RC6/UTX -> /MCU/RB8/I2C_SCL
- U201 pad 18: /MCU/RC7/URX -> /MCU/RB9/I2C_SDA
- U201 pad 19: GND -> Net-(JP204-Pad2)
- U201 pad 20: VDD -> Net-(JP201-Pad1)
- U201 pad 21: Net-(K202-Pad8) -> /MCU/RB10/SPI_MOSI
- U201 pad 22: Net-(K202-Pad7) -> /MCU/RB11/SPI_SCK
- U201 pad 24: Net-(K202-Pad5) -> /MCU/RB13/SPI_MISO
- U201 pad 25: /MCU/RB4/URTS -> Net-(K202-Pad4)
- U201 pad 26: /MCU/RB5/UCTS -> /MCU/RB15/SPI_CS
- U201 pad 27: PGC -> GND
- U201 pad 28: PGD -> VDD
- U201 pad 4: /MCU/RA2/SPI_RESET -> /MCU/RB0/UTX
- U201 pad 5: /MCU/RA3/SPI_INT -> /MCU/RB1/URX
- U201 pad 6: Net-(JP201-Pad1) -> /MCU/RB2/SPI_RESET
- U201 pad 7: /MCU/RA5/SPI_CS -> Net-(K201-Pad7)
Routing:
- net /MCU/RC4/SDA/MISO: track 211.2 -> 0.00 mm, vias 1 -> 0
- net /MCU/RB8/I2C_SCL: track 0.00 -> 193.9 mm, vias 0 -> 1
- net /MCU/RB9/I2C_SDA: track 0.00 -> 190.8 mm, vias 0 -> 1
- net /MCU/RB7/INT: track 0.00 -> 176.0 mm, vias 0 -> 2
- net /MCU/RC3/SCL/SCK: track 172.4 -> 0.00 mm, vias 1 -> 0
- net /MCU/RC5/MOSI: track 155.4 -> 0.00 mm, vias 1 -> 0
- net /MCU/RB11/SPI_SCK: track 0.00 -> 141.1 mm, vias 0 -> 2
- net /MCU/RB10/SPI_MOSI: track 0.00 -> 140.1 mm, vias 0 -> 2
- net /MCU/RB15/SPI_CS: track 0.00 -> 138.5 mm
- net /MCU/RB13/SPI_MISO: track 0.00 -> 138.0 mm, vias 0 -> 2
- net /MCU/RB1/URX: track 0.00 -> 114.6 mm, vias 0 -> 3
- net /MCU/RB0/UTX: track 0.00 -> 111.9 mm, vias 0 -> 3
- net /MCU/RC1/I2C_INT: track 103.5 -> 0.00 mm
- net /MCU/RC2/I2C_RESET: track 101.4 -> 0.00 mm, vias 1 -> 0
- net /MCU/RB5/I2C_RESET: track 0.00 -> 100.3 mm, vias 0 -> 1
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Other:
- board text added: "VDD"
- board text added: "VREG"
- board text removed: "SPI - I2C"

Commit message: Update
Parts:
- removed JP103: HARWIN-JUMPER-0254-06MM-RED, tronixio:HARWIN-M20-7580-7583
- added kibuzzard-6313AD44: G***, kibuzzard-6313AD44, F.Cu at (140.7, 97.5)
- added kibuzzard-6313AD54: G***, kibuzzard-6313AD54, F.Cu at (145.7, 97.5)
- added kibuzzard-6313AEE5: G***, kibuzzard-6313AEE5, F.Cu at (179.3, 106.4)
- added kibuzzard-6313AEF3: G***, kibuzzard-6313AEF3, F.Cu at (179.3, 119.1)
- moved kibuzzard-62ACBAD0 20.3 mm to (224.5, 88.6)
- moved kibuzzard-62A777FA 20.3 mm to (224.5, 91.1)
- moved JP102 8.00 mm to (181.0, 164.0)
- moved JP101 7.00 mm to (181.0, 156.0)
Routing:
- net GND: track 79.3 -> 75.7 mm, vias 17 -> 16
Other:
- board text added: "RA0/CS3 - RB11/SCK"
- board text added: "RA1/CS2 - RB13/MISO"
- board text added: "RA2/RESET - RB10/MOSI"
- board text added: "RB10"
- board text added: "RB11"
- board text added: "RB12"
- board text added: "RB13"
- board text added: "RB14"
- board text added: "RB15"
- board text added: "RB5/RESET"
- board text added: "RB7/INT"
- board text added: "RB7/INT - RB15/CS"
- board text added: "RB8"
- board text added: "RB8/SCL"
- board text added: "RB9"
- board text added: "RB9/SDA"
- board text removed: "GND"
- board text removed: "RA0/CS3 - RC3/SCK"
- board text removed: "RA1/CS2 - RC4/MISO"
- board text removed: "RA2/RST - RC5/MOSI"
- board text removed: "RA3/INT - RA5/CS"
- board text removed: "RA5"
- board text removed: "RA6"
- board text removed: "RA7"
- board text removed: "RC0"
- board text removed: "RC1"
- board text removed: "RC1/INT"
- board text removed: "RC2"
- board text removed: "RC2/RST"
- board text removed: "RC3"
- board text removed: "RC3/SCL"
- board text removed: "RC4"
- board text removed: "RC4/SDA"
- board text removed: "RC5"
- board text removed: "RC6"
- board text removed: "RC7"
- board text removed: "VDD"

Commit message: Update
Connections:
- net Net-(K201-Pad1) renamed /MCU/~{MCLR}
- K201 pad 4: /MCU/RB0/UTX -> /MCU/RB0/UTX/PGD
- K201 pad 5: /MCU/RB1/URX -> /MCU/RB1/URX/PGC
- K203 pad 2: /MCU/RB1/URX -> /MCU/RB1/URX/PGC
- K203 pad 3: /MCU/RB0/UTX -> /MCU/RB0/UTX/PGD
- R314 pad 1: /MCU/RB0/UTX -> /MCU/RB1/URX/PGC
- R315 pad 1: /MCU/RB1/URX -> /MCU/RB0/UTX/PGD
- U201 pad 4: /MCU/RB0/UTX -> /MCU/RB0/UTX/PGD
- U201 pad 5: /MCU/RB1/URX -> /MCU/RB1/URX/PGC
Routing:
- net /MCU/RB1/URX/PGC: track 0.00 -> 116.9 mm, vias 0 -> 3
- net /MCU/RB1/URX: track 114.6 -> 0.00 mm, vias 3 -> 0
- net /MCU/RB0/UTX: track 111.9 -> 0.00 mm, vias 3 -> 0
- net /MCU/RB0/UTX/PGD: track 0.00 -> 110.6 mm, vias 0 -> 3
- net Net-(EB401-Pad15): track 24.4 -> 21.4 mm

Commit message: Update Trainer
Parts:
- RA401: footprint tronixio:4611X -> tronixio:BOURNS-4611X

Commit message: Update Trainer
Routing:
- net /HID/S5: track 32.0 -> 33.2 mm
