File: Kicad/trainer/pic16bit.kicad_pcb (KiCad board)
At the start: 2 copper layers, 160 x 100 mm, 123 parts, among them K101 AC/DC 9-12V, K102 AC/DC 9-12V, K103 PE-450-4X6X-BLACK, K201 MCU 1, K202 MCU 2, K203 ICSP, K204 VIN, K205 VIN, K206 VDD, K207 GND, K208 VDD, K209 GND, K210 HARWIN-254-F-1X10-VERTICAL, K301 I2C/GPIO, K303 SPI/GPIO, K304 EUSART/TTL, K401 HARWIN-254-F-1X10-VERTICAL, K402 HARWIN-254-F-1X10-VERTICAL, K409 HARWIN-254-F-1X16-VERTICAL, P401 AN1, P402 AN2, U101 KEYSTONE-24283, U102 KEYSTONE-24283, U103 KEYSTONE-24283, U104 KEYSTONE-24283, U105 NCP5662-ADJ, U201 PIC24/dsPIC33, X101 3M-SJ5376, X102 3M-SJ5376, X103 3M-SJ5376, X104 3M-SJ5376, X105 3M-SJ5376, X201 XTAL-DIL08

Commit message: Up
Parts:
- U105: footprint tronixio:TO-263-5 -> tronixio:TO-263-5-TABPIN3
- turned U105 to 180 degrees
Routing:
- net POWER-VDD: track 479.4 -> 481.0 mm
- net /MCU/~{MCLR}: track 91.5 -> 92.4 mm

Commit message: Update pic16bit.kicad_pcb
Routing:
- net POWER-VDD: track 481.0 -> 482.0 mm
Changed lines of the file:
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@@
 			(at 2.54 4 0)
 			(layer "F.SilkS")
+			(hide yes)
 			(effects
 				(font
@@
 		(sheetfile "pic16bit-mcu.kicad_sch")
 		(attr through_hole)
+		(fp_line
+			(start -1.27 -2.8)
+			(end -1.27 -1.27)
+			(stroke
+				(width 0.2)
+				(type default)
+			)
+			(layer "F.SilkS")
+		)
+		(fp_line
+			(start -1.27 -1.27)
+			(end 6.35 -1.27)
+			(stroke
+				(width 0.2)
+				(type default)
+			)
+			(layer "F.SilkS")
+		)
+		(fp_line
+			(start 6.35 -1.27)
+			(end 6.35 -2.8)
+			(stroke
+				(width 0.2)
+				(type default)
+			)
+			(layer "F.SilkS")
+		)
 		(fp_rect
 			(start -1.27 1.27)
@@
 			)
 		)
-		(pad "1" thru_hole circle
+		(pad "1" thru_hole roundrect
 			(at 0 0)
-			(size 1.8 1.8)
+			(size 1.6 1.8)
 			(drill 0.8)
 			(layers "*.Cu" "*.Mask")
 			(remove_unused_layers no)
+			(roundrect_rratio 0.1)
 			(net 101 "POWER-VDD")
 			(pinfunction "1")
 			(pintype "passive")
 		)
-		(pad "2" thru_hole circle
+		(pad "2" thru_hole roundrect
 			(at 2.54 0)
-			(size 1.8 1.8)
+			(size 1.6 1.8)
 			(drill 0.8)
 			(layers "*.Cu" "*.Mask")
 			(remove_unused_layers no)
+			(roundrect_rratio 0.1)
 			(net 43 "Net-(K202-Pin_10)")
 			(pinfunction "2")
 			(pintype "passive")
 		)
-		(pad "3" thru_hole circle
+		(pad "3" thru_hole roundrect
 			(at 5.08 0)
-			(size 1.8 1.8)
+			(size 1.6 1.8)
 			(drill 0.8)
 			(layers "*.Cu" "*.Mask")
 			(remove_unused_layers no)
+			(roundrect_rratio 0.1)
 			(net 2 "POWER-GND")
 			(pinfunction "3")
@@
 		)
 		(property "Mouser" "863-NCP5662DSADJR4G"
-			(at 0 0 270)
+			(at 0 0 -90)
 			(layer "F.Fab")
 			(hide yes)
@@
 	)
 	(segment
-		(start 163.52 108.9)
-		(end 162.12 107.5)
+		(start 162.12 107.5)
+		(end 141.5 107.5)
 		(width 1)
 		(layer "F.Cu")
@@
 	)
 	(segment
+		(start 140.66 108.34)
+		(end 140.66 110)
+		(width 1)
+		(layer "F.Cu")
+		(net 101)
+	)
+	(segment
 		(start 131.5 64.25)
 		(end 131.5 75.8)
@@
 	)
 	(segment
-		(start 143.16 107.5)
-		(end 140.66 110)
+		(start 113.65 59.3)
+		(end 117.45 59.3)
 		(width 1)
 		(layer "F.Cu")
@@
 	)
 	(segment
-		(start 113.65 59.3)
-		(end 117.45 59.3)
+		(start 163.52 108.9)
+		(end 162.12 107.5)
 		(width 1)
 		(layer "F.Cu")
@@
 	)
 	(segment
-		(start 162.12 107.5)
-		(end 143.16 107.5)
+		(start 201.79 54.29)
+		(end 202.89 55.39)
 		(width 1)
 		(layer "F.Cu")
@@
 	)
 	(segment
-		(start 201.79 54.29)
-		(end 202.89 55.39)
+		(start 168.6 119.06)
+		(end 166.06 119.06)
 		(width 1)
 		(layer "F.Cu")
@@
 	)
 	(segment
-		(start 168.6 119.06)
-		(end 166.06 119.06)
+		(start 141.5 107.5)
+		(end 140.66 108.34)
 		(width 1)
 		(layer "F.Cu")

Commit message: Up
Parts:
- U101, U102, U103, U104: value KEYSTONE-24283 -> 24283

Commit message: Up
Parts:
- K101: footprint tronixio:CUI-PJ-102AH -> tronixio:SAMESKY-PJ-102AH
- K102: footprint tronixio:CUI-TB006-508-02BE -> tronixio:SAMESKY-TB006-508-02BE
- U101, U102, U103, U104: value 24283 -> KEYSTONE-24283
