File: Kicad/trainer/pic16bit.kicad_pcb (KiCad board)
At the start: 2 copper layers, 160 x 100 mm, 123 parts, among them K101 AC/DC 9-12V, K102 AC/DC 9-12V, K103 PE-450-4X6X-BLACK, K201 MCU 1, K202 MCU 2, K203 ICSP, K204 VIN, K205 VIN, K206 VDD, K207 GND, K208 VDD, K209 GND, K210 HARWIN-254-F-1X10-VERTICAL, K301 I2C/GPIO, K303 SPI/GPIO, K304 EUSART/TTL, K401 HARWIN-254-F-1X10-VERTICAL, K402 HARWIN-254-F-1X10-VERTICAL, K409 HARWIN-254-F-1X16-VERTICAL, P401 AN1, P402 AN2, U101 KEYSTONE-24283, U102 KEYSTONE-24283, U103 KEYSTONE-24283, U104 KEYSTONE-24283, U105 NCP5662-ADJ, U201 PIC24/dsPIC33, X101 3M-SJ5376, X102 3M-SJ5376, X103 3M-SJ5376, X104 3M-SJ5376, X105 3M-SJ5376, X201 XTAL-DIL08

Commit message: Up
Parts:
- removed kibuzzard-65F6F3C0: G***, kibuzzard-65F6F3C0
- K210: value HARWIN-254-F-1X10-VERTICAL -> VDD & GND
- K401: value HARWIN-254-F-1X10-VERTICAL -> LED ARRAY
- K402: value HARWIN-254-F-1X10-VERTICAL -> SWITCH, ENCODER & ANALOG
- K409: value HARWIN-254-F-1X16-VERTICAL -> EXPANSION BOARD
- U201: footprint tronixio:DIP-28-W762-SOCKET -> tronixio:DIP-28-W762
- moved R101 3.20 mm to (101.5, 48.5)
- moved S101 3.01 mm to (86.8, 49.0)
- moved K402 2.83 mm to (188.1, 127.3)
- moved B101 2.83 mm to (83.2, 54.5)
- moved BB401 2.83 mm to (199.5, 103.0)
- moved C101 2.83 mm to (120.0, 60.8)
- moved C102 2.83 mm to (120.0, 51.0)
- moved C201 2.83 mm to (171.7, 70.5)
- moved C202 2.83 mm to (157.5, 105.5)
- moved C203 2.83 mm to (161.5, 105.6)
- moved C204 2.83 mm to (160.9, 87.8)
- moved D301 2.83 mm to (70.7, 122.1)
- moved D302 2.83 mm to (70.7, 94.2)
- moved D303 2.83 mm to (70.7, 89.1)
- moved D304 2.83 mm to (219.3, 58.6)
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Connections:
- S403 pad 4: /HID/S5 -> POWER-GND
- S403 pad 5: POWER-GND -> /HID/S5
Other:
- board text removed: "JLCJLCJLCJLC"
