File: Kicad/trainer/pic16bit-mod.kicad_sch (KiCad schematic)
At the start: 23 parts

Commit message: Update
Parts:
- D301, D302, D303, D304: value (none) -> ESDA14V2SC5Y; footprint (none) -> tronixio:SOT-23-5
- K301: value (none) -> I2C/GPIO; footprint (none) -> tronixio:SAMTEC-SSW-106-02-T-S-RA
- K303: value (none) -> SPI/GPIO; footprint (none) -> tronixio:SAMTEC-SSW-106-02-T-D-RA
- K304: value (none) -> EUSART/TTL; footprint (none) -> tronixio:SAMTEC-SSW-106-02-T-S-RA
- R301, R302, R303, R304, R305, R306, R307, R308, R309, R310, R311, R312, R313, R314, R315, R316: value (none) -> 200Ω; footprint (none) -> tronixio:RESISTOR-SMD-1206

Commit message: Update
Connections:
- net RB0/UTX renamed RB0/UTX/PGD
- net RB1/URX renamed RB1/URX/PGC
Changed lines of the file:
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@@
     (effects (font (size 1.15 1.15)) (justify left))
   )
-  (hierarchical_label "RB1{slash}URX" (shape output) (at 187.96 48.26 180)
+  (hierarchical_label "RB1{slash}URX{slash}PGC" (shape output) (at 187.96 48.26 180)
     (effects (font (size 1.15 1.15)) (justify right))
   )
@@
     (effects (font (size 1.15 1.15)) (justify right))
   )
-  (hierarchical_label "RB0{slash}UTX" (shape input) (at 187.96 45.72 180)
+  (hierarchical_label "RB0{slash}UTX{slash}PGD" (shape input) (at 187.96 45.72 180)
     (effects (font (size 1.15 1.15)) (justify right))
   )

Commit message: Update Trainer
Parts:
- D301, D302, D303, D304: Name ST-ESDA14V2SC5Y-SOT-23 -> (none)
- K301, K304: Name SAMTEC-SSW-106-02-T-S-RA -> (none)
- K303: Name SAMTEC-SSW-106-02-T-D-RA -> (none)
- R301, R302, R303, R304, R305, R306, R307, R308, R309, R310, R311, R312, R313, R314, R315, R316: symbol tronixio:RESISTOR-1206-200R -> tronixio:KOASPEER-RK73B-1206-200R-5P; Name RESISTOR-1206-200R -> (none)

Commit message: Up
Parts:
- R301, R302, R303, R304, R305, R306, R307, R308, R309, R310, R311, R312, R313, R314, R315, R316: symbol tronixio:KOASPEER-RK73B-1206-200R-5P -> tronixio:RESISTOR-1206-200R-5P
