File: Kicad/trainer/pic16bit-mcu.kicad_sch (KiCad schematic)
At the start: 25 parts, among them U201 PIC24/dsPIC33

Commit message: Update
Parts:
- C201, C203: value (none) -> 100n; footprint (none) -> tronixio:KEMET-C315
- C202: footprint (none) -> tronixio:KEMET-C322
- JP201: value (none) -> VCAP; footprint (none) -> tronixio:HARWIN-M20-975024x
- JP202: footprint (none) -> tronixio:HARWIN-M20-999024x
- JP203: value (none) -> SDA; footprint (none) -> tronixio:HARWIN-M20-999024x
- K201: value (none) -> MCU 1; footprint (none) -> tronixio:HARWIN-M20-782144x
- K202: value (none) -> MCU 2; footprint (none) -> tronixio:HARWIN-M20-782144x
- K203: value (none) -> ICSP; footprint (none) -> tronixio:SAMTEC-SSW-106-02-T-S-RA
- K204: value (none) -> VIN; footprint (none) -> tronixio:HARWIN-M20-782044x
- K205: value (none) -> VIN; footprint (none) -> tronixio:HARWIN-M20-999044x
- K206: value (none) -> VDD; footprint (none) -> tronixio:HARWIN-M20-782044x
- K207: value (none) -> GND; footprint (none) -> tronixio:HARWIN-M20-782044x
- K208: value (none) -> VDD; footprint (none) -> tronixio:HARWIN-M20-999044x
- K209: value (none) -> GND; footprint (none) -> tronixio:HARWIN-M20-999044x
- K210: value (none) -> HARWIN-254-F-1X10-VERTICAL; footprint (none) -> tronixio:HARWIN-M20-782104x
- R201: value (none) -> 10K; footprint (none) -> tronixio:RESISTOR-TH-1016
- R202: value (none) -> 1K; footprint (none) -> tronixio:RESISTOR-TH-1016
- R203, R204: value (none) -> 4K7; footprint (none) -> tronixio:RESISTOR-TH-1016
- S201: value (none) -> Reset; footprint (none) -> tronixio:CK-KSA-TH
- U201: footprint (none) -> tronixio:DIP-28-W762-SOCKET
- X201: renamed from X1; value (none) -> XTAL-DIL08; footprint (none) -> tronixio:DIP-08-W762-SOCKET
- gave numbers to parts that had none: 2
Connections:
- net ~{MCLR}: no longer names the net of K201.1 (Pin_1), K203.6, R202.1, U201.1 (~{MCLR})
Other:
- note added: "*X201: Optional mounted on DIL08"
- note removed: "*X1: Optional mounted on DIL08"
- moved on the sheet: C201, C202, C203, C204, JP201, JP202, JP203, JP204, K201, K202, K203, K204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

Commit message: Update
Connections:
- net ~{MCLR}: now reaches K201.1 (Pin_1), K203.6, R202.1, U201.1 (~{MCLR})
- net RB0/UTX renamed RB0/UTX/PGD
- net RB1/URX renamed RB1/URX/PGC
Changed lines of the file:
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@@
     (effects (font (size 1.15 1.15)) (justify right bottom))
+  )
+  (label "~{MCLR}" (at 63.5 60.96 0)
+    (effects (font (size 1.15 1.15)) (justify left bottom))
   )
   (hierarchical_label "RB10{slash}SPI_MOSI" (shape output) (at 220.98 109.22 0)
@@
     (effects (font (size 1.15 1.15)) (justify left))
   )
-  (hierarchical_label "RB0{slash}UTX" (shape input) (at 63.5 114.3 180)
+  (hierarchical_label "RB0{slash}UTX{slash}PGD" (shape input) (at 63.5 114.3 180)
     (effects (font (size 1.15 1.15)) (justify right))
   )
@@
     (effects (font (size 1.15 1.15)) (justify right))
   )
-  (hierarchical_label "RB1{slash}URX" (shape output) (at 63.5 111.76 180)
+  (hierarchical_label "RB1{slash}URX{slash}PGC" (shape output) (at 63.5 111.76 180)
     (effects (font (size 1.15 1.15)) (justify right))
   )

Commit message: Update
Parts:
- U201: footprint tronixio:DIP-28-W762-SOCKET -> (none)
Other:
- moved on the sheet: JP201, JP202, JP203
Changed lines of the file:
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@@
-    (stroke (width 0) (type solid) (color 0 0 0 0))
-  )
-  (wire (pts (xy 190.5 45.72) (xy 190.5 48.26))
     (stroke (width 0) (type solid) (color 0 0 0 0))
   )
@@
     (stroke (width 0) (type default) (color 0 0 0 0))
   )
-  (wire (pts (xy 175.26 104.14) (xy 175.26 106.68))
-    (stroke (width 0) (type solid) (color 0 0 0 0))
-  )
   (wire (pts (xy 63.5 68.58) (xy 78.74 68.58))
     (stroke (width 0) (type default) (color 0 0 0 0))
@@
   (wire (pts (xy 66.04 167.64) (xy 66.04 165.1))
     (stroke (width 0) (type default) (color 0 0 0 0))
-  )
-  (wire (pts (xy 198.12 45.72) (xy 198.12 48.26))
-    (stroke (width 0) (type solid) (color 0 0 0 0))
   )
   (wire (pts (xy 63.5 83.82) (xy 104.14 83.82))
@@
     (effects (font (size 1.15 1.15)) (justify left))
   )
-  (symbol (lib_id "tronixio:HARWIN-254-M-1X02-JUMPER-HORIZONTAL") (at 175.26 99.06 0) (mirror y) (unit 1)
-    (in_bom yes) (on_board yes)
-    (property "Reference" "JP201" (id 0) (at 175.895 96.52 0)
+  (symbol (lib_id "tronixio:HARWIN-254-M-1X02-JUMPER-HORIZONTAL") (at 175.26 101.6 0) (mirror y) (unit 1)
+    (in_bom yes) (on_board yes)
+    (property "Reference" "JP201" (id 0) (at 175.895 97.79 0)
       (effects (font (size 1.15 1.15)) (justify right))
     )
-    (property "Value" "VCAP" (id 1) (at 175.895 104.775 0)
+    (property "Value" "VCAP" (id 1) (at 175.895 105.41 0)
       (effects (font (size 1.15 1.15)) (justify right))
     )
-    (property "Footprint" "tronixio:HARWIN-M20-975024x" (id 2) (at 175.26 114.3 0)
-      (effects (font (size 1 1)) hide)
-    )
-    (property "Datasheet" "https://www.harwin.com/products/M20-9750246/" (id 3) (at 175.26 116.84 0)
-      (effects (font (size 1 1)) hide)
-    )
-    (property "Mouser" "855-M20-975024" (id 4) (at 175.26 119.38 0)
-      (effects (font (size 1 1)) hide)
-    )
-    (property "Name" "HARWIN-254-M-1X02-JUMPER-VERTICAL" (id 5) (at 175.26 111.76 0)
+    (property "Footprint" "tronixio:HARWIN-M20-975024x" (id 2) (at 175.26 116.84 0)
+      (effects (font (size 1 1)) hide)
+    )
+    (property "Datasheet" "https://www.harwin.com/products/M20-9750246/" (id 3) (at 175.26 119.38 0)
+      (effects (font (size 1 1)) hide)
+    )
+    (property "Mouser" "855-M20-975024" (id 4) (at 175.26 121.92 0)
+      (effects (font (size 1 1)) hide)
+    )
+    (property "Name" "HARWIN-254-M-1X02-JUMPER-VERTICAL" (id 5) (at 175.26 114.3 0)
       (effects (font (size 1 1)) hide)
     )
@@
       (effects (font (size 1.15 1.15)) (justify right))
     )
-    (property "Footprint" "tronixio:DIP-28-W762-SOCKET" (id 2) (at 144.78 101.6 0)
+    (property "Footprint" "" (id 2) (at 144.78 101.6 0)
       (effects (font (size 1 1)) hide)
     )
@@
     (pin "1")
   )
-  (symbol (lib_id "tronixio:HARWIN-254-M-1X02-JUMPER-VERTICAL") (at 198.12 50.8 0) (mirror y) (unit 1)
-    (in_bom yes) (on_board yes)
-    (property "Reference" "JP203" (id 0) (at 204.47 48.26 0)
-      (effects (font (size 1.15 1.15)) (justify left))
-    )
-    (property "Value" "SDA" (id 1) (at 202.565 55.88 0)
-      (effects (font (size 1.15 1.15)) (justify left))
+  (symbol (lib_name "HARWIN-254-M-1X02-JUMPER-VERTICAL_1") (lib_id "tronixio:HARWIN-254-M-1X02-JUMPER-VERTICAL") (at 198.12 50.8 0) (mirror y) (unit 1)
+    (in_bom yes) (on_board yes)
+    (property "Reference" "JP203" (id 0) (at 198.755 46.99 0)
+      (effects (font (size 1.15 1.15)) (justify right))
+    )
+    (property "Value" "SDA" (id 1) (at 198.755 55.245 0)
+      (effects (font (size 1.15 1.15)) (justify right))
     )
     (property "Footprint" "tronixio:HARWIN-M20-999024x" (id 2) (at 198.12 66.04 0)
@@
   (symbol (lib_id "tronixio:HARWIN-254-M-1X02-JUMPER-VERTICAL") (at 190.5 50.8 0) (mirror y) (unit 1)
     (in_bom yes) (on_board yes)
-    (property "Reference" "JP202" (id 0) (at 191.135 48.26 0)
+    (property "Reference" "JP202" (id 0) (at 191.135 46.99 0)
       (effects (font (size 1.15 1.15)) (justify right))
     )
-    (property "Value" "SCL" (id 1) (at 191.135 55.88 0)
+    (property "Value" "SCL" (id 1) (at 191.135 55.245 0)
       (effects (font (size 1.15 1.15)) (justify right))
     )

Commit message: Update Trainer
Parts:
- C201, C203, C204: symbol tronixio:KEMET-C315-100N-254 -> tronixio:KEMET-C315-0254-100N-50V-20P; Name KEMET-C315-100N-254 -> (none); Voltage (none) -> 50V
- C202: symbol tronixio:KEMET-C322-10U-508 -> tronixio:KEMET-C322-0508-10U-25V-10P; Name KEMET-C32210U-508 -> (none); Voltage (none) -> 25V
- JP201, JP202, JP203: Name HARWIN-254-M-1X02-JUMPER-VERTICAL -> (none)
- JP204: Name HARWIN-254-M-1X03-RIGHT-ANGLE -> (none)
- K201, K202: Name HARWIN-254-F-1X14-VERTICAL -> (none)
- K203: Name MICROCHIP-ICSP-F-1X06 -> (none)
- K204, K206, K207: Name HARWIN-254-F-1X04-VERTICAL -> (none)
- K205, K208, K209: Name HARWIN-254-M-1X04-VERTICAL -> (none)
- K210: Name HARWIN-254-F-1X10-VERTICAL -> (none)
- R201: Name RESISTOR-1016TH-10K -> (none)
- R202: Name RESISTOR-1016TH-1K -> (none)
- R203, R204: Name RESISTOR-1016TH-4K7 -> (none)
- S201: Name CK-KSA -> (none)
- U201: footprint (none) -> tronixio:DIP-28-W762-SOCKET
- X201: Name XTAL-DIL08 -> (none)

Commit message: Update
Parts:
- K203: symbol tronixio:MICROCHIP-ICSP-F-1X06 -> tronixio:MICROCHIP-ICSP-F-RIGHT-ANGLE-TH
- R201: symbol tronixio:RESISTOR-1016TH-10K -> tronixio:RESISTOR-1016TH-10K-5P
- R202: symbol tronixio:RESISTOR-1016TH-1K -> tronixio:RESISTOR-1016TH-1K-5P
- R203, R204: symbol tronixio:RESISTOR-1016TH-4K7 -> tronixio:RESISTOR-1016TH-4K7-5P
- U201: footprint tronixio:DIP-28-W762-SOCKET -> (none)
Connections:
- net GND: no longer X201.2, X201.7, X201.8
- net at K201.10 (Pin_10), U201.10 (RA3/CLKO), X201.5: no longer X201.6
- net at K201.9 (Pin_9), U201.9 (RA2/CLKI), X201.3: no longer X201.4
- net VDD renamed +VDD
- net VIN renamed +VIN
Changed lines of the file:
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@@
       (effects (font (size 1 1)) hide)
-    )
-    (property "Name" "GND" (at 162.56 120.65 0)
-      (effects (font (size 1.15 1.15)) hide)
     )
     (pin "1")
@@
       (effects (font (size 1 1)) hide)
     )
-    (property "Name" "GND" (at 81.28 58.42 0)
-      (effects (font (size 1.15 1.15)) hide)
-    )
     (pin "1")
     (instances
@@
     )
   )
-  (symbol (lib_id "tronixio:POWER-VDD") (at 167.64 33.02 0) (unit 1)
+  (symbol (lib_id "tronixio:POWER-+VDD") (at 167.64 33.02 0) (unit 1)
     (in_bom yes) (on_board yes) (dnp no) (fields_autoplaced)
     (property "Reference" "#PWR0136" (at 167.64 43.18 0)
@@
     )
   )
-  (symbol (lib_id "tronixio:POWER-VDD") (at 218.44 127 0) (unit 1)
+  (symbol (lib_id "tronixio:POWER-+VDD") (at 218.44 127 0) (unit 1)
     (in_bom yes) (on_board yes) (dnp no)
     (property "Reference" "#PWR0135" (at 218.44 137.16 0)
@@
     (property "Datasheet" "" (at 127 187.96 0)
       (effects (font (size 1 1)) hide)
-    )
-    (property "Name" "GND" (at 127 191.77 0)
-      (effects (font (size 1.15 1.15)) hide)
     )
     (pin "1")
@@
     )
   )
-  (symbol (lib_id "tronixio:POWER-VDD") (at 111.76 160.02 0) (unit 1)
+  (symbol (lib_id "tronixio:POWER-+VDD") (at 111.76 160.02 0) (unit 1)
     (in_bom yes) (on_board yes) (dnp no)
     (property "Reference" "#PWR0123" (at 111.76 170.18 0)
@@
       (effects (font (size 1 1)) hide)
     )
-    (property "Name" "GND" (at 167.64 120.65 0)
-      (effects (font (size 1.15 1.15)) hide)
-    )
     (pin "1")
     (instances
@@
       (effects (font (size 1 1)) hide)
     )
-    (property "Name" "GND" (at 96.52 120.65 0)
-      (effects (font (size 1.15 1.15)) hide)
-    )
     (pin "1")
     (instances
@@
       (effects (font (size 1 1)) hide)
     )
-    (property "Name" "GND" (at 96.52 191.77 0)
-      (effects (font (size 1.15 1.15)) hide)
-    )
     (pin "1")
     (instances
@@
     )
   )
-  (symbol (lib_id "tronixio:POWER-VDD") (at 185.42 33.02 0) (unit 1)
+  (symbol (lib_id "tronixio:POWER-+VDD") (at 185.42 33.02 0) (unit 1)
     (in_bom yes) (on_board yes) (dnp no) (fields_autoplaced)
     (property "Reference" "#PWR0137" (at 185.42 43.18 0)
@@
       (effects (font (size 1.15 1.15)) (justify right))
     )
-    (property "Footprint" "tronixio:DIP-28-W762-SOCKET" (at 144.78 101.6 0)
+    (property "Footprint" "" (at 144.78 101.6 0)
       (effects (font (size 1 1)) hide)
     )
@@
     )
   )
-  (symbol (lib_id "tronixio:POWER-VDD") (at 190.5 33.02 0) (unit 1)
+  (symbol (lib_id "tronixio:POWER-+VDD") (at 190.5 33.02 0) (unit 1)
     (in_bom yes) (on_board yes) (dnp no)
     (property "Reference" "#PWR0138" (at 190.5 43.18 0)
@@
     )
   )
-  (symbol (lib_id "tronixio:POWER-VIN") (at 81.28 160.02 0) (unit 1)
+  (symbol (lib_id "tronixio:POWER-+VIN") (at 81.28 160.02 0) (unit 1)
     (in_bom yes) (on_board yes) (dnp no)
     (property "Reference" "#PWR0116" (at 81.28 170.18 0)
@@
       (effects (font (size 1 1)) hide)
     )
-    (property "Name" "GND" (at 185.42 120.65 0)
-      (effects (font (size 1.15 1.15)) hide)
-    )
     (pin "1")
     (instances
@@
     )
   )
-  (symbol (lib_id "tronixio:POWER-VDD") (at 81.28 33.02 0) (mirror y) (unit 1)
+  (symbol (lib_id "tronixio:POWER-+VDD") (at 81.28 33.02 0) (mirror y) (unit 1)
     (in_bom yes) (on_board yes) (dnp no) (fields_autoplaced)
     (property "Reference" "#PWR0126" (at 81.28 43.18 0)
@@
       (effects (font (size 1 1)) hide)
     )
-    (property "Datasheet" "https://www.harwin.com/products/M20-9990846/" (at 198.12 66.04 0)
+    (property "Datasheet" "https://www.harwin.com/products/M20-9990246/" (at 198.12 66.04 0)
       (effects (font (size 1 1)) hide)
     )
@@
     )
   )
-  (symbol (lib_id "tronixio:RESISTOR-1016TH-1K") (at 96.52 43.18 270) (unit 1)
+  (symbol (lib_id "tronixio:RESISTOR-1016TH-1K-5P") (at 96.52 43.18 270) (unit 1)
     (in_bom yes) (on_board yes) (dnp no)
     (property "Reference" "R202" (at 96.52 40.64 90)
@@
     )
   )
-  (symbol (lib_id "tronixio:POWER-VIN") (at 66.04 160.02 0) (unit 1)
+  (symbol (lib_id "tronixio:POWER-+VIN") (at 66.04 160.02 0) (unit 1)
     (in_bom yes) (on_board yes) (dnp no)
     (property "Reference" "#PWR0115" (at 66.04 170.18 0)
@@
     )
   )
-  (symbol (lib_id "tronixio:RESISTOR-1016TH-4K7") (at 190.5 40.64 0) (unit 1)
+  (symbol (lib_id "tronixio:RESISTOR-1016TH-4K7-5P") (at 190.5 40.64 0) (unit 1)
     (in_bom yes) (on_board yes) (dnp no)
     (property "Reference" "R203" (at 191.135 36.83 0)
@@
     )
   )
-  (symbol (lib_id "tronixio:MICROCHIP-ICSP-F-1X06") (at 223.52 129.54 0) (unit 1)
+  (symbol (lib_id "tronixio:MICROCHIP-ICSP-F-RIGHT-ANGLE-TH") (at 223.52 129.54 0) (unit 1)
     (in_bom yes) (on_board yes) (dnp no)
     (property "Reference" "K203" (at 223.52 127 0)
@@
     )
   )
-  (symbol (lib_id "tronixio:POWER-VDD") (at 127 160.02 0) (unit 1)
+  (symbol (lib_id "tronixio:POWER-+VDD") (at 127 160.02 0) (unit 1)
     (in_bom yes) (on_board yes) (dnp no)
     (property "Reference" "#PWR0122" (at 127 170.18 0)
@@
     )
   )
-  (symbol (lib_id "tronixio:RESISTOR-1016TH-4K7") (at 198.12 40.64 0) (unit 1)
+  (symbol (lib_id "tronixio:RESISTOR-1016TH-4K7-5P") (at 198.12 40.64 0) (unit 1)
     (in_bom yes) (on_board yes) (dnp no)
     (property "Reference" "R204" (at 198.755 36.83 0)
@@
       (effects (font (size 1 1)) hide)
     )
-    (property "Name" "GND" (at 121.92 120.65 0)
-      (effects (font (size 1.15 1.15)) hide)
-    )
     (pin "1")
     (instances
@@
     )
   )
-  (symbol (lib_id "tronixio:RESISTOR-1016TH-10K") (at 81.28 38.1 0) (mirror y) (unit 1)
+  (symbol (lib_id "tronixio:RESISTOR-1016TH-10K-5P") (at 81.28 38.1 0) (mirror y) (unit 1)
     (in_bom yes) (on_board yes) (dnp no)
     (property "Reference" "R201" (at 76.2 34.29 0)
@@
       (effects (font (size 1 1)) hide)
     )
-    (property "Name" "GND" (at 175.26 120.65 0)
-      (effects (font (size 1.15 1.15)) hide)
-    )
     (pin "1")
     (instances
@@
       (effects (font (size 1 1)) hide)
     )
-    (property "Datasheet" "https://www.harwin.com/products/M20-9990846/" (at 190.5 66.04 0)
+    (property "Datasheet" "https://www.harwin.com/products/M20-9990246/" (at 190.5 66.04 0)
       (effects (font (size 1 1)) hide)
     )
@@
       (effects (font (size 1 1)) hide)
     )
-    (property "Name" "GND" (at 127 120.65 0)
-      (effects (font (size 1.15 1.15)) hide)
-    )
     (pin "1")
     (instances
@@
       (effects (font (size 1 1)) hide)
     )
-    (property "Datasheet" "https://www.harwin.com/products/M20-7821446/" (at 121.92 193.04 0)
+    (property "Datasheet" "https://www.harwin.com/products/M20-7821406/" (at 121.92 193.04 0)
       (effects (font (size 1 1)) hide)
     )
@@
     )
   )
-  (symbol (lib_id "tronixio:POWER-VDD") (at 198.12 33.02 0) (unit 1)
+  (symbol (lib_id "tronixio:POWER-+VDD") (at 198.12 33.02 0) (unit 1)
     (in_bom yes) (on_board yes) (dnp no) (fields_autoplaced)
     (property "Reference" "#PWR0140" (at 198.12 43.18 0)
@@
     (property "Datasheet" "" (at 88.9 54.61 0)
       (effects (font (size 1 1)) hide)
-    )
-    (property "Name" "GND" (at 88.9 58.42 0)
-      (effects (font (size 1.15 1.15)) hide)
     )
     (pin "1")
@@
     (property "Datasheet" "" (at 218.44 144.78 0)
       (effects (font (size 1 1)) hide)
-    )
-    (property "Name" "GND" (at 218.44 148.59 0)
-      (effects (font (size 1.15 1.15)) hide)
     )
     (pin "1")
@@
     )
   )
-  (symbol (lib_id "tronixio:POWER-VDD") (at 96.52 160.02 0) (unit 1)
+  (symbol (lib_id "tronixio:POWER-+VDD") (at 96.52 160.02 0) (unit 1)
     (in_bom yes) (on_board yes) (dnp no)
     (property "Reference" "#PWR0125" (at 96.52 170.18 0)
@@
       (effects (font (size 1 1)) hide)
     )
-    (property "Name" "GND" (at 111.76 191.77 0)
-      (effects (font (size 1.15 1.15)) hide)
-    )
     (pin "1")
     (instances
@@
     )
   )
-  (symbol (lib_id "tronixio:POWER-VDD") (at 121.92 33.02 0) (unit 1)
+  (symbol (lib_id "tronixio:POWER-+VDD") (at 121.92 33.02 0) (unit 1)
     (in_bom yes) (on_board yes) (dnp no) (fields_autoplaced)
     (property "Reference" "#PWR0128" (at 121.92 43.18 0)
