File: Kicad/trainer/pic16bit-mcu.kicad_sch (KiCad schematic)
At the start: 25 parts, among them K201 MCU 1, K202 MCU 2, K203 ICSP, K204 VIN, K205 VIN, K206 VDD, K207 GND, K208 VDD, K209 GND, K210 HARWIN-254-F-1X10-VERTICAL, U201 PIC24/dsPIC33, X201 XTAL-DIL08

Commit message: Up
Parts:
- K210: value HARWIN-254-F-1X10-VERTICAL -> VDD & GND
- U201: footprint tronixio:DIP-28-W762-SOCKET -> tronixio:DIP-28-W762
Other:
- note added: "Notes: - *X201: Optional mounted on DIL08"
- note removed: "*X201: Optional mounted on DIL08"
- note removed: "PGC"
- note removed: "PGD"
