File: Kicad/trainer/pic16bit.kicad_sch (KiCad schematic)
At the start: 31 parts, among them K101 AC/DC 9-12V, K102 AC/DC 9-12V, K103 PE-450-4X6X-BLACK, U101 KEYSTONE-24283, U102 KEYSTONE-24283, U103 KEYSTONE-24283, U104 KEYSTONE-24283, U105 NCP5662-ADJ, X101 3M-SJ5376, X102 3M-SJ5376, X103 3M-SJ5376, X104 3M-SJ5376, X105 3M-SJ5376

Commit message: Update
Parts:
- removed JP103: HARWIN-JUMPER-0254-06MM-RED, tronixio:HARWIN-M20-7580-7583, symbol tronixio:HARWIN-JUMPER-0254-06MM-RED
Changed lines of the file:
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@@
     (pin "1")
   )
-  (symbol (lib_id "tronixio:HARWIN-JUMPER-0254-06MM-BLACK") (at 190.5 172.72 0) (unit 1)
-    (in_bom yes) (on_board yes) (fields_autoplaced)
-    (property "Reference" "JP101" (id 0) (at 190.5 170.18 0)
-      (effects (font (size 1 1)) hide)
-    )
-    (property "Value" "HARWIN-JUMPER-0254-06MM-BLACK" (id 1) (at 190.5 175.26 0)
-      (effects (font (size 1 1)) hide)
-    )
-    (property "Footprint" "tronixio:HARWIN-M20-7580-7583" (id 2) (at 190.5 177.8 0)
-      (effects (font (size 1 1)) hide)
-    )
-    (property "Datasheet" "https://cdn.harwin.com/pdfs/M7580-M7583.pdf" (id 3) (at 190.5 180.34 0)
-      (effects (font (size 1 1)) hide)
-    )
-    (property "Mouser" "855-M7582" (id 4) (at 190.5 182.88 0)
+  (symbol (lib_id "tronixio:HARWIN-JUMPER-0254-06MM-BLACK") (at 195.58 172.72 0) (unit 1)
+    (in_bom yes) (on_board yes) (fields_autoplaced)
+    (property "Reference" "JP101" (id 0) (at 195.58 170.18 0)
+      (effects (font (size 1 1)) hide)
+    )
+    (property "Value" "HARWIN-JUMPER-0254-06MM-BLACK" (id 1) (at 195.58 175.26 0)
+      (effects (font (size 1 1)) hide)
+    )
+    (property "Footprint" "tronixio:HARWIN-M20-7580-7583" (id 2) (at 195.58 177.8 0)
+      (effects (font (size 1 1)) hide)
+    )
+    (property "Datasheet" "https://cdn.harwin.com/pdfs/M7580-M7583.pdf" (id 3) (at 195.58 180.34 0)
+      (effects (font (size 1 1)) hide)
+    )
+    (property "Mouser" "855-M7582" (id 4) (at 195.58 182.88 0)
       (effects (font (size 1 1)) hide)
     )
@@
     )
     (pin "1")
-  )
-  (symbol (lib_id "tronixio:HARWIN-JUMPER-0254-06MM-RED") (at 200.66 172.72 0) (unit 1)
-    (in_bom yes) (on_board yes) (fields_autoplaced)
-    (property "Reference" "JP103" (id 0) (at 200.66 170.18 0)
-      (effects (font (size 1 1)) hide)
-    )
-    (property "Value" "HARWIN-JUMPER-0254-06MM-RED" (id 1) (at 200.66 175.26 0)
-      (effects (font (size 1 1)) hide)
-    )
-    (property "Footprint" "tronixio:HARWIN-M20-7580-7583" (id 2) (at 200.66 177.8 0)
-      (effects (font (size 1 1)) hide)
-    )
-    (property "Datasheet" "https://cdn.harwin.com/pdfs/M7580-M7583.pdf" (id 3) (at 200.66 180.34 0)
-      (effects (font (size 1 1)) hide)
-    )
-    (property "Mouser" "855-M7581" (id 4) (at 200.66 182.88 0)
-      (effects (font (size 1 1)) hide)
-    )
   )
   (symbol (lib_id "tronixio:POWER-GND") (at 152.4 60.96 0) (unit 1)
@@
     (pin "1")
   )
-  (symbol (lib_id "tronixio:HARWIN-JUMPER-0254-06MM-RED") (at 195.58 172.72 0) (unit 1)
-    (in_bom yes) (on_board yes) (fields_autoplaced)
-    (property "Reference" "JP102" (id 0) (at 195.58 170.18 0)
-      (effects (font (size 1 1)) hide)
-    )
-    (property "Value" "HARWIN-JUMPER-0254-06MM-RED" (id 1) (at 195.58 175.26 0)
-      (effects (font (size 1 1)) hide)
-    )
-    (property "Footprint" "tronixio:HARWIN-M20-7580-7583" (id 2) (at 195.58 177.8 0)
-      (effects (font (size 1 1)) hide)
-    )
-    (property "Datasheet" "https://cdn.harwin.com/pdfs/M7580-M7583.pdf" (id 3) (at 195.58 180.34 0)
-      (effects (font (size 1 1)) hide)
-    )
-    (property "Mouser" "855-M7581" (id 4) (at 195.58 182.88 0)
+  (symbol (lib_id "tronixio:HARWIN-JUMPER-0254-06MM-RED") (at 200.66 172.72 0) (unit 1)
+    (in_bom yes) (on_board yes) (fields_autoplaced)
+    (property "Reference" "JP102" (id 0) (at 200.66 170.18 0)
+      (effects (font (size 1 1)) hide)
+    )
+    (property "Value" "HARWIN-JUMPER-0254-06MM-RED" (id 1) (at 200.66 175.26 0)
+      (effects (font (size 1 1)) hide)
+    )
+    (property "Footprint" "tronixio:HARWIN-M20-7580-7583" (id 2) (at 200.66 177.8 0)
+      (effects (font (size 1 1)) hide)
+    )
+    (property "Datasheet" "https://cdn.harwin.com/pdfs/M7580-M7583.pdf" (id 3) (at 200.66 180.34 0)
+      (effects (font (size 1 1)) hide)
+    )
+    (property "Mouser" "855-M7581" (id 4) (at 200.66 182.88 0)
       (effects (font (size 1 1)) hide)
     )
@@
     (pin "1")
   )
-  (symbol (lib_id "tronixio:PE-450-4X6X-BLACK") (at 182.88 172.72 0) (unit 1)
-    (in_bom yes) (on_board yes) (fields_autoplaced)
-    (property "Reference" "K103" (id 0) (at 182.88 170.18 0)
-      (effects (font (size 1 1)) hide)
-    )
-    (property "Value" "PE-450-4X6X-BLACK" (id 1) (at 182.88 175.26 0)
-      (effects (font (size 1 1)) hide)
-    )
-    (property "Footprint" "tronixio:PE-450-4X6X" (id 2) (at 182.88 177.8 0)
-      (effects (font (size 1 1)) hide)
-    )
-    (property "Datasheet" "https://www.mouser.fr/datasheet/2/209/EPD-200220-1171146.pdf" (id 3) (at 182.88 180.34 0)
-      (effects (font (size 1 1)) hide)
-    )
-    (property "Mouser" "450-476" (id 4) (at 182.88 182.88 0)
+  (symbol (lib_id "tronixio:PE-450-4X6X-BLACK") (at 187.96 172.72 0) (unit 1)
+    (in_bom yes) (on_board yes) (fields_autoplaced)
+    (property "Reference" "K103" (id 0) (at 187.96 170.18 0)
+      (effects (font (size 1 1)) hide)
+    )
+    (property "Value" "PE-450-4X6X-BLACK" (id 1) (at 187.96 175.26 0)
+      (effects (font (size 1 1)) hide)
+    )
+    (property "Footprint" "tronixio:PE-450-4X6X" (id 2) (at 187.96 177.8 0)
+      (effects (font (size 1 1)) hide)
+    )
+    (property "Datasheet" "https://www.mouser.fr/datasheet/2/209/EPD-200220-1171146.pdf" (id 3) (at 187.96 180.34 0)
+      (effects (font (size 1 1)) hide)
+    )
+    (property "Mouser" "450-476" (id 4) (at 187.96 182.88 0)
       (effects (font (size 1 1)) hide)
     )
@@
       (reference "JP102") (unit 1) (value "HARWIN-JUMPER-0254-06MM-RED") (footprint "tronixio:HARWIN-M20-7580-7583")
     )
-    (path "/8521a876-aa47-4339-a3a8-9eeab785d9c7"
-      (reference "JP103") (unit 1) (value "HARWIN-JUMPER-0254-06MM-RED") (footprint "tronixio:HARWIN-M20-7580-7583")
-    )
     (path "/64edc06d-d6ae-4dac-9759-3f1fbed6457d/1053a8dc-ecbc-4592-be7e-05c72088176f"

Commit message: Update
Other:
- sheet MCU ports: added RB0/UTX/PGD, RB1/URX/PGC; removed RB0/UTX, RB1/URX
- sheet Module ports: added RB0/UTX/PGD, RB1/URX/PGC; removed RB0/UTX, RB1/URX
Changed lines of the file:
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@@
       (effects (font (size 1.27 1.27)) (justify left top))
-    )
-    (pin "RB1{slash}URX" output (at 121.92 119.38 0)
-      (effects (font (size 1.27 1.27)) (justify right))
-    )
-    (pin "RB0{slash}UTX" input (at 121.92 121.92 0)
-      (effects (font (size 1.27 1.27)) (justify right))
     )
     (pin "RA1{slash}SPI_CS2" output (at 121.92 109.22 0)
@@
       (effects (font (size 1.27 1.27)) (justify right))
     )
+    (pin "RB1{slash}URX{slash}PGC" output (at 121.92 119.38 0)
+      (effects (font (size 1.27 1.27)) (justify right))
+    )
+    (pin "RB0{slash}UTX{slash}PGD" input (at 121.92 121.92 0)
+      (effects (font (size 1.27 1.27)) (justify right))
+    )
   )
   (sheet (at 76.2 139.7) (size 45.72 45.72)
@@
       (effects (font (size 1.27 1.27)) (justify left))
     )
-    (pin "RB0{slash}UTX" input (at 167.64 121.92 180)
-      (effects (font (size 1.27 1.27)) (justify left))
-    )
     (pin "RB4{slash}URTS" output (at 167.64 116.84 180)
-      (effects (font (size 1.27 1.27)) (justify left))
-    )
-    (pin "RB1{slash}URX" output (at 167.64 119.38 180)
       (effects (font (size 1.27 1.27)) (justify left))
     )
@@
       (effects (font (size 1.27 1.27)) (justify left))
     )
+    (pin "RB0{slash}UTX{slash}PGD" input (at 167.64 119.38 180)
+      (effects (font (size 1.27 1.27)) (justify left))
+    )
+    (pin "RB1{slash}URX{slash}PGC" output (at 167.64 121.92 180)
+      (effects (font (size 1.27 1.27)) (justify left))
+    )

Commit message: Update Trainer
Parts:
- B101: Name ONSEMI-DF01M -> (none)
- C101, C102: Name NICHICON-UVZ-220U-25V -> (none)
- K101: Name CUI-PJ-102AH-TH -> (none)
- K102: Name CUI-TB006-508-02BE -> (none)
- LED101: Name KINGBRIGHT-LED-05MM-TH -> (none)
- R101: Name VISHAY-5K-64W -> (none)
- R102: Name RESISTOR-1016TH-4K7 -> (none)
- S101: Name CK-1101M2 -> (none)
- TP101, TP102, TP103: Name KEYSTONE-5006 -> (none)
- TP104: Name KEYSTONE-2000-3 -> (none)
- U105: Name ONSEMI-NCP5662-ADJ-TO263 -> (none)

Commit message: Up
Other:
- title: Power -> Root & Power

Commit message: Update
Parts:
- C101, C102: footprint tronixio:CAPACITOR-ELECTROLYTIC-RADIAL-080-110-035 -> tronixio:CAPACITOR-ELECTROLYTIC-RADIAL-080-115-035
Changed lines of the file:
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@@
       (effects (font (size 1.15 1.15)) (justify right))
     )
-    (property "Footprint" "tronixio:CAPACITOR-ELECTROLYTIC-RADIAL-080-110-035" (at 114.3 66.04 0)
+    (property "Footprint" "tronixio:CAPACITOR-ELECTROLYTIC-RADIAL-080-115-035" (at 114.3 66.04 0)
       (effects (font (size 1 1)) hide)
     )
@@
     )
     (property "Voltage" "25V" (at 115.57 60.96 0)
-      (effects (font (size 1.15 1.15)) (justify left) hide)
+      (effects (font (size 1.15 1.15)) (justify left))
     )
     (property "Tolerance" "20%" (at 119.38 60.96 0)
@@
       (effects (font (size 1.15 1.15)) (justify left))
     )
-    (property "Footprint" "tronixio:CAPACITOR-ELECTROLYTIC-RADIAL-080-110-035" (at 152.4 66.04 0)
+    (property "Footprint" "tronixio:CAPACITOR-ELECTROLYTIC-RADIAL-080-115-035" (at 152.4 66.04 0)
       (effects (font (size 1 1)) hide)
     )
@@
     )
     (property "Voltage" "25V" (at 153.67 60.96 0)
-      (effects (font (size 1.15 1.15)) (justify left) hide)
+      (effects (font (size 1.15 1.15)) (justify left))
     )
     (property "Tolerance" "20%" (at 157.48 60.96 0)

Commit message: Update
Parts:
- C101, C102: Life (none) -> 1000H; Serie (none) -> UVZ
- R101: symbol tronixio:VISHAY-5K-64W -> tronixio:TRIMMER-64W-5K
- R102: symbol tronixio:RESISTOR-1016TH-4K7 -> tronixio:RESISTOR-1016TH-4K7-5P
Connections:
- net VDD renamed +VDD
- net VIN renamed +VIN
Changed lines of the file:
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@@
       (effects (font (size 1 1)) hide)
-    )
-    (property "Name" "GND" (at 203.2 64.77 0)
-      (effects (font (size 1.15 1.15)) hide)
     )
     (pin "1")
@@
       (effects (font (size 1 1)) hide)
     )
-    (property "Name" "GND" (at 114.3 64.77 0)
-      (effects (font (size 1.15 1.15)) hide)
-    )
     (pin "1")
     (instances
@@
     (property "Datasheet" "" (at 167.64 60.96 0)
       (effects (font (size 1 1)) hide)
-    )
-    (property "Name" "GND" (at 167.64 64.77 0)
-      (effects (font (size 1.15 1.15)) hide)
     )
     (pin "1")
@@
     )
   )
-  (symbol (lib_id "tronixio:VISHAY-5K-64W") (at 144.78 55.88 0) (mirror y) (unit 1)
+  (symbol (lib_id "tronixio:TRIMMER-64W-5K") (at 144.78 55.88 0) (mirror y) (unit 1)
     (in_bom yes) (on_board yes) (dnp no)
     (property "Reference" "R101" (at 145.415 51.435 0)
@@
       (effects (font (size 1 1)) hide)
     )
-    (property "Name" "GND" (at 96.52 64.77 0)
-      (effects (font (size 1.15 1.15)) hide)
-    )
     (pin "1")
     (instances
@@
     )
   )
-  (symbol (lib_id "tronixio:POWER-VIN") (at 175.26 180.34 0) (unit 1)
+  (symbol (lib_id "tronixio:POWER-+VIN") (at 175.26 180.34 0) (unit 1)
     (in_bom yes) (on_board yes) (dnp no)
     (property "Reference" "#PWR0111" (at 175.26 190.5 0)
@@
       (effects (font (size 1 1)) hide)
     )
-    (property "Name" "GND" (at 167.64 194.31 0)
-      (effects (font (size 1.15 1.15)) hide)
-    )
     (pin "1")
     (instances
@@
     (property "Datasheet" "" (at 152.4 60.96 0)
       (effects (font (size 1 1)) hide)
-    )
-    (property "Name" "GND" (at 152.4 64.77 0)
-      (effects (font (size 1.15 1.15)) hide)
     )
     (pin "1")
@@
       (effects (font (size 1 1)) hide)
     )
+    (property "Life" "1000H" (at 114.3 76.2 0)
+      (effects (font (size 1 1)) hide)
+    )
+    (property "Serie" "UVZ" (at 114.3 73.66 0)
+      (effects (font (size 1 1)) hide)
+    )
     (pin "1")
     (pin "2")
@@
     (property "Datasheet" "" (at 213.36 60.96 0)
       (effects (font (size 1 1)) hide)
-    )
-    (property "Name" "GND" (at 213.36 64.77 0)
-      (effects (font (size 1.15 1.15)) hide)
     )
     (pin "1")
@@
     )
   )
-  (symbol (lib_id "tronixio:RESISTOR-1016TH-4K7") (at 167.64 43.18 0) (unit 1)
+  (symbol (lib_id "tronixio:RESISTOR-1016TH-4K7-5P") (at 167.64 43.18 0) (unit 1)
     (in_bom yes) (on_board yes) (dnp no)
     (property "Reference" "R102" (at 168.275 39.37 0)
@@
     )
   )
-  (symbol (lib_id "tronixio:POWER-VDD") (at 167.64 35.56 0) (unit 1)
+  (symbol (lib_id "tronixio:POWER-+VDD") (at 167.64 35.56 0) (unit 1)
     (in_bom yes) (on_board yes) (dnp no) (fields_autoplaced)
     (property "Reference" "#PWR0108" (at 167.64 45.72 0)
@@
       (effects (font (size 1 1)) hide)
     )
-    (property "Name" "GND" (at 193.04 64.77 0)
-      (effects (font (size 1.15 1.15)) hide)
-    )
     (pin "1")
     (instances
@@
       (effects (font (size 1 1)) hide)
     )
-    (property "Name" "GND" (at 144.78 64.77 0)
-      (effects (font (size 1.15 1.15)) hide)
-    )
     (pin "1")
     (instances
@@
     )
   )
-  (symbol (lib_id "tronixio:POWER-VIN") (at 114.3 35.56 0) (unit 1)
+  (symbol (lib_id "tronixio:POWER-+VIN") (at 114.3 35.56 0) (unit 1)
     (in_bom yes) (on_board yes) (dnp no)
     (property "Reference" "#PWR0102" (at 114.3 45.72 0)
@@
       (effects (font (size 1 1)) hide)
     )
-    (property "Datasheet" "https://www.onsemi.com/products/discretes-drivers/diodes-rectifiers/rectifiers/df01m" (at 104.14 60.96 0)
+    (property "Datasheet" "https://www.onsemi.com/products/discrete-power-modules/rectifiers/DF01M" (at 104.14 60.96 0)
       (effects (font (size 1 1)) hide)
     )
@@
     )
   )
-  (symbol (lib_id "tronixio:POWER-VDD") (at 152.4 35.56 0) (unit 1)
+  (symbol (lib_id "tronixio:POWER-+VDD") (at 152.4 35.56 0) (unit 1)
     (in_bom yes) (on_board yes) (dnp no) (fields_autoplaced)
     (property "Reference" "#PWR0106" (at 152.4 45.72 0)
@@
       (effects (font (size 1 1)) hide)
     )
-    (property "Name" "GND" (at 182.88 64.77 0)
-      (effects (font (size 1.15 1.15)) hide)
-    )
     (pin "1")
     (instances
@@
     (property "Datasheet" "" (at 121.92 60.96 0)
       (effects (font (size 1 1)) hide)
-    )
-    (property "Name" "GND" (at 121.92 64.77 0)
-      (effects (font (size 1.15 1.15)) hide)
     )
     (pin "1")
@@
       (effects (font (size 1 1)) hide)
     )
+    (property "Life" "1000H" (at 152.4 76.2 0)
+      (effects (font (size 1 1)) hide)
+    )
+    (property "Serie" "UVZ" (at 152.4 73.66 0)
+      (effects (font (size 1 1)) hide)
+    )
