File: Kicad/trainer/pic16bit-hid.kicad_sch (KiCad schematic)
At the start: 18 parts, among them K401 HARWIN-254-F-1X10-VERTICAL, K402 HARWIN-254-F-1X10-VERTICAL, K409 HARWIN-254-F-1X16-VERTICAL, P401 AN1, P402 AN2

Commit message: Up
Parts:
- K401: value HARWIN-254-F-1X10-VERTICAL -> LED ARRAY
- K402: value HARWIN-254-F-1X10-VERTICAL -> SWITCH, ENCODER & ANALOG
- K409: value HARWIN-254-F-1X16-VERTICAL -> EXPANSION BOARD
Connections:
- net POWER-GND: now also S403.4; no longer S403.5
- net S5: now also S403.5; no longer S403.4
